File: Current/SweetBusiness/SweetBusinessDaughtercard/SweetBusinessDaughtercard.kicad_pcb (KiCad board)
At the start: 2 copper layers, 82.5 x 14.3 mm, 8 parts, among them K10 Jump Out, K11 Jump Out, K12 Jump Out, K13 Jump Out, SW1 SW_SPDT, SW2 SW_SPDT, SW3 SW_SPDT, SW4 SW_SPDT

Commit message: Nice changelog, idiot.
Parts:
- removed K10, K11, K12, K13: Jump Out, Connector_PinSocket_2.54mm:PinSocket_1x02_P2.54mm_Vertical
- added J0: Toggle Link, Connector_PinHeader_2.54mm:PinHeader_2x04_P2.54mm_Vertical, F.Cu at (88.9, 61.1)
Connections:
- SW1 pad 2: Net-(K10-Pad1) -> GND
- SW1 pad 3: Net-(K10-Pad2) -> col12
- SW2 pad 2: Net-(K11-Pad1) -> GND
- SW2 pad 3: Net-(SW2-Pad3) -> col13
- SW3 pad 2: Net-(K12-Pad1) -> GND
- SW3 pad 3: Net-(SW3-Pad3) -> col14
- SW4 pad 2: Net-(K13-Pad1) -> GND
- SW4 pad 3: Net-(SW4-Pad3) -> col15
Routing:
- net col15: track 0.00 -> 70.4 mm
- net col14: track 0.00 -> 49.3 mm
- net col13: track 0.00 -> 28.7 mm
- net Net-(SW3-Pad3): track 26.5 -> 0.00 mm
- net Net-(SW2-Pad3): track 26.3 -> 0.00 mm
- net Net-(K12-Pad1): track 25.6 -> 0.00 mm
- net Net-(K11-Pad1): track 25.4 -> 0.00 mm
- net Net-(SW4-Pad3): track 11.4 -> 0.00 mm
- net Net-(K10-Pad2): track 11.2 -> 0.00 mm
- net Net-(K13-Pad1): track 10.6 -> 0.00 mm
- net Net-(K10-Pad1): track 10.3 -> 0.00 mm
- net col12: track 0.00 -> 8.53 mm
- added copper zone on B.Cu, net GND
- added copper zone on F.Cu, net GND
Other:
- board text added: "JLCJLCJLCJLC"
- board text added: "Remove Child Before Folding"
- board text removed: "EN: Disengage daughtercard before servicing EO: Remove child before folding"
