File: Current/SweetBusiness/SweetBusinessRGBCore/SweetBusinessRGBCore.kicad_pcb (KiCad board)
At the start: 2 copper layers, 471.5 x 142.9 mm, 269 parts, among them J1 Bridge

Commit message: oh my god just stop
Parts:
- removed R1: 5k1, EDI:Passive_0402_1005Metric
- added G***: LOGO, EDI:BusinessTime, B.Cu at (77.4, 143.0)
- added J2: Toggle Link, Connector_PinHeader_2.54mm:PinHeader_2x04_P2.54mm_Vertical, F.Cu at (298.8, 132.7)
- added T1: Keyswitch, EDI:T8013-Z1BQ, F.Cu at (309.6, 136.5)
- added T2: Keyswitch, EDI:T8013-Z1BQ, F.Cu at (328.6, 136.5)
- added T3: Keyswitch, EDI:T8013-Z1BQ, F.Cu at (347.7, 136.5)
- added T4: Keyswitch, EDI:T8013-Z1BQ, F.Cu at (366.7, 136.5)
- moved G2 4.83 mm to (381.0, 170.7)
Connections:
- net VBUS renamed +3V3
Routing:
- net row0: track 0.00 -> 78.5 mm
- net col15: track 0.00 -> 67.0 mm
- net col14: track 0.00 -> 47.0 mm
- net col13: track 0.00 -> 28.6 mm
- net Net-(LD10-Pad3): track 133.1 -> 108.5 mm
- net LED: track 351.3 -> 373.3 mm
- net col12: track 0.00 -> 11.0 mm
- net Net-(LD12-Pad1): track 85.4 -> 79.9 mm
- net +3V3: track 313.9 -> 312.3 mm
Other:
- outline, holes or cut-outs redrawn
