File: Current/SweetBusiness/SweetBusinessRGBCore/SweetBusinessRGBCore.kicad_sch (KiCad schematic)
At the start: 266 parts, among them J1 Bridge

Commit message: oh my god just stop
Parts:
- removed R1: 5k1, EDI:Passive_0402_1005Metric, symbol Device:R_Small
- added J2: Toggle Link, Connector_PinHeader_2.54mm:PinHeader_2x04_P2.54mm_Vertical, symbol Connector_Generic:Conn_02x04_Odd_Even
- added T1, T2, T3, T4: Keyswitch, EDI:T8013-Z1BQ, symbol EDI:Keyswitch
Connections:
- net VBUS renamed +3V3
- new net col12: J2.8 (Pin_8), T1.2
- new net col13: J2.6 (Pin_6), T2.2
- new net col14: J2.4 (Pin_4), T3.2
- new net col15: J2.2 (Pin_2), T4.2
- new net row0: J2.1 (Pin_1), J2.3 (Pin_3), J2.5 (Pin_5), J2.7 (Pin_7), T1.1, T2.1, T3.1, T4.1
Other:
- moved on the sheet: J1

Commit message: Whole bunch of work!
Parts:
- LD1, LD10, LD100, LD101, LD102, LD103, LD104, LD105, LD106, LD107, LD108, LD109, LD11, LD110, LD111, LD112, LD113, LD114, LD115, LD116, LD117, LD118, LD119, LD12, LD120, LD121, LD122, LD123, LD124, LD125, LD126, LD127, LD13, LD14, LD15, LD16, LD17, LD18, LD19, LD2, LD20, LD21, LD22, LD23, LD24, LD25, LD26, LD27, LD28, LD29, LD3, LD30, LD31, LD32, LD33, LD34, LD35, LD36, LD37, LD38, LD39, LD4, LD40, LD41, LD42, LD43, LD44, LD45, LD46, LD47, LD48, LD49, LD5, LD50, LD51, LD52, LD53, LD54, LD55, LD56, LD57, LD58, LD59, LD6, LD60, LD61, LD62, LD63, LD64, LD65, LD66, LD67, LD68, LD69, LD7, LD70, LD71, LD72, LD73, LD74, LD75, LD76, LD77, LD78, LD79, LD8, LD80, LD81, LD82, LD83, LD84, LD85, LD86, LD87, LD88, LD89, LD9, LD90, LD91, LD92, LD93, LD94, LD95, LD96, LD97, LD98, LD99, LDE1: footprint EDI:WS2812B_2020 -> LED_SMD:LED_WS2812B_PLCC4_5.0x5.0mm_P3.2mm; symbol HL-Mk3-rescue:WS2812C-EDI-Audio-HL-Mk2-rescue -> LED:WS2812B
Connections:
- net +3V3: now also LD1.1 (VDD), LD10.1 (VDD), LD100.1 (VDD), LD101.1 (VDD), LD102.1 (VDD), LD103.1 (VDD), LD104.1 (VDD), LD105.1 (VDD), LD106.1 (VDD), LD107.1 (VDD), LD108.1 (VDD), LD109.1 (VDD), LD11.1 (VDD), LD110.1 (VDD), LD111.1 (VDD), LD112.1 (VDD), LD113.1 (VDD), LD114.1 (VDD), LD115.1 (VDD), LD116.1 (VDD), LD117.1 (VDD), LD118.1 (VDD), LD119.1 (VDD), LD12.1 (VDD), LD120.1 (VDD), LD121.1 (VDD), LD122.1 (VDD), LD123.1 (VDD), LD124.1 (VDD), LD125.1 (VDD), LD126.1 (VDD), LD127.1 (VDD), LD13.1 (VDD), LD14.1 (VDD), LD15.1 (VDD), LD16.1 (VDD), LD17.1 (VDD), LD18.1 (VDD), LD19.1 (VDD), LD2.1 (VDD), LD20.1 (VDD), LD21.1 (VDD), LD22.1 (VDD), LD23.1 (VDD), LD24.1 (VDD), LD25.1 (VDD), LD26.1 (VDD), LD27.1 (VDD), LD28.1 (VDD), LD29.1 (VDD), LD3.1 (VDD), LD30.1 (VDD), LD31.1 (VDD), LD32.1 (VDD), LD33.1 (VDD), LD34.1 (VDD), LD35.1 (VDD), LD36.1 (VDD), LD37.1 (VDD), LD38.1 (VDD), LD39.1 (VDD), LD4.1 (VDD), LD40.1 (VDD), LD41.1 (VDD), LD42.1 (VDD), LD43.1 (VDD), LD44.1 (VDD), LD45.1 (VDD), LD46.1 (VDD), LD47.1 (VDD), LD48.1 (VDD), LD49.1 (VDD), LD5.1 (VDD), LD50.1 (VDD), LD51.1 (VDD), LD52.1 (VDD), LD53.1 (VDD), LD54.1 (VDD), LD55.1 (VDD), LD56.1 (VDD), LD57.1 (VDD), LD58.1 (VDD), LD59.1 (VDD), LD6.1 (VDD), LD60.1 (VDD), LD61.1 (VDD), LD62.1 (VDD), LD63.1 (VDD), LD64.1 (VDD), LD65.1 (VDD), LD66.1 (VDD), LD67.1 (VDD), LD68.1 (VDD), LD69.1 (VDD), LD7.1 (VDD), LD70.1 (VDD), LD71.1 (VDD), LD72.1 (VDD), LD73.1 (VDD), LD74.1 (VDD), LD75.1 (VDD), LD76.1 (VDD), LD77.1 (VDD), LD78.1 (VDD), LD79.1 (VDD), LD8.1 (VDD), LD80.1 (VDD), LD81.1 (VDD), LD82.1 (VDD), LD83.1 (VDD), LD84.1 (VDD), LD85.1 (VDD), LD86.1 (VDD), LD87.1 (VDD), LD88.1 (VDD), LD89.1 (VDD), LD9.1 (VDD), LD90.1 (VDD), LD91.1 (VDD), LD92.1 (VDD), LD93.1 (VDD), LD94.1 (VDD), LD95.1 (VDD), LD96.1 (VDD), LD97.1 (VDD), LD98.1 (VDD), LD99.1 (VDD), LDE1.1 (VDD); no longer LD1.4 (VDD), LD10.4 (VDD), LD100.4 (VDD), LD101.4 (VDD), LD102.4 (VDD), LD103.4 (VDD), LD104.4 (VDD), LD105.4 (VDD), LD106.4 (VDD), LD107.4 (VDD), LD108.4 (VDD), LD109.4 (VDD), LD11.4 (VDD), LD110.4 (VDD), LD111.4 (VDD), LD112.4 (VDD), LD113.4 (VDD), LD114.4 (VDD), LD115.4 (VDD), LD116.4 (VDD), LD117.4 (VDD), LD118.4 (VDD), LD119.4 (VDD), LD12.4 (VDD), LD120.4 (VDD), LD121.4 (VDD), LD122.4 (VDD), LD123.4 (VDD), LD124.4 (VDD), LD125.4 (VDD), LD126.4 (VDD), LD127.4 (VDD), LD13.4 (VDD), LD14.4 (VDD), LD15.4 (VDD), LD16.4 (VDD), LD17.4 (VDD), LD18.4 (VDD), LD19.4 (VDD), LD2.4 (VDD), LD20.4 (VDD), LD21.4 (VDD), LD22.4 (VDD), LD23.4 (VDD), LD24.4 (VDD), LD25.4 (VDD), LD26.4 (VDD), LD27.4 (VDD), LD28.4 (VDD), LD29.4 (VDD), LD3.4 (VDD), LD30.4 (VDD), LD31.4 (VDD), LD32.4 (VDD), LD33.4 (VDD), LD34.4 (VDD), LD35.4 (VDD), LD36.4 (VDD), LD37.4 (VDD), LD38.4 (VDD), LD39.4 (VDD), LD4.4 (VDD), LD40.4 (VDD), LD41.4 (VDD), LD42.4 (VDD), LD43.4 (VDD), LD44.4 (VDD), LD45.4 (VDD), LD46.4 (VDD), LD47.4 (VDD), LD48.4 (VDD), LD49.4 (VDD), LD5.4 (VDD), LD50.4 (VDD), LD51.4 (VDD), LD52.4 (VDD), LD53.4 (VDD), LD54.4 (VDD), LD55.4 (VDD), LD56.4 (VDD), LD57.4 (VDD), LD58.4 (VDD), LD59.4 (VDD), LD6.4 (VDD), LD60.4 (VDD), LD61.4 (VDD), LD62.4 (VDD), LD63.4 (VDD), LD64.4 (VDD), LD65.4 (VDD), LD66.4 (VDD), LD67.4 (VDD), LD68.4 (VDD), LD69.4 (VDD), LD7.4 (VDD), LD70.4 (VDD), LD71.4 (VDD), LD72.4 (VDD), LD73.4 (VDD), LD74.4 (VDD), LD75.4 (VDD), LD76.4 (VDD), LD77.4 (VDD), LD78.4 (VDD), LD79.4 (VDD), LD8.4 (VDD), LD80.4 (VDD), LD81.4 (VDD), LD82.4 (VDD), LD83.4 (VDD), LD84.4 (VDD), LD85.4 (VDD), LD86.4 (VDD), LD87.4 (VDD), LD88.4 (VDD), LD89.4 (VDD), LD9.4 (VDD), LD90.4 (VDD), LD91.4 (VDD), LD92.4 (VDD), LD93.4 (VDD), LD94.4 (VDD), LD95.4 (VDD), LD96.4 (VDD), LD97.4 (VDD), LD98.4 (VDD), LD99.4 (VDD), LDE1.4 (VDD)
- net GND: now also LD1.3 (VSS), LD10.3 (VSS), LD100.3 (VSS), LD101.3 (VSS), LD102.3 (VSS), LD103.3 (VSS), LD104.3 (VSS), LD105.3 (VSS), LD106.3 (VSS), LD107.3 (VSS), LD108.3 (VSS), LD109.3 (VSS), LD11.3 (VSS), LD110.3 (VSS), LD111.3 (VSS), LD112.3 (VSS), LD113.3 (VSS), LD114.3 (VSS), LD115.3 (VSS), LD116.3 (VSS), LD117.3 (VSS), LD118.3 (VSS), LD119.3 (VSS), LD12.3 (VSS), LD120.3 (VSS), LD121.3 (VSS), LD122.3 (VSS), LD123.3 (VSS), LD124.3 (VSS), LD125.3 (VSS), LD126.3 (VSS), LD127.3 (VSS), LD13.3 (VSS), LD14.3 (VSS), LD15.3 (VSS), LD16.3 (VSS), LD17.3 (VSS), LD18.3 (VSS), LD19.3 (VSS), LD2.3 (VSS), LD20.3 (VSS), LD21.3 (VSS), LD22.3 (VSS), LD23.3 (VSS), LD24.3 (VSS), LD25.3 (VSS), LD26.3 (VSS), LD27.3 (VSS), LD28.3 (VSS), LD29.3 (VSS), LD3.3 (VSS), LD30.3 (VSS), LD31.3 (VSS), LD32.3 (VSS), LD33.3 (VSS), LD34.3 (VSS), LD35.3 (VSS), LD36.3 (VSS), LD37.3 (VSS), LD38.3 (VSS), LD39.3 (VSS), LD4.3 (VSS), LD40.3 (VSS), LD41.3 (VSS), LD42.3 (VSS), LD43.3 (VSS), LD44.3 (VSS), LD45.3 (VSS), LD46.3 (VSS), LD47.3 (VSS), LD48.3 (VSS), LD49.3 (VSS), LD5.3 (VSS), LD50.3 (VSS), LD51.3 (VSS), LD52.3 (VSS), LD53.3 (VSS), LD54.3 (VSS), LD55.3 (VSS), LD56.3 (VSS), LD57.3 (VSS), LD58.3 (VSS), LD59.3 (VSS), LD6.3 (VSS), LD60.3 (VSS), LD61.3 (VSS), LD62.3 (VSS), LD63.3 (VSS), LD64.3 (VSS), LD65.3 (VSS), LD66.3 (VSS), LD67.3 (VSS), LD68.3 (VSS), LD69.3 (VSS), LD7.3 (VSS), LD70.3 (VSS), LD71.3 (VSS), LD72.3 (VSS), LD73.3 (VSS), LD74.3 (VSS), LD75.3 (VSS), LD76.3 (VSS), LD77.3 (VSS), LD78.3 (VSS), LD79.3 (VSS), LD8.3 (VSS), LD80.3 (VSS), LD81.3 (VSS), LD82.3 (VSS), LD83.3 (VSS), LD84.3 (VSS), LD85.3 (VSS), LD86.3 (VSS), LD87.3 (VSS), LD88.3 (VSS), LD89.3 (VSS), LD9.3 (VSS), LD90.3 (VSS), LD91.3 (VSS), LD92.3 (VSS), LD93.3 (VSS), LD94.3 (VSS), LD95.3 (VSS), LD96.3 (VSS), LD97.3 (VSS), LD98.3 (VSS), LD99.3 (VSS), LDE1.3 (VSS); no longer LD1.2 (GND), LD10.2 (GND), LD100.2 (GND), LD101.2 (GND), LD102.2 (GND), LD103.2 (GND), LD104.2 (GND), LD105.2 (GND), LD106.2 (GND), LD107.2 (GND), LD108.2 (GND), LD109.2 (GND), LD11.2 (GND), LD110.2 (GND), LD111.2 (GND), LD112.2 (GND), LD113.2 (GND), LD114.2 (GND), LD115.2 (GND), LD116.2 (GND), LD117.2 (GND), LD118.2 (GND), LD119.2 (GND), LD12.2 (GND), LD120.2 (GND), LD121.2 (GND), LD122.2 (GND), LD123.2 (GND), LD124.2 (GND), LD125.2 (GND), LD126.2 (GND), LD127.2 (GND), LD13.2 (GND), LD14.2 (GND), LD15.2 (GND), LD16.2 (GND), LD17.2 (GND), LD18.2 (GND), LD19.2 (GND), LD2.2 (GND), LD20.2 (GND), LD21.2 (GND), LD22.2 (GND), LD23.2 (GND), LD24.2 (GND), LD25.2 (GND), LD26.2 (GND), LD27.2 (GND), LD28.2 (GND), LD29.2 (GND), LD3.2 (GND), LD30.2 (GND), LD31.2 (GND), LD32.2 (GND), LD33.2 (GND), LD34.2 (GND), LD35.2 (GND), LD36.2 (GND), LD37.2 (GND), LD38.2 (GND), LD39.2 (GND), LD4.2 (GND), LD40.2 (GND), LD41.2 (GND), LD42.2 (GND), LD43.2 (GND), LD44.2 (GND), LD45.2 (GND), LD46.2 (GND), LD47.2 (GND), LD48.2 (GND), LD49.2 (GND), LD5.2 (GND), LD50.2 (GND), LD51.2 (GND), LD52.2 (GND), LD53.2 (GND), LD54.2 (GND), LD55.2 (GND), LD56.2 (GND), LD57.2 (GND), LD58.2 (GND), LD59.2 (GND), LD6.2 (GND), LD60.2 (GND), LD61.2 (GND), LD62.2 (GND), LD63.2 (GND), LD64.2 (GND), LD65.2 (GND), LD66.2 (GND), LD67.2 (GND), LD68.2 (GND), LD69.2 (GND), LD7.2 (GND), LD70.2 (GND), LD71.2 (GND), LD72.2 (GND), LD73.2 (GND), LD74.2 (GND), LD75.2 (GND), LD76.2 (GND), LD77.2 (GND), LD78.2 (GND), LD79.2 (GND), LD8.2 (GND), LD80.2 (GND), LD81.2 (GND), LD82.2 (GND), LD83.2 (GND), LD84.2 (GND), LD85.2 (GND), LD86.2 (GND), LD87.2 (GND), LD88.2 (GND), LD89.2 (GND), LD9.2 (GND), LD90.2 (GND), LD91.2 (GND), LD92.2 (GND), LD93.2 (GND), LD94.2 (GND), LD95.2 (GND), LD96.2 (GND), LD97.2 (GND), LD98.2 (GND), LD99.2 (GND), LDE1.2 (GND)
- net LED: now also LD1.4 (DIN); no longer LD1.3 (DIN)
- new net: LD47.2 (DOUT), LD48.4 (DIN)
- new net: LD46.2 (DOUT), LD47.4 (DIN)
- new net: LD45.2 (DOUT), LD46.4 (DIN)
- new net: LD74.2 (DOUT), LD75.4 (DIN)
- new net: LD51.2 (DOUT), LD74.4 (DIN)
- new net: LD21.4 (DIN), LD22.2 (DOUT)
- new net: LD22.4 (DIN), LD23.2 (DOUT)
- new net: LD49.2 (DOUT), LD50.4 (DIN)
- new net: LD48.2 (DOUT), LD49.4 (DIN)
- new net: LD98.4 (DIN), LD99.2 (DOUT)
- new net: LD100.2 (DOUT), LD99.4 (DIN)
- new net: LD76.2 (DOUT), LD77.4 (DIN)
- new net: LD75.2 (DOUT), LD76.4 (DIN)
- new net: LD126.2 (DOUT), LD127.4 (DIN)
- new net: LD102.4 (DIN), LD103.2 (DOUT)
- new net: LD103.4 (DIN), LD104.2 (DOUT)
- new net: LD58.4 (DIN), LD59.2 (DOUT)
- new net: LD59.4 (DIN), LD60.2 (DOUT)
- new net: LD62.4 (DIN), LD63.2 (DOUT)
- new net: LD63.4 (DIN), LD64.2 (DOUT)
- new net: LD101.4 (DIN), LD102.2 (DOUT)
- new net: LD100.4 (DIN), LD101.2 (DOUT)
- new net: LD85.2 (DOUT), LD86.4 (DIN)
- new net: LD84.2 (DOUT), LD85.4 (DIN)
- new net: LD108.4 (DIN), LD109.2 (DOUT)
- new net: LD109.4 (DIN), LD110.2 (DOUT)
- new net: LD53.4 (DIN), LD54.2 (DOUT)
- new net: LD54.4 (DIN), LD55.2 (DOUT)
- new net: LD61.4 (DIN), LD62.2 (DOUT)
- new net: LD13.2 (DOUT), LD28.4 (DIN)
- new net: LD13.4 (DIN), LD14.2 (DOUT)
- new net: LD14.4 (DIN), LD15.2 (DOUT)
- new net: LD15.4 (DIN), LD16.2 (DOUT)
- new net: LD16.4 (DIN), LD17.2 (DOUT)
- new net: LD97.4 (DIN), LD98.2 (DOUT)
- new net: LD55.4 (DIN), LD56.2 (DOUT)
- new net: LD56.4 (DIN), LD57.2 (DOUT)
- new net: LD116.2 (DOUT), LD117.4 (DIN)
- new net: LD115.2 (DOUT), LD116.4 (DIN)
- new net: LD17.4 (DIN), LD18.2 (DOUT)
- new net: LD18.4 (DIN), LD19.2 (DOUT)
- new net: LD111.2 (DOUT), LD112.4 (DIN)
- new net: LD111.4 (DIN), LD93.2 (DOUT)
- new net: LD105.4 (DIN), LD106.2 (DOUT)
- new net: LD106.4 (DIN), LD107.2 (DOUT)
- new net: LD2.2 (DOUT), LD3.4 (DIN)
- new net: LD1.2 (DOUT), LD2.4 (DIN)
- new net: LD11.2 (DOUT), LD12.4 (DIN)
- new net: LD10.2 (DOUT), LD11.4 (DIN)
- new net: LD104.4 (DIN), LD105.2 (DOUT)
- new net: LD122.2 (DOUT), LD123.4 (DIN)
- new net: LD121.2 (DOUT), LD122.4 (DIN)
- new net: LD68.4 (DIN), LD69.2 (DOUT)
- new net: LD69.4 (DIN), LD70.2 (DOUT)
- new net: LD3.2 (DOUT), LD4.4 (DIN)
- new net: LD37.2 (DOUT), LD38.4 (DIN)
- new net: LD36.2 (DOUT), LD37.4 (DIN)
- new net: LD23.4 (DIN), LD24.2 (DOUT)
- new net: LD24.4 (DIN), LD25.2 (DOUT)
- new net: LD112.2 (DOUT), LD113.4 (DIN)
- new net: LD4.2 (DOUT), LD5.4 (DIN)
- new net: LD79.2 (DOUT), LD80.4 (DIN)
- new net: LD78.2 (DOUT), LD79.4 (DIN)
- new net: LD89.2 (DOUT), LD90.4 (DIN)
- new net: LD88.2 (DOUT), LD89.4 (DIN)
- new net: LD38.2 (DOUT), LD39.4 (DIN)
- new net: LD107.4 (DIN), LD108.2 (DOUT)
- new net: LD42.2 (DOUT), LD43.4 (DIN)
- new net: LD41.2 (DOUT), LD42.4 (DIN)
- new net: LD40.2 (DOUT), LD41.4 (DIN)
- new net: LD39.2 (DOUT), LD40.4 (DIN)
- new net: LD91.2 (DOUT), LD92.4 (DIN)
- new net: LD90.2 (DOUT), LD91.4 (DIN)
- new net: LD25.4 (DIN), LD26.2 (DOUT)
- new net: LD35.2 (DOUT), LD36.4 (DIN)
- new net: LD34.2 (DOUT), LD35.4 (DIN)
- new net: LD51.4 (DIN), LD52.2 (DOUT)
- new net: LD123.2 (DOUT), LD124.4 (DIN)
- new net: LD10.4 (DIN), LD9.2 (DOUT)
- new net: LD8.2 (DOUT), LD9.4 (DIN)
- new net: LD87.2 (DOUT), LD88.4 (DIN)
- new net: LD93.4 (DIN), LD94.2 (DOUT)
- new net: LD94.4 (DIN), LD95.2 (DOUT)
- new net: LD19.4 (DIN), LD20.2 (DOUT)
- new net: LD29.2 (DOUT), LD30.4 (DIN)
- new net: LD28.2 (DOUT), LD29.4 (DIN)
- new net: LD110.4 (DIN), LD92.2 (DOUT)
- new net: LD30.2 (DOUT), LD31.4 (DIN)
- new net: LD118.2 (DOUT), LD119.4 (DIN)
- new net: LD117.2 (DOUT), LD118.4 (DIN)
- new net: LD65.4 (DIN), LD66.2 (DOUT)
- new net: LD66.4 (DIN), LD67.2 (DOUT)
- new net: LD83.2 (DOUT), LD84.4 (DIN)
- new net: LD96.4 (DIN), LD97.2 (DOUT)
- new net: LD50.2 (DOUT), LD73.4 (DIN)
- new net: LD33.2 (DOUT), LD34.4 (DIN)
- new net: LD43.2 (DOUT), LD44.4 (DIN)
- new net: LD71.4 (DIN), LD72.2 (DOUT)
- new net: LD72.4 (DIN), LD73.2 (DOUT)
- new net: LD44.2 (DOUT), LD45.4 (DIN)
- new net: LD6.2 (DOUT), LD7.4 (DIN)
- new net: LD5.2 (DOUT), LD6.4 (DIN)
- new net: LD7.2 (DOUT), LD8.4 (DIN)
- new net: LD114.2 (DOUT), LD115.4 (DIN)
- new net: LD113.2 (DOUT), LD114.4 (DIN)
- new net: LD82.2 (DOUT), LD83.4 (DIN)
- new net: LD81.2 (DOUT), LD82.4 (DIN)
- new net: LD80.2 (DOUT), LD81.4 (DIN)
- new net: LD64.4 (DIN), LD65.2 (DOUT)
- new net: LD125.2 (DOUT), LD126.4 (DIN)
- new net: LD124.2 (DOUT), LD125.4 (DIN)
- new net: LD70.4 (DIN), LD71.2 (DOUT)
- new net: LD119.2 (DOUT), LD120.4 (DIN)
- new net: LD57.4 (DIN), LD58.2 (DOUT)
- new net: LD52.4 (DIN), LD53.2 (DOUT)
- new net: LD20.4 (DIN), LD21.2 (DOUT)
- new net: LD67.4 (DIN), LD68.2 (DOUT)
- new net: LD31.2 (DOUT), LD32.4 (DIN)
- new net: LD120.2 (DOUT), LD121.4 (DIN)
- new net: LD86.2 (DOUT), LD87.4 (DIN)
- new net: LD32.2 (DOUT), LD33.4 (DIN)
- new net: LD26.4 (DIN), LD27.2 (DOUT)
- new net: LD27.4 (DIN), LDE1.2 (DOUT)
- new net: LD77.2 (DOUT), LD78.4 (DIN)
- new net: LD12.2 (DOUT), LDE1.4 (DIN)
- new net: LD60.4 (DIN), LD61.2 (DOUT)
- new net: LD95.4 (DIN), LD96.2 (DOUT)

Commit message: Yep, moved some stuff to archives.
Parts:
- H1, H2, H3, H4, H5, H6, H7, H8: footprint EDI:SolderableHole-M2 -> MountingHole:MountingHole_3.2mm_M3; symbol Mechanical:MountingHole_Pad -> Mechanical:MountingHole
- LD1, LD10, LD100, LD101, LD102, LD103, LD104, LD105, LD106, LD107, LD108, LD109, LD11, LD110, LD111, LD112, LD113, LD114, LD115, LD116, LD117, LD118, LD119, LD12, LD120, LD121, LD122, LD123, LD124, LD125, LD126, LD127, LD13, LD14, LD15, LD16, LD17, LD18, LD19, LD2, LD20, LD21, LD22, LD23, LD24, LD25, LD26, LD27, LD28, LD29, LD3, LD30, LD31, LD32, LD33, LD34, LD35, LD36, LD37, LD38, LD39, LD4, LD40, LD41, LD42, LD43, LD44, LD45, LD46, LD47, LD48, LD49, LD5, LD50, LD51, LD52, LD53, LD54, LD55, LD56, LD57, LD58, LD59, LD6, LD60, LD61, LD62, LD63, LD64, LD65, LD66, LD67, LD68, LD69, LD7, LD70, LD71, LD72, LD73, LD74, LD75, LD76, LD77, LD78, LD79, LD8, LD80, LD81, LD82, LD83, LD84, LD85, LD86, LD87, LD88, LD89, LD9, LD90, LD91, LD92, LD93, LD94, LD95, LD96, LD97, LD98, LD99, LDE1: value WS2812C-2020 -> WS2812C
Connections:
- net GND: no longer H1.1, H2.1, H3.1, H4.1, H5.1, H6.1, H7.1, H8.1
- net row0: no longer J2.3 (Pin_3), J2.7 (Pin_7), T2.1, T4.1
- net col12 renamed col6
- net col6: now also J2.2 (Pin_2), J2.4 (Pin_4), T2.2; no longer J2.8 (Pin_8)
- net col13 renamed col7
- net col7: now also J2.8 (Pin_8), T3.2, T4.2; no longer T2.2
- removed net col14: J2.4 (Pin_4), T3.2
- removed net col15: J2.2 (Pin_2), T4.2
- new net row1: J2.3 (Pin_3), J2.7 (Pin_7), T2.1, T4.1

Commit message: So much stuff
Wow it's been a while.
Parts:
- LD1, LD10, LD100, LD101, LD102, LD103, LD104, LD105, LD106, LD107, LD108, LD109, LD11, LD110, LD111, LD112, LD113, LD114, LD115, LD116, LD117, LD118, LD119, LD12, LD120, LD121, LD122, LD123, LD124, LD125, LD126, LD127, LD13, LD14, LD15, LD16, LD17, LD18, LD19, LD2, LD20, LD21, LD22, LD23, LD24, LD25, LD26, LD27, LD28, LD29, LD3, LD30, LD31, LD32, LD33, LD34, LD35, LD36, LD37, LD38, LD39, LD4, LD40, LD41, LD42, LD43, LD44, LD45, LD46, LD47, LD48, LD49, LD5, LD50, LD51, LD52, LD53, LD54, LD55, LD56, LD57, LD58, LD59, LD6, LD60, LD61, LD62, LD63, LD64, LD65, LD66, LD67, LD68, LD69, LD7, LD70, LD71, LD72, LD73, LD74, LD75, LD76, LD77, LD78, LD79, LD8, LD80, LD81, LD82, LD83, LD84, LD85, LD86, LD87, LD88, LD89, LD9, LD90, LD91, LD92, LD93, LD94, LD95, LD96, LD97, LD98, LD99, LDE1: footprint LED_SMD:LED_WS2812B_PLCC4_5.0x5.0mm_P3.2mm -> EDI:LED_WS2812C_PLCC4_5.0x5.0mm_P3.2mm
