File: Current/HardLight2040/HL-2040.kicad_sch (KiCad schematic)
At the start: 41 parts, among them J0 USB, U0 RP2040, U1 LDO-3.3, U2 USBLC6-2SC6, U3 W25Q128JVS, Y0 12MHz

Commit message: Whole bunch of work!
Parts:
- renumbered R2 to RC1, R3 to RC2, R5 to RD0, R4 to RD1, R1 to RF1, R6 to RR1, R7 to RX1
Connections:
- no-connect marks 2 -> 4
Other:
- moved on the sheet: F0, H1, H2, H3, H4, H5, H6, J0, RC1, RC2, U2
