File: Current/HardLightMicro/HardLightMicro.kicad_pcb (KiCad board)
At the start: 2 copper layers, 85 x 40 mm, 172 parts, among them J1 USB, K1 Keyswitch, K10 Keyswitch, K11 Keyswitch, K12 Keyswitch, K13 Keyswitch, K14 Keyswitch, K15 Keyswitch, K16 Keyswitch, K17 Keyswitch, K18 Keyswitch, K19 Keyswitch, K2 Keyswitch, K20 Keyswitch, K21 Keyswitch, K22 Keyswitch, K23 Keyswitch, K24 Keyswitch, K25 Keyswitch, K26 Keyswitch, K27 Keyswitch, K28 Keyswitch, K29 Keyswitch, K3 Keyswitch, K30 Keyswitch, K31 Keyswitch, K32 Keyswitch, K33 Keyswitch, K34 Keyswitch, K35 Keyswitch, K36 Keyswitch, K37 Keyswitch, K38 Keyswitch, K39 Keyswitch, K4 Keyswitch, K40 Keyswitch, K41 Keyswitch, K42 Keyswitch, K43 Keyswitch, K44 Keyswitch, K45 Keyswitch, K46 Keyswitch, K47 Keyswitch, K48 Keyswitch, K49 Keyswitch, K5 Keyswitch, K50 Keyswitch, K51 Keyswitch, K52 Keyswitch, K53 Keyswitch, K54 Keyswitch, K55 Keyswitch, K56 Keyswitch, K57 Keyswitch, K58 Keyswitch, K59 Keyswitch, K6 Keyswitch, K60 Keyswitch, K61 Keyswitch, K62 Keyswitch, K63 Keyswitch, K64 Keyswitch, K7 Keyswitch, K8 Keyswitch, K9 Keyswitch, U1 STM32F411CEU6, U2 LDO-3.3, Y1 8MHz

Commit message: oh my god just stop
Parts:
- moved C1 56.6 mm to (181.6, 68.3)
- moved C6 49.2 mm to (169.9, 68.7)
- moved C5 46.5 mm to (167.6, 75.7)
- moved R2 43.3 mm to (176.9, 68.3)
- moved C3 43.2 mm to (169.5, 74.7)
- moved C4 43.2 mm to (159.8, 74.4), turned to -90 degrees
- moved CV1 33.9 mm to (161.9, 66.3), turned to 180 degrees
- moved C2 23.8 mm to (159.3, 67.4), turned to 180 degrees
Changed lines of the file:
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@@
   )
   (footprint "EDI:Passive_0402_1005Metric" (layer "F.Cu")
-    (at 130.045998 57.134128)
+    (at 169.545 74.676)
     (descr "Capacitor SMD 0402 (1005 Metric), square (rectangular) end terminal, IPC_7351 nominal, (Body size source: http://www.tortai-tech.com/upload/download/2011102023233369053.pdf), generated with kicad-footprint-generator")
     (tags "capacitor")
@@
       (effects (font (size 1 1) (thickness 0.15)))
     )
-    (fp_text user "${REFERENCE}" (at 0 -0.7937) (layer "F.SilkS")
+    (fp_text user "${REFERENCE}" (at 1.27 0) (layer "F.SilkS")
       (effects (font (size 0.25 0.25) (thickness 0.04)))
     )
@@
   )
   (footprint "EDI:Passive_0402_1005Metric" (layer "F.Cu")
-    (at 128.2645 62.604064)
+    (at 161.925 66.294 180)
     (descr "Capacitor SMD 0402 (1005 Metric), square (rectangular) end terminal, IPC_7351 nominal, (Body size source: http://www.tortai-tech.com/upload/download/2011102023233369053.pdf), generated with kicad-footprint-generator")
     (tags "capacitor")
@@
     (fp_line (start 0.5 -0.25) (end 0.5 0.25) (layer "F.Fab") (width 0.1))
     (fp_line (start -0.5 0.25) (end -0.5 -0.25) (layer "F.Fab") (width 0.1))
-    (pad "1" smd roundrect (at -0.485 0) (size 0.59 0.64) (layers "F.Cu" "F.Paste" "F.Mask") (roundrect_rratio 0.25)
+    (pad "1" smd roundrect (at -0.485 0 180) (size 0.59 0.64) (layers "F.Cu" "F.Paste" "F.Mask") (roundrect_rratio 0.25)
       (net 7 "Net-(CV1-Pad1)") (pintype "passive"))
-    (pad "2" smd roundrect (at 0.485 0) (size 0.59 0.64) (layers "F.Cu" "F.Paste" "F.Mask") (roundrect_rratio 0.25)
+    (pad "2" smd roundrect (at 0.485 0 180) (size 0.59 0.64) (layers "F.Cu" "F.Paste" "F.Mask") (roundrect_rratio 0.25)
       (net 2 "GND") (pintype "passive"))
     (model "${KISYS3DMOD}/Capacitor_SMD.3dshapes/C_0402_1005Metric.wrl"
@@
     (property "Sheetname" "")
     (attr smd)
-    (fp_text reference "Y1" (at 0 3) (layer "F.SilkS")
+    (fp_text reference "Y1" (at -1.525 2.950251) (layer "F.SilkS")
       (effects (font (size 1 1) (thickness 0.15)))
     )
@@
       (effects (font (size 1 1) (thickness 0.15)))
     )
-    (fp_text user "${REFERENCE}" (at -1.5 0) (layer "F.SilkS")
+    (fp_text user "${REFERENCE}" (at -1.16 0) (layer "F.SilkS")
       (effects (font (size 0.25 0.25) (thickness 0.04)))
     )
@@
   )
   (footprint "EDI:Passive_0402_1005Metric" (layer "F.Cu")
-    (at 124.0445 59.624065)
+    (at 167.64 75.692)
     (descr "Capacitor SMD 0402 (1005 Metric), square (rectangular) end terminal, IPC_7351 nominal, (Body size source: http://www.tortai-tech.com/upload/download/2011102023233369053.pdf), generated with kicad-footprint-generator")
     (tags "capacitor")
@@
   )
   (footprint "EDI:Passive_0402_1005Metric" (layer "F.Cu")
-    (at 121.115998 62.554129)
+    (at 169.926 68.707)
     (descr "Capacitor SMD 0402 (1005 Metric), square (rectangular) end terminal, IPC_7351 nominal, (Body size source: http://www.tortai-tech.com/upload/download/2011102023233369053.pdf), generated with kicad-footprint-generator")
     (tags "capacitor")
@@
   )
   (footprint "EDI:Passive_0402_1005Metric" (layer "F.Cu")
-    (at 138.303 56.134)
+    (at 159.258 67.437 180)
     (descr "Capacitor SMD 0402 (1005 Metric), square (rectangular) end terminal, IPC_7351 nominal, (Body size source: http://www.tortai-tech.com/upload/download/2011102023233369053.pdf), generated with kicad-footprint-generator")
     (tags "capacitor")
@@
     (fp_line (start 0.5 -0.25) (end 0.5 0.25) (layer "F.Fab") (width 0.1))
     (fp_line (start 0.5 0.25) (end -0.5 0.25) (layer "F.Fab") (width 0.1))
-    (pad "1" smd roundrect (at -0.485 0) (size 0.59 0.64) (layers "F.Cu" "F.Paste" "F.Mask") (roundrect_rratio 0.25)
+    (pad "1" smd roundrect (at -0.485 0 180) (size 0.59 0.64) (layers "F.Cu" "F.Paste" "F.Mask") (roundrect_rratio 0.25)
       (net 3 "+3V3") (pintype "passive"))
-    (pad "2" smd roundrect (at 0.485 0) (size 0.59 0.64) (layers "F.Cu" "F.Paste" "F.Mask") (roundrect_rratio 0.25)
+    (pad "2" smd roundrect (at 0.485 0 180) (size 0.59 0.64) (layers "F.Cu" "F.Paste" "F.Mask") (roundrect_rratio 0.25)
       (net 2 "GND") (pintype "passive"))
     (model "${KISYS3DMOD}/Capacitor_SMD.3dshapes/C_0402_1005Metric.wrl"
@@
   )
   (footprint "EDI:Passive_0402_1005Metric" (layer "F.Cu")
-    (at 126.105996 57.284129)
+    (at 181.61 68.326)
     (descr "Capacitor SMD 0402 (1005 Metric), square (rectangular) end terminal, IPC_7351 nominal, (Body size source: http://www.tortai-tech.com/upload/download/2011102023233369053.pdf), generated with kicad-footprint-generator")
     (tags "capacitor")
@@
   )
   (footprint "EDI:Passive_0402_1005Metric" (layer "F.Cu")
-    (at 118.206 62.70413)
+    (at 159.766 74.422 -90)
     (descr "Capacitor SMD 0402 (1005 Metric), square (rectangular) end terminal, IPC_7351 nominal, (Body size source: http://www.tortai-tech.com/upload/download/2011102023233369053.pdf), generated with kicad-footprint-generator")
     (tags "capacitor")
@@
     (property "Sheetname" "")
     (attr smd)
-    (fp_text reference "C4" (at 0 -1.17) (layer "F.SilkS") hide
+    (fp_text reference "C4" (at 0 -1.17 90) (layer "F.SilkS") hide
       (effects (font (size 1.25 1.25) (thickness 0.15)))
     )
-    (fp_text value "100nF" (at 0 1.17) (layer "F.Fab")
+    (fp_text value "100nF" (at 0 1.17 90) (layer "F.Fab")
       (effects (font (size 1 1) (thickness 0.15)))
     )
-    (fp_text user "${REFERENCE}" (at 0 -0.7937) (layer "F.SilkS")
+    (fp_text user "${REFERENCE}" (at 0 -0.7937 90) (layer "F.SilkS")
       (effects (font (size 0.25 0.25) (thickness 0.04)))
     )
@@
     (fp_line (start 0.5 0.25) (end -0.5 0.25) (layer "F.Fab") (width 0.1))
     (fp_line (start -0.5 -0.25) (end 0.5 -0.25) (layer "F.Fab") (width 0.1))
-    (pad "1" smd roundrect (at -0.485 0) (size 0.59 0.64) (layers "F.Cu" "F.Paste" "F.Mask") (roundrect_rratio 0.25)
+    (pad "1" smd roundrect (at -0.485 0 270) (size 0.59 0.64) (layers "F.Cu" "F.Paste" "F.Mask") (roundrect_rratio 0.25)
       (net 3 "+3V3") (pintype "passive"))
-    (pad "2" smd roundrect (at 0.485 0) (size 0.59 0.64) (layers "F.Cu" "F.Paste" "F.Mask") (roundrect_rratio 0.25)
+    (pad "2" smd roundrect (at 0.485 0 270) (size 0.59 0.64) (layers "F.Cu" "F.Paste" "F.Mask") (roundrect_rratio 0.25)
       (net 2 "GND") (pintype "passive"))
     (model "${KISYS3DMOD}/Capacitor_SMD.3dshapes/C_0402_1005Metric.wrl"
@@
   )
   (footprint "EDI:Passive_0402_1005Metric" (layer "F.Cu")
-    (at 134.753 58.584)
+    (at 176.911 68.326)
     (descr "Capacitor SMD 0402 (1005 Metric), square (rectangular) end terminal, IPC_7351 nominal, (Body size source: http://www.tortai-tech.com/upload/download/2011102023233369053.pdf), generated with kicad-footprint-generator")
     (tags "capacitor")
@@
     (property "Sheetname" "")
     (attr smd)
-    (fp_text reference "U1" (at -5 -4) (layer "F.SilkS")
+    (fp_text reference "U1" (at -5.24325 -5.2) (layer "F.SilkS")
       (effects (font (size 1 1) (thickness 0.15)))
     )

Commit message: Whole bunch of work!
Parts:
- removed CL1, CL2: 0.012nF, EDI:Passive_0402_1005Metric
- removed CV1: 4.7uF, EDI:Passive_0402_1005Metric
- removed RB1: 100K, EDI:Passive_0402_1005Metric
- removed RB2: 100k, EDI:Passive_0402_1005Metric
- added C10: 1uf, EDI:Passive_0402_1005Metric, F.Cu at (104.0, 48.8)
- added C11: 10uf, EDI:Passive_0402_1005Metric, F.Cu at (109.2, 42.0)
- added C9: 100nF, EDI:Passive_0402_1005Metric, F.Cu at (104.0, 50.8)
- added CF1: 100nF, EDI:Passive_0402_1005Metric, F.Cu at (106.3, 44.0)
- added CP1: 100nF, EDI:Passive_0402_1005Metric, F.Cu at (101.1, 48.8)
- added CP2: 10uF, EDI:Passive_0402_1005Metric, F.Cu at (112.1, 42.0)
- added CX1: 100nF, EDI:Passive_0402_1005Metric, F.Cu at (109.2, 46.0)
- added CX2: 100nF, EDI:Passive_0402_1005Metric, F.Cu at (106.9, 48.0)
- added R5: 1k, EDI:Passive_0402_1005Metric, F.Cu at (106.3, 46.0)
- added RU1: 5k1, EDI:Passive_0402_1005Metric, F.Cu at (106.3, 42.0)
- added RU2: 5k1, EDI:Passive_0402_1005Metric, F.Cu at (109.2, 44.0)
- added RX1: 1k, EDI:Passive_0402_1005Metric, F.Cu at (101.1, 50.8)
- added U3: W25Q128JVS, Package_SO:SOIC-8_5.23x5.23mm_P1.27mm, F.Cu at (99.6, 44.4)
- added U4: USBLC6-2SC6, Package_TO_SOT_SMD:SOT-23-6, F.Cu at (97.0, 50.0)
- C2: value 100nF -> 1uf
- C6: value 4.7uF -> 100nF
- C8: value 10uF -> 100nF
- F1: footprint Fuse:Fuse_0603_1608Metric_Pad1.05x0.95mm_HandSolder -> Fuse:Fuse_0603_1608Metric
- R2: value 10k -> 1k
- R3, R4: value 5k1 -> 27
- S1: value RESET -> USB BOOT
- S2: value LDR -> RESET
- U1: value STM32F411CEU6 -> RP2040; footprint Package_DFN_QFN:QFN-48-1EP_7x7mm_P0.5mm_EP5.6x5.6mm -> Package_DFN_QFN:QFN-56-1EP_7x7mm_P0.4mm_EP5.6x5.6mm_ThermalVias
- Y1: value 8MHz -> 12MHz
Connections:
- C1 pad 1: NRST -> +1V1
- C2 pad 1: +3V3 -> +1V1
- C7 pad 1: GND -> +3V3
- C7 pad 2: VBUS -> GND
- C8 pad 1: GND -> +3V3
- C8 pad 2: +3V3 -> GND
- LD1 pad 3: LED -> 26/A0
- R1 pad 1: LED -> 26/A0
- R2 pad 1: BOOT0 -> CS
- R2 pad 2: GND -> Net-(R2-Pad2)
- R3 pad 1: GND -> DB+
- R3 pad 2: Net-(J1-PadB5) -> Net-(R3-Pad2)
- R4 pad 1: Net-(J1-PadA5) -> DB-
- R4 pad 2: GND -> Net-(R4-Pad2)
- S1 pad 1: NRST -> GND
- S1 pad 2: GND -> Net-(R2-Pad2)
- S2 pad 1: BOOT0 -> ~{RESET}
- S2 pad 2: +3V3 -> GND
- U1 pad 10: unconnected-(U1-Pad10) -> +3V3
- U1 pad 11: row3 -> col7
- U1 pad 12: row2 -> col6
- U1 pad 13: row0 -> col5
- U1 pad 14: row1 -> col4
- U1 pad 15: LED -> col3
- U1 pad 16: colB -> 13
- U1 pad 17: colC -> 14
- U1 pad 18: colD -> 15
- U1 pad 19: colE -> GND
- U1 pad 2: unconnected-(U1-Pad2) -> colF
- U1 pad 20: Net-(RB2-Pad1) -> XTAL-
- U1 pad 21: col0 -> XTAL+
- U1 pad 22: Net-(CV1-Pad1) -> +3V3
- U1 pad 23: GND -> +1V1
- U1 pad 24: +3V3 -> unconnected-(U1-Pad24)
- U1 pad 25: colF -> unconnected-(U1-Pad25)
- U1 pad 26: col1 -> ~{RESET}
- U1 pad 27: unconnected-(U1-Pad27) -> 16
- U1 pad 28: unconnected-(U1-Pad28) -> 17
- U1 pad 29: unconnected-(U1-Pad29) -> 18
- U1 pad 3: unconnected-(U1-Pad3) -> colE
- U1 pad 30: unconnected-(U1-Pad30) -> col2
- U1 pad 31: Net-(RB1-Pad2) -> col1
- U1 pad 32: D- -> col0
- U1 pad 33: D+ -> +3V3
- U1 pad 34: unconnected-(U1-Pad34) -> row3
- U1 pad 35: GND -> row2
- U1 pad 36: +3V3 -> row1
- U1 pad 37: colA -> row0
- U1 pad 38: col9 -> 26/A0
- U1 pad 39: col8 -> 27/A1
- U1 pad 4: unconnected-(U1-Pad4) -> colD
- U1 pad 40: col7 -> 28/A2
- U1 pad 41: col6 -> 29/A3
- U1 pad 42: col5 -> +3V3
- U1 pad 43: col4 -> +3V3
- U1 pad 44: BOOT0 -> +3V3
- U1 pad 45: col3 -> +1V1
- U1 pad 46: col2 -> Net-(R4-Pad2)
- U1 pad 47: GND -> Net-(R3-Pad2)
- U1 pad 49: GND -> +3V3
- U1 pad 5: OSC+ -> colC
- U1 pad 6: OSC- -> colB
- U1 pad 7: NRST -> colA
- U1 pad 8: GND -> col9
- U1 pad 9: +3V3 -> col8
- Y1 pad 1: OSC+ -> Net-(CX2-Pad2)
- Y1 pad 3: OSC- -> XTAL+
Routing:
- net OSC+: track 6.13 -> 0.00 mm
- net colB: track 15.2 -> 21.4 mm
- net OSC-: track 3.56 -> 0.00 mm
- net colA: track 15.2 -> 18.8 mm
- net LED: track 1.78 -> 0.00 mm
- net 26/A0: track 0.00 -> 1.78 mm
