File: Current/HardLight/HL-2040.kicad_sch (KiCad schematic)
At the start: 46 parts, among them J0 USB, J1 EXT_I2C, J2 Conn_01x02, J3 Conn_01x03, Q0 BSS138, U0 RP2040, U1 LDO-3.3, U2 USBLC6-2SC6, U3 W25Q128JVS, Y0 12MHz

Commit message: HL Mk7 Done Correctly
Parts:
- removed C1: 10uf, EDI:Passive_0402_1005Metric, symbol Device:C_Small
- removed CP2: 10uF, EDI:Passive_0402_1005Metric, symbol Device:C_Small
- removed J2: Conn_01x02, EDI:MicroCon-2, symbol Connector_Generic:Conn_01x02
- removed J3: Conn_01x03, EDI:MicroCon-3, symbol Connector_Generic:Conn_01x03
- removed Q0: BSS138, Package_TO_SOT_SMD:SOT-23, symbol Transistor_FET:BSS138
- removed RQ0, RQ1: 10K, EDI:Passive_0402_1005Metric, symbol Device:R
- added C2: 100nF, EDI:Passive_0402_1005Metric, symbol Device:C_Small
- added CP0: 1uf, EDI:Passive_0402_1005Metric, symbol Device:C_Small
- added H7, H8: Mount, MountingHole:MountingHole_2.2mm_M2_ISO7380_Pad, symbol Mechanical:MountingHole_Pad
- added RF2: 1k, EDI:Passive_0402_1005Metric, symbol Device:R_Small
- added S1: RESET, Button_Switch_SMD:SW_SPST_SKQG_WithoutStem, symbol Switch:SW_SPST
- C10: value 1uf -> 100nF; LCSC C52923 -> C1525
- CP1: value 100nF -> 1uf; LCSC C1525 -> C52923
- CX1, CX2: value 100nF -> 13pf; LCSC C1525 -> C48936
- H1, H2, H3, H4, H5, H6: footprint EDI:SolderableHole -> MountingHole:MountingHole_2.2mm_M2_ISO7380_Pad
- J1: value EXT_I2C -> qwiic; footprint Connector_PinSocket_2.54mm:PinSocket_1x05_P2.54mm_Vertical -> Connector_JST:JST_SH_SM04B-SRSS-TB_1x04-1MP_P1.00mm_Horizontal; symbol Connector_Generic:Conn_01x05 -> Connector_Generic:Conn_01x04; LCSC (none) -> C145956
- RD0, RD1: value 27 -> 27.4; LCSC C413051 -> C172043
- S2: footprint EDI:SW_EVPBB4A9B000 -> Button_Switch_SMD:SW_SPST_SKQG_WithoutStem
- Y0: footprint Crystal:Crystal_SMD_3225-4Pin_3.2x2.5mm -> Crystal:Crystal_SMD_2520-4Pin_2.5x2.0mm; LCSC C9002 -> C2149205
- renumbered C2 to C1
Connections:
- net +1V1: now also C9.1
- net +3V3: now also CP1.1, J1.2 (Pin_2), C2.1, RF2.1; no longer C9.1, J1.4 (Pin_4)
- net 16: now also TX1.1; no longer TX0.1
- net 17: now also TX0.1; no longer TX1.1
- net 20: no longer J1.2 (Pin_2)
- net 21: no longer J1.1 (Pin_1)
- net 28/A2: now also J1.3 (Pin_3)
- net 29/A3: now also J1.4 (Pin_4)
- net CS: now also RF2.2
- net GND: now also CP1.2, J1.1 (Pin_1), C2.2, CP0.1, H7.1, H8.1, S1.1 (A); no longer CP1.1, J1.5 (Pin_5)
- net VBUS: now also CP0.2; no longer CP1.2, J1.3 (Pin_3)
- net ~{RESET}: now also S1.2 (B)
- net XIN: now reaches CX2.2, Y0.1
- net XIN: now also U0.20 (XIN); no longer RX1.2
- net XTAL+ renamed XOUT1
- net XOUT1: now also RX1.2; no longer U0.21 (XOUT)
- net XTAL- renamed XOUT
- net XOUT: now also U0.21 (XOUT); no longer U0.20 (XIN)
- no-connect marks 4 -> 9
Other:
- note added: "C1 near Pin44"
- note added: "C11 near Pin45"
- note added: "qwiic Modular Interface"
- note removed: "Extra Pin Breakouts"
- moved on the sheet: C1, C3, C4, C5, C6, C7, C8, CF1, CX1, CX2, F0, H1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
