File: Current/HardLight/HardLight.kicad_pcb (KiCad board)
At the start: 2 copper layers, 304.8 x 76.2 mm, 237 parts, among them J0 USB, J1 qwiic, J2 SPI Connector, K1 Keyswitch, K10 Keyswitch, K11 Keyswitch, K12 Keyswitch, K13 Keyswitch, K14 Keyswitch, K15 Keyswitch, K16 Keyswitch, K17 Keyswitch, K18 Keyswitch, K19 Keyswitch, K2 Keyswitch, K20 Keyswitch, K21 Keyswitch, K22 Keyswitch, K23 Keyswitch, K24 Keyswitch, K25 Keyswitch, K26 Keyswitch, K27 Keyswitch, K28 Keyswitch, K29 Keyswitch, K3 Keyswitch, K30 Keyswitch, K31 Keyswitch, K32 Keyswitch, K33 Keyswitch, K34 Keyswitch, K35 Keyswitch, K36 Keyswitch, K37 Keyswitch, K38 Keyswitch, K39 Keyswitch, K4 Keyswitch, K40 Keyswitch, K41 Keyswitch, K42 Keyswitch, K43 Keyswitch, K44 Keyswitch, K45 Keyswitch, K46 Keyswitch, K47 Keyswitch, K48 Keyswitch, K49 Keyswitch, K5 Keyswitch, K50 Keyswitch, K51 Keyswitch, K52 Keyswitch, K53 Keyswitch, K54 Keyswitch, K54.1 Keyswitch, K55 Keyswitch, K56 Keyswitch, K57 Keyswitch, K58 Keyswitch, K58.1 Keyswitch, K59 Keyswitch, K6 Keyswitch, K60 Keyswitch, K61 Keyswitch, K62 Keyswitch, K63 Keyswitch, K64 Keyswitch, K7 Keyswitch, K8 Keyswitch, K9 Keyswitch, U0 RP2040, U1 LDO-3.3, U2 USBLC6-2SC6, U3 W25Q128JVS, Y0 CSTCE12M0G55-R0

Commit message: Bulk catchup commit 2023-01-21
Parts:
- TP0: value 22 -> Pin 22
- moved RD1 8.27 mm to (78.2, 84.8), turned to 0 degrees
- moved RD0 7.73 mm to (78.2, 85.9), turned to 0 degrees
- moved CF1 0.82 mm to (82.6, 73.2)
- moved RF2 0.82 mm to (81.5, 73.2)
- moved U3 0.82 mm to (86.6, 76.3)
- moved C4 0.13 mm to (80.6, 91.6)
Routing:
- net GND: track 128.1 -> 457.8 mm, vias 32 -> 27
- net +3V3: track 184.3 -> 39.8 mm, vias 7 -> 13
- net 16: track 63.0 -> 0.00 mm, vias 2 -> 0
- net 14: track 146.8 -> 96.6 mm
- net 13: track 129.6 -> 79.6 mm
- net 15: track 164.1 -> 114.5 mm
- net 17: track 37.8 -> 0.00 mm, vias 2 -> 0
- net Net-(D58-Pad2): track 13.2 -> 0.00 mm
- net Net-(D54-Pad2): track 13.1 -> 0.00 mm
- net DB+: track 40.0 -> 30.4 mm
- net DR+: track 4.53 -> 13.9 mm
- net DR-: track 4.47 -> 13.6 mm
- net DB-: track 40.8 -> 32.4 mm
- net 27/A1: track 60.9 -> 68.4 mm
- net 26/A0: track 308.2 -> 301.0 mm
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- added copper zone on In1.Cu, net +3V3
- added copper zone on In2.Cu, net GND
- removed copper zone on B.Cu, net GND
- removed copper zone on F.Cu, net GND
Other:
- copper layers 2 -> 4
- board text added: ".5"
- board text added: "Test Point"
- board text added: "qwiic SCL SDA 3v3 GND"
- board text removed: ".3"
