File: Current/HardLight/QuicksilverStorm-Matrix.kicad_sch (KiCad schematic)
At the start: 258 parts, among them K1 Keyswitch, K10 Keyswitch, K11 Keyswitch, K12 Keyswitch, K13 Keyswitch, K14 Keyswitch, K15 Keyswitch, K16 Keyswitch, K17 Keyswitch, K18 Keyswitch, K19 Keyswitch, K2 Keyswitch, K20 Keyswitch, K21 Keyswitch, K22 Keyswitch, K23 Keyswitch, K24 Keyswitch, K25 Keyswitch, K26 Keyswitch, K27 Keyswitch, K28 Keyswitch, K29 Keyswitch, K3 Keyswitch, K30 Keyswitch, K31 Keyswitch, K32 Keyswitch, K33 Keyswitch, K34 Keyswitch, K35 Keyswitch, K36 Keyswitch, K37 Keyswitch, K38 Keyswitch, K39 Keyswitch, K4 Keyswitch, K40 Keyswitch, K41 Keyswitch, K42 Keyswitch, K43 Keyswitch, K44 Keyswitch, K45 Keyswitch, K46 Keyswitch, K47 Keyswitch, K48 Keyswitch, K49 Keyswitch, K5 Keyswitch, K50 Keyswitch, K51 Keyswitch, K52 Keyswitch, K53 Keyswitch, K54 Keyswitch, K54.1 Keyswitch, K55 Keyswitch, K56 Keyswitch, K57 Keyswitch, K58 Keyswitch, K58.1 Keyswitch, K59 Keyswitch, K6 Keyswitch, K60 Keyswitch, K61 Keyswitch, K62 Keyswitch, K63 Keyswitch, K64 Keyswitch, K7 Keyswitch, K8 Keyswitch, K9 Keyswitch

Commit message: Final Warning begins. Sweet Business done.
Parts:
- K1, K10, K11, K12, K13, K14, K15, K16, K17, K18, K19, K2, K20, K21, K22, K23, K24, K25, K26, K27, K28, K29, K3, K30, K31, K32, K33, K34, K35, K36, K37, K38, K39, K4, K40, K41, K42, K43, K44, K45, K46, K47, K48, K49, K5, K50, K51, K52, K53, K54, K54.1, K55, K56, K57, K58, K58.1, K59, K6, K60, K61, K62, K63, K64, K7, K8, K9: footprint EDI:SW_PG1350 -> EDI:MX-Choc
- LD1, LD10, LD11, LD12, LD13, LD14, LD15, LD16, LD17, LD18, LD19, LD2, LD20, LD21, LD22, LD23, LD24, LD25, LD26, LD27, LD28, LD29, LD3, LD30, LD31, LD32, LD4, LD5, LD6, LD7, LD8, LD9: footprint EDI:WS2812B_2020 -> EDI:WS2812C_2020
