File: Current/SweetBusiness2040/SweetBusiness.kicad_sch (KiCad schematic)
At the start: 60 parts, among them J2 I2C, J3 Bridge, J4 USB, U0 RP2040, U1 MT2492, U2 W25Q128JVS, U3 USBLC6-2SC6, Y1 12MHz

Commit message: HL, WE, SB updates.
Parts:
- added S2: RESET, Button_Switch_SMD:SW_SPST_SKQG_WithoutStem, symbol Switch:SW_SPST
- C10, C2: value 1uf -> 100nF; LCSC C52923 -> C1525
- C11: value 10uf -> 100nF; LCSC C23733 -> C1525
- C8, C9: value 100nF -> 1uf; LCSC C1525 -> C52923
- CX1, CX2: value 100nF -> 13pf; LCSC C1525 -> C48936
- H1, H2, H3, H4, H5, H6, H7, H8: footprint EDI:SolderableHole-M2 -> MountingHole:MountingHole_3.2mm_M3; symbol Mechanical:MountingHole_Pad -> Mechanical:MountingHole
- S1: footprint EDI:SW_EVPBB4A9B000 -> Button_Switch_SMD:SW_SPST_SKQG_WithoutStem; LCSC C140848 -> C139779
- Y1: value 12MHz -> 2TJ412000NYGBC 12MHz; footprint Crystal:Crystal_SMD_3225-4Pin_3.2x2.5mm -> Crystal:Crystal_SMD_2520-4Pin_2.5x2.0mm; LCSC C9002 -> C2149205
Connections:
- net +1V1: now also C10.1, C11.1, C9.1; no longer C1.1, C2.1
- net +3V3: now also C1.1, C2.1; no longer C10.1, C11.1, C9.1
- net GND: now also S2.1 (A); no longer H1.1, H2.1, H3.1, H4.1, H5.1, H6.1, H7.1, H8.1
- net ~{RESET}: now reaches RR1.2, U0.26 (RUN)
- net ~{RESET}: now also S2.2 (B)
- net XIN: now reaches CX2.2, Y1.1
- net XIN: now also U0.20 (XIN); no longer RX2.2
- net XTAL+ renamed XOUT1
- net XOUT1: now also RX2.2; no longer U0.21 (XOUT)
- net XTAL- renamed XOUT
- net XOUT: now also U0.21 (XOUT); no longer U0.20 (XIN)
Other:
- note added: "C8 near Pin44"
- note added: "C9 near Pin45"
