File: Current/SweetBusiness2040/SweetBusinessRGBCore/SweetBusinessRGBCore.kicad_sch (KiCad schematic)
At the start: 270 parts, among them J1 Bridge, J2 Toggle Link, T1 Keyswitch, T2 Keyswitch, T3 Keyswitch, T4 Keyswitch

Commit message: HL, WE, SB updates.
Parts:
- H1, H2, H3, H4, H5, H6, H7, H8: footprint EDI:SolderableHole-M2 -> MountingHole:MountingHole_3.2mm_M3; symbol Mechanical:MountingHole_Pad -> Mechanical:MountingHole
Connections:
- net GND: no longer H1.1, H2.1, H3.1, H4.1, H5.1, H6.1, H7.1, H8.1
- net row1: now also J2.3 (Pin_3), J2.7 (Pin_7)
