File: Current/TwoTailed/TwoTailed.kicad_sch (KiCad schematic)
At the start: 44 parts, among them J1 USB, J2 I2C, U1 STM32F411VETx, U2 LDO-3.3, U3 USBLC6-2SC6, Y1 8MHz

Commit message: Nice changelog, idiot.
Parts:
- removed CF7, CF8: 100nF, EDI:Passive_0402_1005Metric, symbol Device:C_Small
- removed CV2: 4.7uF, EDI:Passive_0402_1005Metric, symbol Device:C_Small
- removed RM1: 100k, EDI:Passive_0402_1005Metric, symbol Device:R_Small
- removed RM2: 100K, EDI:Passive_0402_1005Metric, symbol Device:R_Small
- removed RR1: 47, EDI:Passive_0402_1005Metric, symbol Device:R_Small
- removed U1: STM32F411VETx, Package_QFP:LQFP-100_14x14mm_P0.5mm, symbol MCU_ST_STM32F4:STM32F411VETx
- removed U3: USBLC6-2SC6, Package_TO_SOT_SMD:SOT-23-6, symbol Power_Protection:USBLC6-2SC6
- added RB2: 100K, EDI:Passive_0402_1005Metric, symbol Device:R_Small
- added RB3: 100k, EDI:Passive_0402_1005Metric, symbol Device:R_Small
- added U0: STM32F411RETx, Package_QFP:LQFP-64_10x10mm_P0.5mm, symbol MCU_ST_STM32F4:STM32F411RETx
- H1, H2, H3, H4, H5, H6, H7, H8: footprint MountingHole:MountingHole_2.7mm_M2.5_ISO14580_Pad -> EDI:SolderableHole-M2
Connections:
- net +3V3: now also RB2.1, U0.1 (VBAT), U0.13 (VDDA), U0.19 (VDD), U0.32 (VDD), U0.48 (VDD), U0.64 (VDD); no longer DK2.2 (A)
- net BOOT0: now also U0.60 (BOOT0)
- net CAPS: now also U0.39 (PC8)
- net D+: now also U0.45 (PA12)
- net D-: now also U0.44 (PA11)
- net GND: now also DK2.1 (K), RB3.2, U0.12 (VSSA), U0.18 (VSS), U0.31 (VSS), U0.47 (VSS), U0.63 (VSS)
- net NRST: now also U0.7 (NRST)
- net NUM: now also U0.41 (PA8)
- net OSC+: now also U0.5 (PH0)
- net OSC-: now also U0.6 (PH1)
- net SCL: now also U0.58 (PB6)
- net SCRL: now also U0.40 (PC9)
- net SDA: now also U0.59 (PB7)
- net col0: now also U0.38 (PC7)
- net col1: now also U0.37 (PC6)
- net col10: now also U0.52 (PC11)
- net col11: now also U0.51 (PC10)
- net col12: now also U0.50 (PA15)
- net col2: now also U0.20 (PA4)
- net col3: now also U0.21 (PA5)
- net col4: now also U0.22 (PA6)
- net col5: now also U0.23 (PA7)
- net col6: now also U0.24 (PC4)
- net col7: now also U0.25 (PC5)
- net col8: now also U0.26 (PB0)
- net col9: now also U0.62 (PB9)
- net colA: now also U0.61 (PB8)
- net colB: now also U0.57 (PB5)
- net colC: now also U0.56 (PB4)
- net colD: now also U0.55 (PB3)
- net colE: now also U0.54 (PD2)
- net colF: now also U0.53 (PC12)
- net enc0A: now also U0.46 (PA13)
- net enc0B: now also U0.49 (PA14)
- net row0: now also U0.29 (PB10)
- net row1: now also U0.33 (PB12)
- net row2: now also U0.17 (PA3)
- net row3: now also U0.16 (PA2)
- net row4: now also U0.15 (PA1)
- net row5: now also U0.14 (PA0)
- net row6: now also U0.11 (PC3)
- net at CV1.1: now also U0.30 (VCAP1)
- net at RL2.1: now also DK2.2 (A); no longer DK2.1 (K)
- new net: RB2.2, U0.43 (PA10)
- new net: RB3.1, U0.28 (PB2)
Other:
- note removed: "ESD Isolator"
- moved on the sheet: DK2

Commit message: oh my god just stop
Parts:
- removed C1: 100nF, EDI:Passive_0402_1005Metric, symbol Device:C_Small
- removed C2: 10uF, EDI:Passive_0402_1005Metric, symbol Device:C_Small
- removed U2: LDO-3.3, Package_TO_SOT_SMD:SOT-23, symbol Regulator_Linear:LD1117S33TR_SOT223
- added CP1: 100nF, EDI:Passive_0402_1005Metric, symbol Device:C_Small
- added CP10, CP11, CP12, CP13, CP14, CP15, CP16, CP17, CP2, CP3, CP4, CP5, CP6, CP7, CP8, CP9: 22uf, EDI:Passive_0402_1005Metric, symbol Device:C_Small
- added LP1: 10uH, Inductor_SMD:L_Wuerth_HCI-1040, symbol Device:L
- added RP1: 100K, EDI:Passive_0402_1005Metric, symbol Device:R_Small
- added RP2: 22.1K, EDI:Passive_0402_1005Metric, symbol Device:R_Small
- added U1: MT2492, Package_TO_SOT_SMD:SOT-23-6, symbol EDI:MT2492
- S1, S2: footprint Button_Switch_SMD:SW_SPST_SKQG_WithoutStem -> EDI:SW_EVPBB4A9B000
Connections:
- net +3V3: now also CP10.1, CP11.1, CP12.1, CP13.1, CP14.1, CP15.1, CP16.1, CP17.1, LP1.2, RP1.1
- net GND: now also CP10.2, CP11.2, CP12.2, CP13.2, CP14.2, CP15.2, CP16.2, CP17.2, CP2.1, CP3.1, CP4.1, CP5.1, CP6.1, CP7.1, CP8.1, CP9.1, RP2.2, U1.2 (GND)
- net VBUS: now also CP2.2, CP3.2, CP4.2, CP5.2, CP6.2, CP7.2, CP8.2, CP9.2, U1.4 (EN), U1.5 (VIN)
- new net: CP1.1, U1.1 (BS)
- new net: RP1.2, RP2.1, U1.3 (FB)
- new net: CP1.2, LP1.1, U1.6 (SW)
Other:
- moved on the sheet: CV1, RB2, RB3, U0

Commit message: Whole bunch of work!
Parts:
- removed CF2, CF3, CF4, CF6, CR1: 100nF, EDI:Passive_0402_1005Metric, symbol Device:C_Small
- removed CF5, CV1: 4.7uF, EDI:Passive_0402_1005Metric, symbol Device:C_Small
- removed CP10, CP11, CP12, CP13, CP14, CP15, CP16, CP17, CP3, CP4, CP5, CP6, CP7, CP8, CP9: 22uf, EDI:Passive_0402_1005Metric, symbol Device:C_Small
- removed CY1, CY2: 0.012nF, EDI:Passive_0402_1005Metric, symbol Device:C_Small
- removed DK1: Caps, LED_THT:LED_D1.8mm_W3.3mm_H2.4mm, symbol Device:LED
- removed DK2: Scroll, LED_THT:LED_D1.8mm_W3.3mm_H2.4mm, symbol Device:LED
- removed DK3: Num, LED_THT:LED_D1.8mm_W3.3mm_H2.4mm, symbol Device:LED
- removed H7, H8: Mount, EDI:SolderableHole-M2, symbol Mechanical:MountingHole_Pad
- removed J1: USB, Connector_USB:USB_C_Receptacle_HRO_TYPE-C-31-M-12, symbol HL-Mk3-rescue:USB_C_Receptacle_USB2.0-Connector-HL-Mk2-rescue
- removed LP1: 10uH, Inductor_SMD:L_Wuerth_HCI-1040, symbol Device:L
- removed RB1: 10k, EDI:Passive_0402_1005Metric, symbol Device:R_Small
- removed RB2, RP1: 100K, EDI:Passive_0402_1005Metric, symbol Device:R_Small
- removed RB3: 100k, EDI:Passive_0402_1005Metric, symbol Device:R_Small
- removed RL1, RL2, RL3: 270, EDI:Passive_0402_1005Metric, symbol Device:R_Small
- removed RP2: 22.1K, EDI:Passive_0402_1005Metric, symbol Device:R_Small
- removed RU1, RU2: 5k1, EDI:Passive_0402_1005Metric, symbol Device:R_Small
- removed U0: STM32F411RETx, Package_QFP:LQFP-64_10x10mm_P0.5mm, symbol MCU_ST_STM32F4:STM32F411RETx
- removed U1: MT2492, Package_TO_SOT_SMD:SOT-23-6, symbol EDI:MT2492
- removed Y1: 8MHz, Crystal:Crystal_SMD_3225-4Pin_3.2x2.5mm, symbol Device:Crystal_GND24_Small
- added C1, C3, C4, C5, C6, C7, C8, C9, CX1, CX2: 100nF, EDI:Passive_0402_1005Metric, symbol Device:C_Small
- added C10, C2: 1uf, EDI:Passive_0402_1005Metric, symbol Device:C_Small
- added C11: 10uf, EDI:Passive_0402_1005Metric, symbol Device:C_Small
- added J1: USB, Connector_USB:USB_C_Receptacle_HRO_TYPE-C-31-M-12, symbol HL-Mk2-rescue:USB_C_Receptacle_USB2.0-Connector
- added RC1, RC2: 5k1, EDI:Passive_0402_1005Metric, symbol Device:R_Small
- added RD1, RD2: 27, EDI:Passive_0402_1005Metric, symbol Device:R_Small
- added RF1, RR1, RX2: 1k, EDI:Passive_0402_1005Metric, symbol Device:R_Small
- added U0: RP2040, Package_DFN_QFN:QFN-56-1EP_7x7mm_P0.4mm_EP5.6x5.6mm_ThermalVias, symbol RP2040:RP2040
- added U1: LDO-3.3, Package_TO_SOT_SMD:SOT-23, symbol Regulator_Linear:LD1117S33TR_SOT223
- added U2: USBLC6-2SC6, Package_TO_SOT_SMD:SOT-23-6, symbol Power_Protection:USBLC6-2SC6
- added U3: W25Q128JVS, Package_SO:SOIC-8_5.23x5.23mm_P1.27mm, symbol Memory_Flash:W25Q128JVS
- added Y1: 12MHz, Crystal:Crystal_SMD_3225-4Pin_3.2x2.5mm, symbol Device:Crystal_GND24
- CP2: value 22uf -> 10uF; LCSC C415703 -> C15525
- H1, H2, H3, H4, H5, H6: footprint EDI:SolderableHole-M2 -> EDI:SolderableHole
- S1: value RESET -> USB BOOT; LCSC C115351 -> C140848
- S2: value BOOTLOADER -> RESET; LCSC C115351 -> C140848
Connections:
- net NRST is gone; now on net GND: S1.1 (A)
- net +3V3: now also CP2.2, C10.1, C11.1, C3.1, C4.1, C5.1, C6.1, C7.1, C8.1, C9.1, RR1.1, U0.1 (IOVDD), U0.10 (IOVDD), U0.22 (IOVDD), U0.33 (IOVDD), U0.42 (IOVDD), U0.43 (ADC_AVDD), U0.44 (VREG_VIN), U0.48 (USB_VDD), U0.49 (IOVDD), U1.2 (VO), U3.8 (VCC); no longer S2.2 (B)
- net D+: now also J1.A6 (D+), J1.B6 (D+), U2.6 (I/O1)
- net D-: now also J1.A7 (D-), J1.B7 (D-), U2.4 (I/O2)
- net GND: now also CP1.1, S2.2 (B), C1.2, C10.2, C11.2, C2.2, C3.2, C4.2, C5.2, C6.2, C7.2, C8.2, C9.2, CX1.2, CX2.1, J1.A1 (GND), J1.A12 (GND), J1.B1 (GND), J1.B12 (GND), J1.S1 (SHIELD), RC1.1, RC2.2, U0.19 (TESTEN), U0.57 (GND), U1.1 (GND), U2.2 (GND), U3.4 (GND), Y1.2, Y1.4; no longer S1.2 (B)
- net VBUS: now also CP1.2, U1.3 (VI), U2.5 (VBUS); no longer CP2.2
- net +5V renamed +5v
- net +5v: now also J1.A4 (VBUS), J1.A9 (VBUS), J1.B4 (VBUS), J1.B9 (VBUS)
- net BOOT0 renamed ~{RESET}
- net ~{RESET}: now also RR1.2, U0.26 (RUN)
- new net: RD1.2, U0.47 (USB_DP)
- new net: RF1.2, S1.2 (B)
- new net: RD2.2, U0.46 (USB_DM)
- new net: CX2.2, RX2.2, Y1.1
- new net: J1.A5 (CC1), RC2.1
- new net: J1.B5 (CC2), RC1.2
- new net +1V1: C1.1, C2.1, U0.23 (DVDD), U0.45 (VREG_VOUT), U0.50 (DVDD)
- new net 0: U0.2 (GPIO0)
- new net 1: U0.3 (GPIO1)
- new net 10: U0.13 (GPIO10)
- new net 11: U0.14 (GPIO11)
- new net 12: U0.15 (GPIO12)
- new net 13: U0.16 (GPIO13)
- new net 14: U0.17 (GPIO14)
- new net 15: U0.18 (GPIO15)
- new net 16: U0.27 (GPIO16)
- new net 17: U0.28 (GPIO17)
- new net 18: U0.29 (GPIO18)
- new net 19: U0.30 (GPIO19)
- new net 2: U0.4 (GPIO2)
- new net 20: U0.31 (GPIO20)
- new net 21: U0.32 (GPIO21)
- new net 22: U0.34 (GPIO22)
- new net 23: U0.35 (GPIO23)
- new net 24: U0.36 (GPIO24)
- new net 25: U0.37 (GPIO25)
- new net 26/A0: U0.38 (GPIO26/ADC0)
- new net 27/A1: U0.39 (GPIO27/ADC1)
- new net 28/A2: U0.40 (GPIO28/ADC2)
- new net 29/A3: U0.41 (GPIO29/ADC3)
- new net 3: U0.5 (GPIO3)
- new net 4: U0.6 (GPIO4)
- new net 5: U0.7 (GPIO5)
- new net 6: U0.8 (GPIO6)
- new net 7: U0.9 (GPIO7)
- new net 8: U0.11 (GPIO8)
- new net 9: U0.12 (GPIO9)
- new net CLOCK: U0.52 (QSPI_SCLK), U3.6 (CLK)
- new net CS: RF1.1, U0.56 (QSPI_SS_N), U3.1 (~{CS})
- new net DB+: RD1.1, U2.1 (I/O1)
- new net DB-: RD2.1, U2.3 (I/O2)
- new net SD0: U0.53 (QSPI_SD0), U3.5 (DI(IO0))
- new net SD1: U0.55 (QSPI_SD1), U3.2 (DO(IO1))
- new net SD2: U0.54 (QSPI_SD2), U3.3 (IO2)
- new net SD3: U0.51 (QSPI_SD3), U3.7 (IO3)
- new net XTAL+: CX1.1, U0.21 (XOUT), Y1.3
- new net XTAL-: RX2.1, U0.20 (XIN)
- no-connect marks 3 -> 4
Other:
- note added: "Chassis Ground Mount Points"
- note added: "Clock Reference"
- note added: "ESD Isolator"
- note added: "External Interface System"
- note added: "Flash (128MB)"
- note added: "GPIO Interface Map"
- note added: "Microcontroller Core"
- note added: "Microcontroller Power Regulation"
- note added: "USB port"
- moved on the sheet: J2

Commit message: HL Mk7 READY FOR PRIMETIME
Parts:
- removed S2: RESET, EDI:SW_EVPBB4A9B000, symbol Switch:SW_SPST
- renumbered RX2 to RX1
Connections:
- net SCL is gone; now on net 1: J2.3 (Pin_3)
- net SDA is gone; now on net 0: J2.4 (Pin_4)
- net ~{RESET}: no longer names the net of RR1.2, U0.26 (RUN)
Other:
- moved on the sheet: J2, RR1

Commit message: So much stuff
Wow it's been a while.
Parts:
- removed C11: 10uf, EDI:Passive_0402_1005Metric, symbol Device:C_Small
- removed CF1, CX2: 100nF, EDI:Passive_0402_1005Metric, symbol Device:C_Small
- removed CP2: 10uF, EDI:Passive_0402_1005Metric, symbol Device:C_Small
- removed F1: 6v 500ma, Fuse:Fuse_0603_1608Metric, symbol Device:Polyfuse_Small
- removed H1, H2, H3, H4, H5, H6: Mount, EDI:SolderableHole, symbol Mechanical:MountingHole_Pad
- removed J1: USB, Connector_USB:USB_C_Receptacle_HRO_TYPE-C-31-M-12, symbol HL-Mk2-rescue:USB_C_Receptacle_USB2.0-Connector
- removed J2: I2C, Connector_PinHeader_2.54mm:PinHeader_1x04_P2.54mm_Vertical, symbol Connector:Conn_01x04_Male
- removed RC2: 5k1, EDI:Passive_0402_1005Metric, symbol Device:R_Small
- removed RD2: 27, EDI:Passive_0402_1005Metric, symbol Device:R_Small
- removed RR1, RX1: 1k, EDI:Passive_0402_1005Metric, symbol Device:R_Small
- removed U3: W25Q128JVS, Package_SO:SOIC-8_5.23x5.23mm_P1.27mm, symbol Memory_Flash:W25Q128JVS
- removed Y1: 12MHz, Crystal:Crystal_SMD_3225-4Pin_3.2x2.5mm, symbol Device:Crystal_GND24
- added C0, CP0: 1uf, EDI:Passive_0402_1005Metric, symbol Device:C_Small
- added CF0: 100nF, EDI:Passive_0402_1005Metric, symbol Device:C_Small
- added CX0: 13pf, EDI:Passive_0402_1005Metric, symbol Device:C_Small
- added F0: 6v 500ma, Fuse:Fuse_0603_1608Metric, symbol Device:Polyfuse_Small
- added H0, H1, H2, H3, H4, H5, H6, H7: Mount, MountingHole:MountingHole_3.2mm_M3, symbol Mechanical:MountingHole
- added J0: USB, Connector_USB:USB_C_Receptacle_HRO_TYPE-C-31-M-12, symbol HL-Mk2-rescue:USB_C_Receptacle_USB2.0-Connector
- added J1: qwiic, Connector_JST:JST_SH_SM04B-SRSS-TB_1x04-1MP_P1.00mm_Horizontal, symbol Connector_Generic:Conn_01x05
- added RC0: 5k1, EDI:Passive_0402_1005Metric, symbol Device:R_Small
- added RD0: 27.4, EDI:Passive_0402_1005Metric, symbol Device:R_Small
- added RF0, RR0, RX0: 1k, EDI:Passive_0402_1005Metric, symbol Device:R_Small
- added S0: RESET, Button_Switch_SMD:SW_SPST_SKQG_WithoutStem, symbol Switch:SW_SPST
- added TX0, TX1: Transducer, Buzzer_Beeper:Buzzer_CUI_CPT-9019S-SMT, symbol Device:Speaker_Crystal
- added U3: W25Q128JVS, Package_SON:WSON-8-1EP_6x5mm_P1.27mm_EP3.4x4.3mm, symbol Memory_Flash:W25Q32JVZP
- added Y0: 2TJ412000NYGBC 12MHz, Crystal:Crystal_SMD_2520-4Pin_2.5x2.0mm, symbol Device:Crystal_GND24
- C2: value 1uf -> 100nF; LCSC C52923 -> C1525
- CP1: value 100nF -> 1uf; LCSC C1525 -> C52923
- CX1: value 100nF -> 13pf; LCSC C1525 -> C48936
- RD1: value 27 -> 27.4; LCSC C413051 -> C172043
- S1: footprint EDI:SW_EVPBB4A9B000 -> Button_Switch_SMD:SW_SPST_SKQG_WithoutStem; LCSC C140848 -> C139779
Connections:
- net +1V1: now also C10.1, C8.1, C9.1; no longer C1.1, C2.1
- net +3V3: now also C1.1, C2.1, CP1.1, C0.1, CF0.1, J1.2 (Pin_2), RF0.1, RR0.1, U3.8 (VCC); no longer C10.1, C8.1, C9.1
- net 16: now also TX1.1
- net 17: now also TX0.1
- net 28/A2: now also J1.3 (Pin_3)
- net 29/A3: now also J1.4 (Pin_4)
- net CLOCK: now also U3.6 (CLK)
- net CS: now also RF0.2, U3.1 (~{CS})
- net D+: now also J0.A6 (D+), J0.B6 (D+)
- net D-: now also J0.A7 (D-), J0.B7 (D-)
- net DB+: now also RD0.1; no longer RD1.1
- net DB-: now also RD1.1
- net GND: now also CP1.2, CX1.1, C0.2, CF0.2, CP0.1, CX0.2, J0.A1 (GND), J0.A12 (GND), J0.B1 (GND), J0.B12 (GND), J0.S1 (SHIELD), J1.1 (Pin_1), J1.MP, RC0.2, S0.1 (A), TX0.2, TX1.2, U3.4 (GND), U3.9 (EP), Y0.2, Y0.4; no longer CP1.1, CX1.2
- net SD0: now also U3.5 (DI(IO0))
- net SD1: now also U3.2 (DO(IO1))
- net SD2: now also U3.3 (IO2)
- net SD3: now also U3.7 (IO3)
- net VBUS: now also CP0.2, F0.2; no longer CP1.2
- net DR+: now reaches U0.47 (USB_DP)
- net DR+: now also RD0.2; no longer RD1.2
- net DR-: now reaches U0.46 (USB_DM)
- net DR-: now also RD1.2
- net ~{RESET}: now reaches U0.26 (RUN)
- net ~{RESET}: now also RR0.2, S0.2 (B)
- net at RC1.2: now also J0.B5 (CC2)
- net XTAL+ renamed XOUT
- net XOUT: now also RX0.1; no longer CX1.1
- net XTAL- renamed XIN
- net XIN: now also CX1.2, Y0.1
- new net: J0.A5 (CC1), RC0.1
- new net XOUT1: CX0.1, RX0.2, Y0.3
- new net vUSB: F0.1, J0.A4 (VBUS), J0.A9 (VBUS), J0.B4 (VBUS), J0.B9 (VBUS)
Other:
- note added: "Audio Feedback System"
- note added: "C0 near Pin44"
- note added: "C10 near Pin45"
- note added: "Flash (16MB)"
- note added: "Power Control System"
- note added: "qwiic Modular Interface"
- note removed: "Flash (128MB)"
