File: Current/TwoTailed/borealis-mtx.kicad_sch (KiCad schematic)
At the start: 250 parts, among them K1 Keyswitch, K10 Keyswitch, K100 Keyswitch, K101 Keyswitch, K102 Keyswitch, K103 Keyswitch, K104 Keyswitch, K105 Keyswitch, K106 Keyswitch, K107 Keyswitch, K108 Keyswitch, K109 Keyswitch, K11 Keyswitch, K110 Keyswitch, K111 Keyswitch, K112 Keyswitch, K113 Keyswitch, K114 Keyswitch, K115 Keyswitch, K116 Keyswitch, K117 Keyswitch, K118 Keyswitch, K12 Keyswitch, K13 Keyswitch, K14 Keyswitch, K15 Keyswitch, K16 Keyswitch, K17 Keyswitch, K18 Keyswitch, K19 Keyswitch, K2 Keyswitch, K20 Keyswitch, K21 Keyswitch, K22 Keyswitch, K23 Keyswitch, K24 Keyswitch, K25 Keyswitch, K26 Keyswitch, K27 Keyswitch, K28 Keyswitch, K29 Keyswitch, K3 Keyswitch, K30 Keyswitch, K31 Keyswitch, K32 Keyswitch, K33 Keyswitch, K34 Keyswitch, K35 Keyswitch, K36 Keyswitch, K37 Keyswitch, K38 Keyswitch, K39 Keyswitch, K4 Keyswitch, K40 Keyswitch, K41 Keyswitch, K42 Keyswitch, K43 Keyswitch, K44 Keyswitch, K45 Keyswitch, K46 Keyswitch, K47 Keyswitch, K48 Keyswitch, K49 Keyswitch, K5 Keyswitch, K50 Keyswitch, K51 Keyswitch, K52 Keyswitch, K53 Keyswitch, K54 Keyswitch, K55 Keyswitch, K56 Keyswitch, K57 Keyswitch, K58 Keyswitch, K59 Keyswitch, K6 Keyswitch, K60 Keyswitch, K61 Keyswitch, K62 Keyswitch, K63 Keyswitch, K64 Keyswitch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

Commit message: Nice changelog, idiot.
Parts:
- removed D109: 1N4148W-T4, EDI:D_SOD-523, symbol Device:D_Small
- removed K109: Keyswitch, EDI:MX-Choc, symbol EDI:Keyswitch
- K108: footprint EDI:MX-Choc-Double -> EDI:MX-Choc
- K111: renamed from K112; footprint EDI:MX-Choc-Double -> EDI:MX-Choc
- renumbered D110 to D109, D111 to D110, D112 to D111, D113 to D112, D114 to D113, D115 to D114, D116 to D115, D117 to D116, D118 to D117, DR0 to DR1, JT0 to JT1, JT1 to JT2, K110 to K109, K111 to K110, K113 to K112, K114 to K113, K115 to K114, K116 to K115, K117 to K116, K118 to K117, RX0 to RX1

Commit message: oh my god just stop
Parts:
- K1, K10, K100, K101, K102, K103, K104, K105, K106, K107, K108, K109, K11, K110, K111, K112, K113, K114, K115, K116, K117, K12, K13, K14, K15, K16, K17, K18, K19, K2, K20, K21, K22, K23, K24, K25, K26, K27, K28, K29, K3, K30, K31, K32, K33, K34, K35, K36, K37, K38, K39, K4, K40, K41, K42, K43, K44, K45, K46, K47, K48, K49, K5, K50, K51, K52, K53, K54, K55, K56, K57, K58, K59, K6, K60, K61, K62, K63, K64, K65, K66, K67, K68, K69, K7, K70, K71, K72, K73, K74, K75, K76, K77, K78, K79, K8, K80, K81, K82, K83, K84, K85, K86, K87, K88, K89, K9, K90, K91, K92, K93, K94, K95, K96, K97, K98, K99: footprint EDI:MX-Choc -> EDI:MX-Choc-RGB

Commit message: Whole bunch of work!
Parts:
- removed DR1: SOD-523, EDI:D_SOD-523, symbol Device:D_Small
- removed RX1: Volume, EDI:MX-Choc-Enc, symbol Device:Rotary_Encoder_Switch
- K1, K10, K100, K101, K102, K103, K104, K105, K106, K107, K108, K109, K11, K110, K111, K112, K113, K114, K115, K116, K117, K12, K13, K14, K15, K16, K17, K18, K19, K2, K20, K21, K22, K23, K24, K25, K26, K27, K28, K29, K3, K30, K31, K32, K33, K34, K35, K36, K37, K38, K39, K4, K40, K41, K42, K43, K44, K45, K46, K47, K48, K49, K5, K50, K51, K52, K53, K54, K55, K56, K57, K58, K59, K6, K60, K61, K62, K63, K64, K65, K66, K67, K68, K69, K7, K70, K71, K72, K73, K74, K75, K76, K77, K78, K79, K8, K80, K81, K82, K83, K84, K85, K86, K87, K88, K89, K9, K90, K91, K92, K93, K94, K95, K96, K97, K98, K99: footprint EDI:MX-Choc-RGB -> EDI:MX-Choc
Other:
- moved on the sheet: JT2

Commit message: So much stuff
Wow it's been a while.
Parts:
- removed D1, D10, D2, D3, D4, D5, D6, D7, D8, D9: 1N4148W-T4, EDI:D_SOD-523, symbol Device:D_Small
- removed DT1, DT10, DT2, DT3, DT4, DT5, DT6, DT7, DT8, DT9: SOD-523, EDI:D_SOD-523, symbol Device:D_Small
- removed JT1: Toggle Block N, Connector_PinHeader_2.54mm:PinHeader_2x05_P2.54mm_Vertical, symbol Connector_Generic:Conn_02x05_Odd_Even
- removed JT2: Toggle Block E, Connector_PinHeader_2.54mm:PinHeader_2x05_P2.54mm_Vertical, symbol Connector_Generic:Conn_02x05_Odd_Even
- removed K1, K10, K2, K3, K4, K5, K6, K7, K8, K9: Keyswitch, EDI:MX-Choc, symbol EDI:Keyswitch
- renumbered D11 to D0, D12 to D1, D21 to D10, D111 to D100, D112 to D101, D113 to D102, D114 to D103, D115 to D104, D116 to D105, D117 to D106, D22 to D11, D23 to D12, D24 to D13, D25 to D14, D26 to D15, D27 to D16, D28 to D17, D29 to D18, D30 to D19, D13 to D2, D31 to D20, D32 to D21, D33 to D22, D34 to D23, D35 to D24, D36 to D25, D37 to D26, D38 to D27, D39 to D28, D40 to D29, D14 to D3, D41 to D30, D42 to D31, D43 to D32, D44 to D33, D45 to D34, D46 to D35, D47 to D36, D48 to D37, D49 to D38, D50 to D39, D15 to D4, D51 to D40, D52 to D41, D53 to D42, D54 to D43, D55 to D44, D56 to D45, D57 to D46, D58 to D47, D59 to D48, D60 to D49, D16 to D5, D61 to D50, D62 to D51, D63 to D52, D64 to D53, D65 to D54, D66 to D55, D67 to D56, D68 to D57, D69 to D58, D70 to D59, D17 to D6, D71 to D60, D72 to D61, D73 to D62, D74 to D63, D75 to D64, D76 to D65, D77 to D66, D78 to D67, D79 to D68, D80 to D69, D18 to D7, D81 to D70, D82 to D71, D83 to D72, D84 to D73, D85 to D74, D86 to D75, D87 to D76, D88 to D77, D89 to D78, D90 to D79, D19 to D8, D91 to D80, D92 to D81, D93 to D82, D94 to D83, D95 to D84, D96 to D85, D97 to D86, D98 to D87, D99 to D88, D100 to D89, D20 to D9, D101 to D90, D102 to D91, D103 to D92, D104 to D93, D105 to D94, D106 to D95, D107 to D96, D108 to D97, D109 to D98, D110 to D99, K11 to K0, K12 to K1, K21 to K10, K111 to K100, K112 to K101, K113 to K102, K114 to K103, K115 to K104, K116 to K105, K117 to K106, K22 to K11, K23 to K12, K24 to K13, K25 to K14, K26 to K15, K27 to K16, K28 to K17, K29 to K18, K30 to K19, K13 to K2, K31 to K20, K32 to K21, K33 to K22, K34 to K23, K35 to K24, K36 to K25, K37 to K26, K38 to K27, K39 to K28, K40 to K29, K14 to K3, K41 to K30, K42 to K31, K43 to K32, K44 to K33, K45 to K34, K46 to K35, K47 to K36, K48 to K37, K49 to K38, K50 to K39, K15 to K4, K51 to K40, K52 to K41, K53 to K42, K54 to K43, K55 to K44, K56 to K45, K57 to K46, K58 to K47, K59 to K48, K60 to K49, K16 to K5, K61 to K50, K62 to K51, K63 to K52, K64 to K53, K65 to K54, K66 to K55, K67 to K56, K68 to K57, K69 to K58, K70 to K59, K17 to K6, K71 to K60, K72 to K61, K73 to K62, K74 to K63, K75 to K64, K76 to K65, K77 to K66, K78 to K67, K79 to K68, K80 to K69, K18 to K7, K81 to K70, K82 to K71, K83 to K72, K84 to K73, K85 to K74, K86 to K75, K87 to K76, K88 to K77, K89 to K78, K90 to K79, K19 to K8, K91 to K80, K92 to K81, K93 to K82, K94 to K83, K95 to K84, K96 to K85, K97 to K86, K98 to K87, K99 to K88, K100 to K89, K20 to K9, K101 to K90, K102 to K91, K103 to K92, K104 to K93, K105 to K94, K106 to K95, K107 to K96, K108 to K97, K109 to K98, K110 to K99
Connections:
- net row6 is gone; now on net row5: D100.1 (K), D101.1 (K), D102.1 (K), D103.1 (K), D104.1 (K), D105.1 (K), D106.1 (K), D90.1 (K), D91.1 (K), D92.1 (K), D93.1 (K), D94.1 (K), D95.1 (K), D96.1 (K), D97.1 (K), D98.1 (K), D99.1 (K)
- net row0: now also D0.1 (K), D1.1 (K), D10.1 (K), D11.1 (K), D12.1 (K), D13.1 (K), D14.1 (K), D15.1 (K), D16.1 (K), D17.1 (K), D2.1 (K), D3.1 (K), D4.1 (K), D5.1 (K), D6.1 (K), D7.1 (K), D8.1 (K), D9.1 (K)
- net row1: now also D18.1 (K), D19.1 (K), D20.1 (K), D21.1 (K), D22.1 (K), D23.1 (K), D24.1 (K), D25.1 (K), D26.1 (K), D27.1 (K), D28.1 (K), D29.1 (K), D30.1 (K), D31.1 (K), D32.1 (K), D33.1 (K), D34.1 (K), D35.1 (K); no longer D0.1 (K), D1.1 (K), D10.1 (K), D11.1 (K), D12.1 (K), D13.1 (K), D14.1 (K), D15.1 (K), D16.1 (K), D17.1 (K), D2.1 (K), D3.1 (K), D4.1 (K), D5.1 (K), D6.1 (K), D7.1 (K), D8.1 (K), D9.1 (K)
- net row2: now also D36.1 (K), D37.1 (K), D38.1 (K), D39.1 (K), D40.1 (K), D41.1 (K), D42.1 (K), D43.1 (K), D44.1 (K), D45.1 (K), D46.1 (K), D47.1 (K), D48.1 (K), D49.1 (K), D50.1 (K), D51.1 (K), D52.1 (K), D53.1 (K); no longer D18.1 (K), D19.1 (K), D20.1 (K), D21.1 (K), D22.1 (K), D23.1 (K), D24.1 (K), D25.1 (K), D26.1 (K), D27.1 (K), D28.1 (K), D29.1 (K), D30.1 (K), D31.1 (K), D32.1 (K), D33.1 (K), D34.1 (K), D35.1 (K)
- net row3: now also D54.1 (K), D55.1 (K), D56.1 (K), D57.1 (K), D58.1 (K), D59.1 (K), D60.1 (K), D61.1 (K), D62.1 (K), D63.1 (K), D64.1 (K), D65.1 (K), D66.1 (K), D67.1 (K), D68.1 (K), D69.1 (K), D70.1 (K), D71.1 (K); no longer D36.1 (K), D37.1 (K), D38.1 (K), D39.1 (K), D40.1 (K), D41.1 (K), D42.1 (K), D43.1 (K), D44.1 (K), D45.1 (K), D46.1 (K), D47.1 (K), D48.1 (K), D49.1 (K), D50.1 (K), D51.1 (K), D52.1 (K), D53.1 (K)
- net row4: now also D72.1 (K), D73.1 (K), D74.1 (K), D75.1 (K), D76.1 (K), D77.1 (K), D78.1 (K), D79.1 (K), D80.1 (K), D81.1 (K), D82.1 (K), D83.1 (K), D84.1 (K), D85.1 (K), D86.1 (K), D87.1 (K), D88.1 (K), D89.1 (K); no longer D54.1 (K), D55.1 (K), D56.1 (K), D57.1 (K), D58.1 (K), D59.1 (K), D60.1 (K), D61.1 (K), D62.1 (K), D63.1 (K), D64.1 (K), D65.1 (K), D66.1 (K), D67.1 (K), D68.1 (K), D69.1 (K), D70.1 (K), D71.1 (K)
- net row5: no longer D72.1 (K), D73.1 (K), D74.1 (K), D75.1 (K), D76.1 (K), D77.1 (K), D78.1 (K), D79.1 (K), D80.1 (K), D81.1 (K), D82.1 (K), D83.1 (K), D84.1 (K), D85.1 (K), D86.1 (K), D87.1 (K), D88.1 (K), D89.1 (K)
Other:
- moved on the sheet: D103, D104, D105, D106, D14, D15, D16, D17, D32, D33, D34, D35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
