File: Current/TwoTailed/Daughtercard/Daughtercard.kicad_pcb (KiCad board)
At the start: 2 copper layers, 103.2 x 19 mm, 7 parts, among them J1 Conn_02x05_Odd_Even, SW1 SW_SPDT, SW2 SW_SPDT, SW3 SW_SPDT, SW4 SW_SPDT, SW5 SW_SPDT

Commit message: So much stuff
Wow it's been a while.
Parts:
- removed G***: LOGO, EDI:sweethaz
- added C1: 100nF, EDI:Passive_0402_1005Metric, B.Cu at (72.2, 139.8)
- added DT1: 1N4148W-T4, EDI:D_SOD-523, B.Cu at (100.0, 135.0)
- added DT10: 1N4148W-T4, EDI:D_SOD-523, B.Cu at (271.5, 135.0)
- added DT11: 1N4148W-T4, EDI:D_SOD-523, B.Cu at (290.5, 135.0)
- added DT12: 1N4148W-T4, EDI:D_SOD-523, B.Cu at (309.6, 135.0)
- added DT13: 1N4148W-T4, EDI:D_SOD-523, B.Cu at (328.6, 135.0)
- added DT14: 1N4148W-T4, EDI:D_SOD-523, B.Cu at (347.7, 135.0)
- added DT15: 1N4148W-T4, EDI:D_SOD-523, B.Cu at (366.7, 135.0)
- added DT16: 1N4148W-T4, EDI:D_SOD-523, B.Cu at (385.8, 135.0)
- added DT2: 1N4148W-T4, EDI:D_SOD-523, B.Cu at (119.1, 135.0)
- added DT3: 1N4148W-T4, EDI:D_SOD-523, B.Cu at (138.1, 135.0)
- added DT4: 1N4148W-T4, EDI:D_SOD-523, B.Cu at (157.2, 135.0)
- added DT5: 1N4148W-T4, EDI:D_SOD-523, B.Cu at (176.2, 135.0)
- added DT6: 1N4148W-T4, EDI:D_SOD-523, B.Cu at (195.3, 135.0)
- added DT7: 1N4148W-T4, EDI:D_SOD-523, B.Cu at (214.3, 135.0)
- added DT8: 1N4148W-T4, EDI:D_SOD-523, B.Cu at (233.4, 135.0)
- added DT9: 1N4148W-T4, EDI:D_SOD-523, B.Cu at (252.4, 135.0)
- added J1.1: qwiic, Connector_JST:JST_SH_SM04B-SRSS-TB_1x04-1MP_P1.00mm_Horizontal, B.Cu at (57.9, 126.2)
- added J2: Display, Connector_PinHeader_2.54mm:PinHeader_1x04_P2.54mm_Vertical, B.Cu at (47.6, 128.8)
- added J3: Matrix Expansion, Connector_JST:JST_PH_S8B-PH-K_1x08_P2.00mm_Horizontal, B.Cu at (42.1, 139.6)
- added R1: 2K2, EDI:Passive_0402_1005Metric, B.Cu at (70.6, 139.8)
- added R2: 2K2, EDI:Passive_0402_1005Metric, B.Cu at (69.1, 139.8)
- added SW10: SW_SPDT, EDI:T8013-Z1BQ, F.Cu at (271.5, 132.6)
- added SW11: SW_SPDT, EDI:T8013-Z1BQ, F.Cu at (290.5, 132.6)
- added SW12: SW_SPDT, EDI:T8013-Z1BQ, F.Cu at (309.6, 132.6)
- added SW13: SW_SPDT, EDI:T8013-Z1BQ, F.Cu at (328.6, 132.6)
- added SW14: SW_SPDT, EDI:T8013-Z1BQ, F.Cu at (347.7, 132.6)
- added SW15: SW_SPDT, EDI:T8013-Z1BQ, F.Cu at (366.7, 132.6)
- added SW16: SW_SPDT, EDI:T8013-Z1BQ, F.Cu at (385.8, 132.6)
- added SW6: SW_SPDT, EDI:T8013-Z1BQ, F.Cu at (195.3, 132.6)
- added SW7: SW_SPDT, EDI:T8013-Z1BQ, F.Cu at (214.3, 132.6)
- added SW8: SW_SPDT, EDI:T8013-Z1BQ, F.Cu at (233.4, 132.6)
- added SW9: SW_SPDT, EDI:T8013-Z1BQ, F.Cu at (252.4, 132.6)
- added U1: MCP23018-E/SO, Package_SO:SOIC-28W_7.5x18.7mm_P1.27mm, B.Cu at (76.2, 132.6)
- added kibuzzard-62BE768D: G***, kibuzzard-62BE768D, B.Cu at (57.9, 132.6)
- J1: value Conn_02x05_Odd_Even -> qwiic; footprint Connector_PinHeader_2.54mm:PinHeader_2x05_P2.54mm_Vertical -> Connector_JST:JST_SH_SM04B-SRSS-TB_1x04-1MP_P1.00mm_Horizontal
- moved J1 159.6 mm to (57.9, 139.0)
- moved SW1 104.6 mm to (100.0, 132.6)
- moved SW5 88.3 mm to (176.2, 132.6)
- moved SW2 76.2 mm to (119.1, 132.6)
- moved SW4 65.0 mm to (157.2, 132.6)
- moved SW3 59.7 mm to (138.1, 132.6)
Connections:
- J1 pad 2: LV1 -> +3V3
- J1 pad 3: GND -> SDA
- J1 pad 4: LV2 -> SCL
- SW1 pad 2: GND -> cX0
- SW1 pad 3: LV1 -> Net-(DT1-Pad2)
- SW2 pad 2: GND -> cX0
- SW2 pad 3: LV2 -> Net-(DT2-Pad2)
- SW3 pad 2: GND -> cX0
- SW3 pad 3: LV3 -> Net-(DT3-Pad2)
- SW4 pad 2: GND -> cX0
- SW4 pad 3: LV4 -> Net-(DT4-Pad2)
- SW5 pad 2: GND -> cX1
- SW5 pad 3: LV5 -> Net-(DT5-Pad2)
Routing:
- net rX3: track 0.00 -> 319.8 mm, vias 0 -> 5
- net cX3: track 0.00 -> 313.4 mm, vias 0 -> 1
- net rX2: track 0.00 -> 300.7 mm, vias 0 -> 5
- net rX1: track 0.00 -> 280.1 mm, vias 0 -> 5
- net rX0: track 0.00 -> 260.5 mm, vias 0 -> 5
- net cX2: track 0.00 -> 236.4 mm, vias 0 -> 1
- net cX1: track 0.00 -> 161.7 mm, vias 0 -> 1
- net LV5: track 90.2 -> 0.00 mm
- net cX0: track 0.00 -> 86.6 mm, vias 0 -> 1
- net LV4: track 71.8 -> 0.00 mm
- net LV3: track 53.4 -> 0.00 mm
- net +3V3: track 0.00 -> 47.7 mm, vias 0 -> 1
- net SCL: track 0.00 -> 44.8 mm, vias 0 -> 1
- net cX7: track 0.00 -> 44.7 mm, vias 0 -> 2
- net cX6: track 0.00 -> 43.7 mm, vias 0 -> 2
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Other:
- board size 103.2 x 19 mm -> 361.9 x 19 mm
- board text added: "C4"
- board text added: "C5"
- board text added: "C6"
- board text added: "C7"
- board text added: "R4"
- board text added: "R5"
- board text added: "R6"
- board text added: "R7"
- board text removed: "Everywhere Defense Industries General-Purpose Toggle Daughterboard Mk1 - For Use With T8013-Z1BQ"
- board text removed: "This Side Towards User For Two-Tailed North Array"
