File: Current/ArrowOfTime/Arrow.kicad_sch (KiCad schematic)
At the start: 74 parts, among them J0 USB, J1 Main Drive, J2 R/T Tuning, J3 Display, J4 GripSwitches, J5 GripAnalog, K1 key, K10 key, K11 key, K12 key, K13 tog, K14 tog, K15 tog, K2 key, K3 key, K4 key, K5 key, K6 key, K7 key, K8 key, K9 key, U0 STM32F103CBT6, U1 LDO-3.3, Y0 DST1610A

Commit message: eat shit and die
Parts:
- removed C1: 4.7uF, EDI:Passive_0402_1005Metric, symbol Device:C_Small
- removed C2, C3, C4, C5, C7, C8: 100nF, EDI:Passive_0402_1005Metric, symbol Device:C_Small
- removed C6: 10uF, EDI:Passive_0402_1005Metric, symbol Device:C_Small
- removed CX0, CX1: 22pf, EDI:Passive_0402_1005Metric, symbol Device:C_Small
- removed D1, D10, D11, D12, D13, D14, D15, D2, D3, D4, D5, D6, D7, D8, D9, DG1, DG10, DG2, DG3, DG4, DG5, DG6, DG7, DG8, DG9: 1N4148, EDI:D_SOD-523, symbol Device:D_Small
- removed F0: 6v 500ma, Fuse:Fuse_0603_1608Metric_Castellated, symbol Device:Polyfuse_Small
- removed H1, H2, H3, H4: Mount, MountingHole:MountingHole_3.2mm_M3_DIN965_Pad, symbol Mechanical:MountingHole_Pad
- removed J0: USB, Connector_USB:USB_C_Receptacle_HRO_TYPE-C-31-M-12, symbol HL-Mk2-rescue:USB_C_Receptacle_USB2.0-Connector
- removed J1: Main Drive, Connector_PinSocket_2.54mm:PinSocket_1x03_P2.54mm_Vertical, symbol Connector_Generic:Conn_01x03
- removed J2: R/T Tuning, Connector_PinSocket_2.54mm:PinSocket_1x03_P2.54mm_Vertical, symbol Connector_Generic:Conn_01x03
- removed J3: Display, Connector_PinHeader_2.54mm:PinHeader_1x04_P2.54mm_Vertical, symbol Connector_Generic:Conn_01x04
- removed J4: GripSwitches, Connector_PinSocket_2.54mm:PinSocket_2x10_P2.54mm_Vertical, symbol Connector_Generic:Conn_02x10_Odd_Even
- removed J5: GripAnalog, Connector_PinSocket_2.54mm:PinSocket_2x05_P2.54mm_Vertical, symbol Connector_Generic:Conn_02x05_Odd_Even
- removed K1, K10, K11, K12, K2, K3, K4, K5, K6, K7, K8, K9: key, EDI:SW_MX, symbol HL-Mk2-rescue:KEYSW-keyboard_parts
- removed K13, K14, K15: tog, Connector_PinSocket_2.54mm:PinSocket_1x02_P2.54mm_Vertical, symbol HL-Mk2-rescue:KEYSW-keyboard_parts
- removed R1: 10k, EDI:Passive_0402_1005Metric, symbol Device:R_Small
- removed R2, R3: 5k1, EDI:Passive_0402_1005Metric, symbol Device:R_Small
- removed R4, R5: 2k2, EDI:Passive_0402_1005Metric, symbol Device:R_Small
- removed S1: RESET, Button_Switch_SMD:SW_SPST_SKQG_WithoutStem, symbol Switch:SW_SPST
- removed S2: LDR, Button_Switch_SMD:SW_SPST_SKQG_WithoutStem, symbol Switch:SW_SPST
- removed TX0, TX1: Speaker_Crystal, Buzzer_Beeper:Buzzer_CUI_CPT-9019S-SMT, symbol Device:Speaker_Crystal
- removed U0: STM32F103CBT6, Package_QFP:LQFP-48_7x7mm_P0.5mm, symbol MCU_ST_STM32F1:STM32F103CBTx
- removed U1: LDO-3.3, Package_TO_SOT_SMD:SOT-23, symbol Regulator_Linear:LD1117S33TR_SOT223
- removed Y0: DST1610A, Crystal:Crystal_SMD_2012-2Pin_2.0x1.2mm, symbol Device:Crystal_Small
- added C? (x9), CF?: 100nF, EDI:Passive_0402_1005Metric, symbol Device:C_Small
- added C? (x2), CP? (x2): 1uf, EDI:Passive_0402_1005Metric, symbol Device:C_Small
- added CX? (x2): 13pf, EDI:Passive_0402_1005Metric, symbol Device:C_Small
- added F?: 6v 500ma, Fuse:Fuse_0603_1608Metric, symbol Device:Polyfuse_Small
- added H? (x8): Mount, MountingHole:MountingHole_2.2mm_M2_ISO7380_Pad, symbol Mechanical:MountingHole_Pad
- added J?: qwiic, Connector_JST:JST_SH_SM04B-SRSS-TB_1x04-1MP_P1.00mm_Horizontal, symbol Connector_Generic:Conn_01x05
- added J?: USB, Connector_USB:USB_C_Receptacle_HRO_TYPE-C-31-M-12, symbol HL-Mk2-rescue:USB_C_Receptacle_USB2.0-Connector
- added RC? (x2): 5k1, EDI:Passive_0402_1005Metric, symbol Device:R_Small
- added RD? (x2): 27.4, EDI:Passive_0402_1005Metric, symbol Device:R_Small
- added RF? (x2), RR?, RX?: 1k, EDI:Passive_0402_1005Metric, symbol Device:R_Small
- added S?: USB BOOT, Button_Switch_SMD:SW_SPST_SKQG_WithoutStem, symbol Switch:SW_SPST
- added S?: RESET, Button_Switch_SMD:SW_SPST_SKQG_WithoutStem, symbol Switch:SW_SPST
- added TX? (x2): Transducer, Buzzer_Beeper:Buzzer_CUI_CPT-9019S-SMT, symbol Device:Speaker_Crystal
- added U?: LDO-3.3, Package_TO_SOT_SMD:SOT-23, symbol Regulator_Linear:LD1117S33TR_SOT223
- added U?: USBLC6-2SC6, Package_TO_SOT_SMD:SOT-23-6, symbol Power_Protection:USBLC6-2SC6
- added U?: RP2040, Package_DFN_QFN:QFN-56-1EP_7x7mm_P0.4mm_EP5.6x5.6mm_ThermalVias, symbol RP2040:RP2040
- added U?: W25Q128JVS, Package_SON:WSON-8-1EP_6x5mm_P1.27mm_EP3.4x4.3mm, symbol Memory_Flash:W25Q32JVZP
- added Y?: 12MHz, Crystal:Crystal_SMD_2520-4Pin_2.5x2.0mm, symbol Device:Crystal_GND24
Connections:
- net +3V3: now also C?.1, C?.1, C?.1, C?.1, C?.1, C?.1, C?.1, C?.1, CF?.1, CP?.1, J?.2 (Pin_2), RF?.1, RR?.1, U?.1 (IOVDD), U?.10 (IOVDD), U?.2 (VO), U?.22 (IOVDD), U?.33 (IOVDD), U?.42 (IOVDD), U?.43 (ADC_AVDD), U?.44 (VREG_VIN), U?.48 (USB_VDD), U?.49 (IOVDD), U?.8 (VCC)
- net D+: now also J?.A6 (D+), J?.B6 (D+), U?.6 (I/O1)
- net D-: now also J?.A7 (D-), J?.B7 (D-), U?.4 (I/O2)
- net GND: now also C?.2, C?.2, C?.2, C?.2, C?.2, C?.2, C?.2, C?.2, C?.2, C?.2, C?.2, CF?.2, CP?.1, CP?.2, CX?.1, CX?.2, H?.1, H?.1, H?.1, H?.1, H?.1, H?.1, H?.1, H?.1, J?.1 (Pin_1), J?.A1 (GND), J?.A12 (GND), J?.B1 (GND), J?.B12 (GND), J?.MP, J?.S1 (SHIELD), RC?.1, RC?.2, S?.1 (A), S?.1 (A), TX?.2, TX?.2, U?.1 (GND), U?.19 (TESTEN), U?.2 (GND), U?.4 (GND), U?.57 (GND), U?.9 (EP), Y?.2, Y?.4
- net VBUS: now also CP?.2, F?.2, U?.3 (VI), U?.5 (VBUS)
- new net: RF?.2, S?.2 (B)
- new net: J?.A5 (CC1), RC?.1
- new net: J?.B5 (CC2), RC?.2
- new net +1V1: C?.1, C?.1, C?.1, U?.23 (DVDD), U?.45 (VREG_VOUT), U?.50 (DVDD)
- new net 0: U?.2 (GPIO0)
- new net 1: U?.3 (GPIO1)
- new net 10: U?.13 (GPIO10)
- new net 11: U?.14 (GPIO11)
- new net 12: U?.15 (GPIO12)
- new net 13: U?.16 (GPIO13)
- new net 14: U?.17 (GPIO14)
- new net 15: U?.18 (GPIO15)
- new net 16: TX?.1, U?.27 (GPIO16)
- new net 17: TX?.1, U?.28 (GPIO17)
- new net 18: U?.29 (GPIO18)
- new net 19: U?.30 (GPIO19)
- new net 2: U?.4 (GPIO2)
- new net 20: U?.31 (GPIO20)
- new net 21: U?.32 (GPIO21)
- new net 22: U?.34 (GPIO22)
- new net 23: U?.35 (GPIO23)
- new net 24: U?.36 (GPIO24)
- new net 25: U?.37 (GPIO25)
- new net 26/A0: U?.38 (GPIO26/ADC0)
- new net 27/A1: U?.39 (GPIO27/ADC1)
- new net 28/A2: J?.3 (Pin_3), U?.40 (GPIO28/ADC2)
- new net 29/A3: J?.4 (Pin_4), U?.41 (GPIO29/ADC3)
- new net 3: U?.5 (GPIO3)
- new net 4: U?.6 (GPIO4)
- new net 5: U?.7 (GPIO5)
- new net 6: U?.8 (GPIO6)
- new net 7: U?.9 (GPIO7)
- new net 8: U?.11 (GPIO8)
- new net 9: U?.12 (GPIO9)
- new net CLOCK: U?.52 (QSPI_SCLK), U?.6 (CLK)
- new net CS: RF?.1, RF?.2, U?.1 (~{CS}), U?.56 (QSPI_SS_N)
- new net DB+: RD?.1, U?.1 (I/O1)
- new net DB-: RD?.1, U?.3 (I/O2)
- new net DR+: RD?.2, U?.47 (USB_DP)
- new net DR-: RD?.2, U?.46 (USB_DM)
- new net SD0: U?.5 (DI(IO0)), U?.53 (QSPI_SD0)
- new net SD1: U?.2 (DO(IO1)), U?.55 (QSPI_SD1)
- new net SD2: U?.3 (IO2), U?.54 (QSPI_SD2)
- new net SD3: U?.51 (QSPI_SD3), U?.7 (IO3)
- new net XIN: CX?.2, U?.20 (XIN), Y?.1
- new net XOUT: RX?.1, U?.21 (XOUT)
- new net XOUT1: CX?.1, RX?.2, Y?.3
- new net vUSB: F?.1, J?.A4 (VBUS), J?.A9 (VBUS), J?.B4 (VBUS), J?.B9 (VBUS)
- new net ~{RESET}: RR?.2, S?.2 (B), U?.26 (RUN)
- no-connect marks 2 -> 4
Other:
- note added: "Audio Feedback System"
- note added: "C1 near Pin44"
- note added: "C11 near Pin45"
- note added: "Chassis Ground Mount Points"
- note added: "Clock Reference"
- note added: "ESD Isolator"
- note added: "External Interface System"
- note added: "Flash (128MB)"
- note added: "GPIO Interface Map"
- note added: "Microcontroller Core"
- note added: "Microcontroller Power Regulation"
- note added: "Power Control System"
- note added: "USB port"
- note added: "qwiic Modular Interface"

Commit message: Arrow of Time changes, updates to Sweet Business Six
Parts:
- removed CX? (x2): 13pf, EDI:Passive_0402_1005Metric, symbol Device:C_Small
- removed H? (x4): Mount, MountingHole:MountingHole_2.2mm_M2_ISO7380_Pad, symbol Mechanical:MountingHole_Pad
- removed RX?: 1k, EDI:Passive_0402_1005Metric, symbol Device:R_Small
- removed S?: USB BOOT, Button_Switch_SMD:SW_SPST_SKQG_WithoutStem, symbol Switch:SW_SPST
- removed Y?: 12MHz, Crystal:Crystal_SMD_2520-4Pin_2.5x2.0mm, symbol Device:Crystal_GND24
- added RX0: 1k, EDI:Passive_0402_1005Metric, symbol Device:R_Small
- added Y0: CSTCE12M0G55-R0, Crystal:Resonator_SMD_Murata_CSTxExxV-3Pin_3.0x1.1mm, symbol Device:Crystal_GND2_Small
- gave numbers to parts that had none: 35
Connections:
- net 16: no longer TX1.1
- net 17: no longer TX0.1
- net 28/A2: no longer J0.3 (Pin_3)
- net 29/A3: no longer J0.4 (Pin_4)
- net GND: now also RF1.2, Y0.2
- net XIN: now also Y0.1
- net XOUT: now also RX0.1
- new net: RX0.2, Y0.3
- new net AUDIO+: TX0.1
- new net AUDIO-: TX1.1
- new net SCL: J0.4 (Pin_4)
- new net SDA: J0.3 (Pin_3)
Other:
- added sheet Interface (interface.kicad_sch)
- moved on the sheet: H1, H2, H3, H4
