File: Current/ArrowOfTime/Arrow.kicad_pcb (KiCad board)
At the start: 2 copper layers, 100 x 100 mm, 74 parts, among them J0 USB, J1 Main Drive, J2 R/T Tuning, J3 Display, J4 GripSwitches, J5 GripAnalog, K1 key, K10 key, K11 key, K12 key, K13 tog, K14 tog, K15 tog, K2 key, K3 key, K4 key, K5 key, K6 key, K7 key, K8 key, K9 key, U0 STM32F103CBT6, U1 LDO-3.3, Y0 DST1610A

Commit message: Arrow of Time changes, updates to Sweet Business Six
Parts:
- removed CX0, CX1: 22pf, EDI:Passive_0402_1005Metric
- removed DG1, DG10, DG2, DG3, DG4, DG5, DG6, DG7, DG8, DG9: 1N4148, EDI:D_SOD-523
- removed J5: GripAnalog, Connector_PinSocket_2.54mm:PinSocket_2x05_P2.54mm_Vertical
- removed R1: 10k, EDI:Passive_0402_1005Metric
- removed R2, R3: 5k1, EDI:Passive_0402_1005Metric
- removed R4, R5: 2k2, EDI:Passive_0402_1005Metric
- removed S2: LDR, Button_Switch_SMD:SW_SPST_SKQG_WithoutStem
- added C0: 1uf, EDI:Passive_0402_1005Metric, F.Cu at (-119.9, 89.7)
- added C10: 1uf, EDI:Passive_0402_1005Metric, F.Cu at (-122.4, 94.3)
- added C9: 100nF, EDI:Passive_0402_1005Metric, F.Cu at (-119.9, 85.7)
- added CF0: 100nF, EDI:Passive_0402_1005Metric, F.Cu at (-119.5, 91.7)
- added CP0: 1uf, EDI:Passive_0402_1005Metric, F.Cu at (-116.9, 87.7)
- added CP1: 1uf, EDI:Passive_0402_1005Metric, F.Cu at (-114.0, 87.7)
- added D16: SOD523, Diode_SMD:D_SOD-523, F.Cu at (-95.3, 71.6)
- added D17: SOD523, Diode_SMD:D_SOD-523, F.Cu at (-109.5, 71.6)
- added D18: SOD523, Diode_SMD:D_SOD-523, F.Cu at (-113.0, 74.1)
- added D19: SOD523, Diode_SMD:D_SOD-523, F.Cu at (-120.1, 71.6)
- added D20: SOD523, Diode_SMD:D_SOD-523, F.Cu at (-116.6, 74.1)
- added D21: SOD523, Diode_SMD:D_SOD-523, F.Cu at (-123.7, 79.0)
- added D22: SOD523, Diode_SMD:D_SOD-523, F.Cu at (-123.7, 71.6)
- added D23: SOD523, Diode_SMD:D_SOD-523, F.Cu at (-109.5, 74.1)
- added D24: SOD523, Diode_SMD:D_SOD-523, F.Cu at (-116.6, 76.5)
- added D25: SOD523, Diode_SMD:D_SOD-523, F.Cu at (-120.1, 79.0)
- added D26: SOD523, Diode_SMD:D_SOD-523, F.Cu at (-120.1, 74.1)
- added D27: SOD523, Diode_SMD:D_SOD-523, F.Cu at (-105.9, 74.1)
- added D28: SOD523, Diode_SMD:D_SOD-523, F.Cu at (-123.7, 76.5)
- added D29: SOD523, Diode_SMD:D_SOD-523, F.Cu at (-123.7, 74.1)
- added D30: SOD523, Diode_SMD:D_SOD-523, F.Cu at (-127.2, 74.1)
- added D31: SOD523, Diode_SMD:D_SOD-523, F.Cu at (-127.2, 79.0)
- added D32: SOD523, Diode_SMD:D_SOD-523, F.Cu at (-98.8, 71.6)
- added D33: SOD523, Diode_SMD:D_SOD-523, F.Cu at (-116.6, 71.6)
- added D34: SOD523, Diode_SMD:D_SOD-523, F.Cu at (-102.4, 71.6)
- added D35: SOD523, Diode_SMD:D_SOD-523, F.Cu at (-98.8, 74.1)
- added D36: SOD523, Diode_SMD:D_SOD-523, F.Cu at (-113.0, 71.6)
- added DT1: SOD523, Diode_SMD:D_SOD-523, F.Cu at (-127.2, 76.5)
- added DT2: SOD523, Diode_SMD:D_SOD-523, F.Cu at (-120.1, 76.5)
- added DT3: SOD523, Diode_SMD:D_SOD-523, F.Cu at (-127.2, 71.6)
- added DT4: SOD523, Diode_SMD:D_SOD-523, F.Cu at (-102.4, 74.1)
- added DT5: SOD523, Diode_SMD:D_SOD-523, F.Cu at (-116.6, 79.0)
- added DT6: SOD523, Diode_SMD:D_SOD-523, F.Cu at (-105.9, 71.6)
- added K16: Keyswitch, EDI:SW_MX, F.Cu at (181.1, 58.7)
- added K17: Keyswitch, EDI:SW_MX, F.Cu at (196.2, 58.7)
- added K18: Keyswitch, EDI:SW_MX, F.Cu at (226.4, 58.7)
- added K19: Keyswitch, EDI:SW_MX, F.Cu at (120.8, 88.9)
- added K20: Keyswitch, EDI:SW_MX, F.Cu at (135.9, 88.9)
- added K21: Keyswitch, EDI:SW_MX, F.Cu at (166.1, 88.9)
- added K22: Keyswitch, EDI:SW_MX, F.Cu at (181.1, 88.9)
- added K23: Keyswitch, EDI:SW_MX, F.Cu at (196.2, 88.9)
- added K24: Keyswitch, EDI:SW_MX, F.Cu at (226.4, 88.1)
- added K25: Keyswitch, EDI:SW_MX, F.Cu at (120.8, 104.0)
- added K26: Keyswitch, EDI:SW_MX, F.Cu at (135.9, 104.0)
- added K27: Keyswitch, EDI:SW_MX, F.Cu at (166.1, 104.0)
- added K28: Keyswitch, EDI:SW_MX, F.Cu at (181.1, 104.0)
- added K29: Keyswitch, EDI:SW_MX, F.Cu at (196.2, 104.0)
- added K30: Keyswitch, EDI:SW_MX, F.Cu at (226.4, 103.2)
- added K31: Keyswitch, EDI:SW_MX, F.Cu at (120.8, 134.1)
- added K32: Keyswitch, EDI:SW_MX, F.Cu at (135.9, 134.1)
- added K33: Keyswitch, EDI:SW_MX, F.Cu at (151.0, 134.1)
- added K34: Keyswitch, EDI:SW_MX, F.Cu at (166.0, 134.1)
- added K35: Keyswitch, EDI:SW_MX, F.Cu at (181.1, 134.1)
- added K36: Keyswitch, EDI:SW_MX, F.Cu at (196.2, 134.1)
- added LC1: 100nF, EDI:Passive_0402_1005Metric, F.Cu at (-75.2, 76.5)
- added LC10: 100nF, EDI:Passive_0402_1005Metric, F.Cu at (-81.4, 80.7)
- added LC11: 100nF, EDI:Passive_0402_1005Metric, F.Cu at (-88.6, 71.4)
- added LC12: 100nF, EDI:Passive_0402_1005Metric, F.Cu at (-75.6, 80.5)
- added LC13: 100nF, EDI:Passive_0402_1005Metric, F.Cu at (-65.9, 71.4)
- added LC14: 100nF, EDI:Passive_0402_1005Metric, F.Cu at (-78.5, 80.5)
- added LC15: 100nF, EDI:Passive_0402_1005Metric, F.Cu at (-93.1, 80.1)
- added LC16: 100nF, EDI:Passive_0402_1005Metric, F.Cu at (-71.7, 73.4)
- added LC17: 100nF, EDI:Passive_0402_1005Metric, F.Cu at (-8.55, 9.91)
- added LC18: 100nF, EDI:Passive_0402_1005Metric, F.Cu at (-92.1, 74.5)
- added LC19: 100nF, EDI:Passive_0402_1005Metric, F.Cu at (-49.0, 55.3)
- added LC2: 100nF, EDI:Passive_0402_1005Metric, F.Cu at (-72.3, 75.4)
- added LC20: 100nF, EDI:Passive_0402_1005Metric, F.Cu at (-96.0, 80.7)
- added LC21: 100nF, EDI:Passive_0402_1005Metric, F.Cu at (-87.3, 80.7)
- added LC22: 100nF, EDI:Passive_0402_1005Metric, F.Cu at (-75.2, 74.5)
- added LC23: 100nF, EDI:Passive_0402_1005Metric, F.Cu at (-51.9, 57.3)
- added LC24: 100nF, EDI:Passive_0402_1005Metric, F.Cu at (-35.7, 39.1)
- added LC25: 100nF, EDI:Passive_0402_1005Metric, F.Cu at (-84.4, 80.7)
- added LC26: 100nF, EDI:Passive_0402_1005Metric, F.Cu at (-62.9, 69.4)
- added LC27: 100nF, EDI:Passive_0402_1005Metric, F.Cu at (-8.55, 11.9)
- added LC28: 100nF, EDI:Passive_0402_1005Metric, F.Cu at (-75.7, 78.5)
- added LC3: 100nF, EDI:Passive_0402_1005Metric, F.Cu at (-68.8, 71.4)
- added LC4: 100nF, EDI:Passive_0402_1005Metric, F.Cu at (-71.7, 71.4)
- added LC5: 100nF, EDI:Passive_0402_1005Metric, F.Cu at (-72.3, 77.4)
- added LC6: 100nF, EDI:Passive_0402_1005Metric, F.Cu at (-90.2, 80.7)
- added LC7: 100nF, EDI:Passive_0402_1005Metric, F.Cu at (-51.9, 55.3)
- added LC8: 100nF, EDI:Passive_0402_1005Metric, F.Cu at (-68.8, 73.4)
- added LC9: 100nF, EDI:Passive_0402_1005Metric, F.Cu at (-78.6, 77.6)
- added LD1: WS2812C, EDI:WS2812C_2020, F.Cu at (-78.4, 72.0)
- added LD10: WS2812C, EDI:WS2812C_2020, F.Cu at (-91.8, 72.0)
- added LD11: WS2812C, EDI:WS2812C_2020, F.Cu at (-95.7, 77.5)
- added LD12: WS2812C, EDI:WS2812C_2020, F.Cu at (-85.3, 78.2)
- added LD13: WS2812C, EDI:WS2812C_2020, F.Cu at (-106.1, 80.0)
- added LD14: WS2812C, EDI:WS2812C_2020, F.Cu at (-102.7, 80.0)
- added LD15: WS2812C, EDI:WS2812C_2020, F.Cu at (-81.8, 78.2)
- added LD16: WS2812C, EDI:WS2812C_2020, F.Cu at (-113.1, 80.0)
- added LD17: WS2812C, EDI:WS2812C_2020, F.Cu at (-109.6, 80.0)
- added LD18: WS2812C, EDI:WS2812C_2020, F.Cu at (-85.3, 72.0)
- added LD19: WS2812C, EDI:WS2812C_2020, F.Cu at (-88.8, 78.2)
- added LD2: WS2812C, EDI:WS2812C_2020, F.Cu at (-81.8, 75.1)
- added LD20: WS2812C, EDI:WS2812C_2020, F.Cu at (-74.9, 72.0)
- added LD21: WS2812C, EDI:WS2812C_2020, F.Cu at (-81.8, 72.0)
- added LD22: WS2812C, EDI:WS2812C_2020, F.Cu at (-30.4, 35.6)
- added LD23: WS2812C, EDI:WS2812C_2020, F.Cu at (-8.26, 7.37)
- added LD24: WS2812C, EDI:WS2812C_2020, F.Cu at (-102.7, 76.9)
- added LD25: WS2812C, EDI:WS2812C_2020, F.Cu at (-78.4, 75.1)
- added LD26: WS2812C, EDI:WS2812C_2020, F.Cu at (-88.8, 75.1)
- added LD27: WS2812C, EDI:WS2812C_2020, F.Cu at (-85.3, 75.1)
- added LD28: WS2812C, EDI:WS2812C_2020, F.Cu at (-4.79, 7.37)
- added LD3: WS2812C, EDI:WS2812C_2020, F.Cu at (-99.2, 76.9)
- added LD4: WS2812C, EDI:WS2812C_2020, F.Cu at (-92.2, 77.5)
- added LD5: WS2812C, EDI:WS2812C_2020, F.Cu at (-106.1, 76.9)
- added LD6: WS2812C, EDI:WS2812C_2020, F.Cu at (-95.3, 74.4)
- added LD7: WS2812C, EDI:WS2812C_2020, F.Cu at (-113.1, 76.9)
- added LD8: WS2812C, EDI:WS2812C_2020, F.Cu at (-99.2, 80.0)
- added LD9: WS2812C, EDI:WS2812C_2020, F.Cu at (-109.6, 76.9)
- added RC0: 5k1, EDI:Passive_0402_1005Metric, F.Cu at (-116.9, 85.7)
- added RC1: 5k1, EDI:Passive_0402_1005Metric, F.Cu at (-111.1, 85.7)
- added RD0: 27.4, EDI:Passive_0402_1005Metric, F.Cu at (-122.4, 92.3)
- added RD1: 27.4, EDI:Passive_0402_1005Metric, F.Cu at (-116.9, 89.7)
- added RF0: 1k, EDI:Passive_0402_1005Metric, F.Cu at (-119.5, 93.7)
- added RF1: 1k, EDI:Passive_0402_1005Metric, F.Cu at (-116.6, 91.7)
- added RR0: 1k, EDI:Passive_0402_1005Metric, F.Cu at (-119.9, 87.7)
- added RX0: 1k, EDI:Passive_0402_1005Metric, F.Cu at (-114.0, 85.7)
- added T1: Keyswitch, EDI:KeyToggle, F.Cu at (254.0, 25.4)
- added T2: Keyswitch, EDI:KeyToggle, F.Cu at (254.0, 50.8)
- added T3: Keyswitch, EDI:KeyToggle, F.Cu at (254.0, 76.2)
- added T4: Keyswitch, EDI:KeyToggle, F.Cu at (254.0, 101.6)
- added T5: Keyswitch, EDI:KeyToggle, F.Cu at (254.0, 127.0)
- added T6: Keyswitch, EDI:KeyToggle, F.Cu at (254.0, 152.4)
- added U2: W25Q128JVS, Package_SON:WSON-8-1EP_6x5mm_P1.27mm_EP3.4x4.3mm, F.Cu at (-125.2, 88.0)
- added U3: USBLC6-2SC6, Package_TO_SOT_SMD:SOT-23-6, F.Cu at (-126.4, 93.5)
- C1: value 4.7uF -> 100nF
- C6: value 10uF -> 100nF
- D1, D10, D11, D12, D13, D14, D15, D2, D3, D4, D5, D6, D7, D8, D9: value 1N4148 -> SOD523; footprint EDI:D_SOD-523 -> Diode_SMD:D_SOD-523
- F0: footprint Fuse:Fuse_0603_1608Metric_Castellated -> Fuse:Fuse_0603_1608Metric
- H1, H2, H3, H4: footprint MountingHole:MountingHole_3.2mm_M3_DIN965_Pad -> MountingHole:MountingHole_2.2mm_M2_ISO7380_Pad
- J0: value USB -> qwiic; footprint Connector_USB:USB_C_Receptacle_HRO_TYPE-C-31-M-12 -> Connector_JST:JST_SH_SM04B-SRSS-TB_1x04-1MP_P1.00mm_Horizontal
- J1: value Main Drive -> Z Main Drive; footprint Connector_PinSocket_2.54mm:PinSocket_1x03_P2.54mm_Vertical -> Connector_JST:JST_SH_SM03B-SRSS-TB_1x03-1MP_P1.00mm_Horizontal
- J2: value R/T Tuning -> X Radiotelescope Tuner; footprint Connector_PinSocket_2.54mm:PinSocket_1x03_P2.54mm_Vertical -> Potentiometer_THT:Potentiometer_Bourns_PTV09A-1_Single_Vertical
- J3: value Display -> Y DRADIS range; footprint Connector_PinHeader_2.54mm:PinHeader_1x04_P2.54mm_Vertical -> Potentiometer_THT:Potentiometer_Bourns_PTA4543_Single_Slide
- J4: value GripSwitches -> USB; footprint Connector_PinSocket_2.54mm:PinSocket_2x10_P2.54mm_Vertical -> Connector_USB:USB_C_Receptacle_HRO_TYPE-C-31-M-12
- K1, K10, K11, K12, K2, K3, K4, K5, K6, K7, K8, K9: value key -> Keyswitch
- K13, K14, K15: value tog -> Keyswitch; footprint Connector_PinSocket_2.54mm:PinSocket_1x02_P2.54mm_Vertical -> EDI:SW_MX; moved to F.Cu
- TX0, TX1: value Speaker_Crystal -> Transducer
- U0: value STM32F103CBT6 -> RP2040; footprint Package_QFP:LQFP-48_7x7mm_P0.5mm -> EDI:RP2040
- Y0: value DST1610A -> CSTCE12M0G55-R0; footprint Crystal:Crystal_SMD_2012-2Pin_2.0x1.2mm -> Crystal:Resonator_SMD_Murata_CSTxExxV-3Pin_3.0x1.1mm
- moved C1 218.2 mm to (-156.3, 80.3)
- moved C2 218.2 mm to (-147.6, 71.6)
- moved C4 218.2 mm to (-157.9, 66.8)
- moved C5 218.2 mm to (-161.1, 77.6)
- moved C8 218.2 mm to (-148.4, 87.5)
- moved TX0 218.2 mm to (-152.3, 35.1)
- moved TX1 218.2 mm to (-152.3, 45.4)
- moved U0 218.2 mm to (-154.7, 73.2)
- moved Y0 218.2 mm to (-161.1, 81.2)
- moved C3 218.2 mm to (-152.6, 80.3)
- moved S1 218.2 mm to (-154.1, 89.6)
- moved Z0 212.6 mm to (-155.5, 106.5)
- moved J2 201.7 mm to (228.7, 128.1)
- moved J0 151.2 mm to (-27.0, 75.4)
- moved C6 142.0 mm to (-26.2, 61.9)
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Connections:
- C1 pad 1: +3V3 -> +1V1
- C2 pad 1: +3V3 -> +1V1
- C6 pad 1: GND -> +3V3
- C6 pad 2: +3V3 -> GND
- C7 pad 1: GND -> +3V3
- C7 pad 2: VBUS -> GND
- C8 pad 1: NRST -> +3V3
- D1 pad 1: row0 -> Net-(D1-Pad1)
- D10 pad 1: row3 -> Net-(D10-Pad1)
- D11 pad 1: row3 -> Net-(D10-Pad1)
- D12 pad 1: row3 -> Net-(D10-Pad1)
- D13 pad 1: row4 -> Net-(D13-Pad1)
- D14 pad 1: row4 -> Net-(D13-Pad1)
- D15 pad 1: row4 -> Net-(D13-Pad1)
- D2 pad 1: row0 -> Net-(D1-Pad1)
- D3 pad 1: row0 -> Net-(D1-Pad1)
- D4 pad 1: row1 -> Net-(D1-Pad1)
- D5 pad 1: row1 -> Net-(D1-Pad1)
- D6 pad 1: row1 -> Net-(D1-Pad1)
- D7 pad 1: row2 -> Net-(D10-Pad1)
- D8 pad 1: row2 -> Net-(D10-Pad1)
- D9 pad 1: row2 -> Net-(D10-Pad1)
- F0 pad 1: 5v -> vUSB
- J1 pad 1: Z -> unconnected-(J1-Pad1)
- J1 pad 2: +3V3 -> unconnected-(J1-Pad2)
- J1 pad 3: GND -> unconnected-(J1-Pad3)
- J2 pad 1: +3V3 -> unconnected-(J2-Pad1)
- J2 pad 2: rY -> unconnected-(J2-Pad2)
- J2 pad 3: GND -> unconnected-(J2-Pad3)
- J3 pad 1: GND -> unconnected-(J3-Pad1)
- J3 pad 2: +3V3 -> unconnected-(J3-Pad2)
- J3 pad 3: I2C-SDA -> unconnected-(J3-Pad3)
- K1 pad 1: col0 -> Net-(D1-Pad2)
- K1 pad 2: Net-(D1-Pad2) -> Net-(K1-Pad2)
- K10 pad 1: col0 -> Net-(D10-Pad2)
- K10 pad 2: Net-(D10-Pad2) -> Net-(K10-Pad2)
- K11 pad 1: col1 -> Net-(D11-Pad2)
- K11 pad 2: Net-(D11-Pad2) -> Net-(K11-Pad2)
- K12 pad 1: col2 -> Net-(D12-Pad2)
- K12 pad 2: Net-(D12-Pad2) -> Net-(K12-Pad2)
- K13 pad 1: col0 -> Net-(D13-Pad2)
- K13 pad 2: Net-(D13-Pad2) -> Net-(K1-Pad2)
- K14 pad 1: col1 -> Net-(D14-Pad2)
- K14 pad 2: Net-(D14-Pad2) -> Net-(K14-Pad2)
- K15 pad 1: col2 -> Net-(D15-Pad2)
- K15 pad 2: Net-(D15-Pad2) -> Net-(K15-Pad2)
- K2 pad 1: col1 -> Net-(D2-Pad2)
- K2 pad 2: Net-(D2-Pad2) -> Net-(K14-Pad2)
- K3 pad 1: col2 -> Net-(D3-Pad2)
- K3 pad 2: Net-(D3-Pad2) -> Net-(K15-Pad2)
- K4 pad 1: col0 -> Net-(D4-Pad2)
- K4 pad 2: Net-(D4-Pad2) -> Net-(K10-Pad2)
- K5 pad 1: col1 -> Net-(D5-Pad2)
- K5 pad 2: Net-(D5-Pad2) -> Net-(K11-Pad2)
- K6 pad 1: col2 -> Net-(D6-Pad2)
- K6 pad 2: Net-(D6-Pad2) -> Net-(K12-Pad2)
- K7 pad 1: col0 -> Net-(D7-Pad2)
- K7 pad 2: Net-(D7-Pad2) -> Net-(K1-Pad2)
- K8 pad 1: col1 -> Net-(D8-Pad2)
- K8 pad 2: Net-(D8-Pad2) -> Net-(K14-Pad2)
- K9 pad 1: col2 -> Net-(D9-Pad2)
- K9 pad 2: Net-(D9-Pad2) -> Net-(K15-Pad2)
- S1 pad 1: NRST -> GND
- S1 pad 2: GND -> ~{RESET}
- TX0 pad 1: AUDIO0 -> AUDIO+
- TX1 pad 1: AUDIO1 -> AUDIO-
- U0 pad 10: X -> +3V3
- U0 pad 11: Y -> 8
- U0 pad 12: rX -> 9
- U0 pad 13: Z -> 10
- U0 pad 14: AUDIO0 -> 11
- U0 pad 15: AUDIO1 -> 12
- U0 pad 16: rY -> 13
- U0 pad 17: E0A -> 14
- U0 pad 18: E0B -> 15
- U0 pad 19: unconnected-(U0-Pad19) -> GND
- U0 pad 2: unconnected-(U0-Pad2) -> 0
- U0 pad 20: unconnected-(U0-Pad20) -> XIN
- U0 pad 21: unconnected-(U0-Pad21) -> XOUT
- U0 pad 22: unconnected-(U0-Pad22) -> +3V3
- U0 pad 23: GND -> +1V1
- U0 pad 24: +3V3 -> unconnected-(U0-Pad24)
- U0 pad 25: row4 -> unconnected-(U0-Pad25)
- U0 pad 26: row3 -> ~{RESET}
- U0 pad 27: row2 -> 16
- U0 pad 28: row1 -> 17
- U0 pad 29: row0 -> 18
- U0 pad 3: C+ -> 1
- U0 pad 30: unconnected-(U0-Pad30) -> 19
- U0 pad 31: unconnected-(U0-Pad31) -> 20
- U0 pad 32: D- -> 21
- U0 pad 33: D+ -> +3V3
- U0 pad 34: unconnected-(U0-Pad34) -> 22
- U0 pad 35: GND -> 23
- U0 pad 36: +3V3 -> 24
- U0 pad 37: col4 -> 25
- U0 pad 38: col3 -> 26/A0
- U0 pad 39: col2 -> 27/A1
- U0 pad 4: C- -> 2
- U0 pad 40: col1 -> 28/A2
- U0 pad 41: col0 -> 29/A3
- U0 pad 42: unconnected-(U0-Pad42) -> +3V3
- U0 pad 43: I2C-SCL -> +3V3
- U0 pad 44: BOOT0 -> +3V3
- U0 pad 45: I2C-SDA -> +1V1
- U0 pad 46: unconnected-(U0-Pad46) -> DR-
- U0 pad 47: GND -> DR+
- U0 pad 5: unconnected-(U0-Pad5) -> 3
- U0 pad 6: unconnected-(U0-Pad6) -> 4
- U0 pad 7: NRST -> 5
- U0 pad 8: GND -> 6
- U0 pad 9: +3V3 -> 7
- Y0 pad 1: C- -> XIN
- Y0 pad 2: C+ -> GND
Routing:
- net +3V3: track 27.7 -> 0.00 mm
- net GND: track 19.8 -> 0.00 mm, vias 1 -> 0
- net col3: track 18.6 -> 0.00 mm
- net col4: track 18.6 -> 0.00 mm
- net 5v: track 9.76 -> 0.00 mm, vias 2 -> 0
- net NRST: track 8.44 -> 0.00 mm
- net C-: track 8.35 -> 0.00 mm
- net C+: track 8.32 -> 0.00 mm
- net BOOT0: track 8.30 -> 0.00 mm
- net Net-(J4-Pad20): track 5.48 -> 0.00 mm
- net Net-(J4-Pad2): track 5.42 -> 0.00 mm
- net Net-(J4-Pad18): track 4.53 -> 0.00 mm
- net Net-(J4-Pad4): track 4.47 -> 0.00 mm
- net Net-(J4-Pad16): track 3.81 -> 0.00 mm
- net Net-(J4-Pad6): track 3.79 -> 0.00 mm
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- removed copper zone on B.Cu, net GND
- removed copper zone on F.Cu, net GND
Other:
- board size 100 x 100 mm -> 254 x 158.8 mm
- board text added: "Main Drive"
- board text added: "R/T Tuner"
- board text added: "Sensor Range"
- board text removed: "ATK TGT"
- board text removed: "BAY DOOR"
- board text removed: "Boot Loader"
- board text removed: "CGO SCP"
- board text removed: "ENGAGE"
- board text removed: "Everywhere Defense Industries - Systems Integration Group Prototype Development Laboratory - Test Platform Design 227 "Arrow of Time" Pilot Interface System, Throttle Control Bank Module A - Designed 2021 in Pittsburgh, PA, USA, Earth, Sol"
- board text removed: "FTR AGG"
- board text removed: "FTR DEF"
- board text removed: "FULL SPECTRUM TRACK SCANNER"
- board text removed: "GND 3V3 Z"
- board text removed: "GND rY 3v3"
- board text removed: "GXY MAP"
- board text removed: "HOLD FIRE"
- board text removed: "HOLD POS"
- board text removed: "JUMP DRIVE"
- board text removed: "LDG GEAR"
- board text removed: "NAV SYS"
- board text removed: "NEXT SYS"
- board text removed: "POWER"
- board text removed: "PULSE"
- board text removed: "RADIO COMM"
- board text removed: "SILENT"
- board text removed: "SYS MAP"
- board text removed: "System Reset"
- board text removed: "X Hat Enc A Enc B GND GND"
- board text removed: "Y Hat rX 3v3 3v3 GND"

Commit message: Final backup Factory B
Parts:
- moved J2 323.8 mm to (-95.0, 135.4)
Changed lines of the file:
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@@
   )
   (footprint "Potentiometer_THT:Potentiometer_Bourns_PTV09A-1_Single_Vertical" (layer "B.Cu")
-    (at 228.71875 128.09375 -90)
+    (at -95 135.45 -90)
     (descr "Potentiometer, vertical, Bourns PTV09A-1 Single, http://www.bourns.com/docs/Product-Datasheets/ptv09.pdf")
     (tags "Potentiometer vertical Bourns PTV09A-1 Single")
@@
   (gr_line (start -161.234049 92.268875) (end -162.027799 92.268875) (layer "B.SilkS") (width 0.15))
   (gr_line (start 66.173166 129.238795) (end 62.346331 138.477592) (layer "F.SilkS") (width 0.15))
-  (gr_arc (start 62.346331 138.477592) (mid 70 99.999999) (end 77.653669 138.477591) (layer "F.SilkS") (width 0.15))
+  (gr_arc (start 62.346331 138.477592) (mid 69.999998 99.999999) (end 77.653669 138.477591) (layer "F.SilkS") (width 0.15))
   (gr_rect (start 65 20) (end 75 90) (layer "F.SilkS") (width 0.15) (fill none))
   (gr_rect (start 20 20) (end 40 160) (layer "F.SilkS") (width 0.15) (fill none))
   (gr_line (start 73.826834 129.238796) (end 77.653669 138.477591) (layer "F.SilkS") (width 0.15))
-  (gr_arc (start 66.173166 129.238795) (mid 70 110) (end 73.826834 129.238796) (layer "F.SilkS") (width 0.15))
+  (gr_arc (start 66.173166 129.238795) (mid 70.000002 110) (end 73.826834 129.238796) (layer "F.SilkS") (width 0.15))
   (gr_line (start 12.8471 15.0579) (end 12.7 169.06875) (layer "Edge.Cuts") (width 0.15))
   (gr_line (start 200.81875 12.67665) (end 15.22835 12.67665) (layer "Edge.Cuts") (width 0.15))
