File: Current/HardLight2L/HardLight.kicad_pcb (KiCad board)
At the start: 2 copper layers, 304.8 x 76.2 mm, 237 parts, among them J0 USB, J1 qwiic, J2 SPI Connector, K1 Keyswitch, K10 Keyswitch, K11 Keyswitch, K12 Keyswitch, K13 Keyswitch, K14 Keyswitch, K15 Keyswitch, K16 Keyswitch, K17 Keyswitch, K18 Keyswitch, K19 Keyswitch, K2 Keyswitch, K20 Keyswitch, K21 Keyswitch, K22 Keyswitch, K23 Keyswitch, K24 Keyswitch, K25 Keyswitch, K26 Keyswitch, K27 Keyswitch, K28 Keyswitch, K29 Keyswitch, K3 Keyswitch, K30 Keyswitch, K31 Keyswitch, K32 Keyswitch, K33 Keyswitch, K34 Keyswitch, K35 Keyswitch, K36 Keyswitch, K37 Keyswitch, K38 Keyswitch, K39 Keyswitch, K4 Keyswitch, K40 Keyswitch, K41 Keyswitch, K42 Keyswitch, K43 Keyswitch, K44 Keyswitch, K45 Keyswitch, K46 Keyswitch, K47 Keyswitch, K48 Keyswitch, K49 Keyswitch, K5 Keyswitch, K50 Keyswitch, K51 Keyswitch, K52 Keyswitch, K53 Keyswitch, K54 Keyswitch, K54.1 Keyswitch, K55 Keyswitch, K56 Keyswitch, K57 Keyswitch, K58 Keyswitch, K58.1 Keyswitch, K59 Keyswitch, K6 Keyswitch, K60 Keyswitch, K61 Keyswitch, K62 Keyswitch, K63 Keyswitch, K64 Keyswitch, K7 Keyswitch, K8 Keyswitch, K9 Keyswitch, U0 RP2040, U1 LDO-3.3, U2 USBLC6-2SC6, U3 W25Q128JVS, Y0 CSTCE12M0G55-R0

Commit message: oh god there's too much
Parts:
- added J3: LED Expansion, Connector_PinHeader_1.27mm:PinHeader_1x03_P1.27mm_Vertical, F.Cu at (320.7, 108.0)
- TP0: value Pin 22 -> 22
Connections:
- LD32 pad 1: unconnected-(LD32-Pad1) -> Net-(LD32-Pad1)
Routing:
- net VBUS: track 381.6 -> 392.8 mm
- net GND: track 125.9 -> 131.1 mm
- net Net-(LD32-Pad1): track 0.00 -> 4.90 mm
Other:
- board text added: ".5"
- board text added: "GND DATA +5V"
- board text removed: ".3.1"
Changed lines of the file:
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@@
   (net 150 "Net-(LD30-Pad1)")
   (net 151 "Net-(LD31-Pad1)")
-  (net 152 "unconnected-(LD32-Pad1)")
+  (net 152 "Net-(LD32-Pad1)")
   (net 153 "Net-(RX1-Pad2)")
   (footprint "EDI:SW_MX" (layer "F.Cu")
@@
     (pad "" np_thru_hole circle locked (at 0 0 180) (size 3.2 3.2) (drill 3.2) (layers *.Cu *.Mask))
   )
+  (footprint "Connector_PinHeader_1.27mm:PinHeader_1x03_P1.27mm_Vertical" (layer "F.Cu")
+    (at 320.675 107.95)
+    (descr "Through hole straight pin header, 1x03, 1.27mm pitch, single row")
+    (tags "Through hole pin header THT 1x03 1.27mm single row")
+    (property "Sheetfile" "HardLight-Matrix.kicad_sch")
+    (property "Sheetname" "User Interface Element")
+    (attr through_hole)
+    (fp_text reference "J3" (at 0 -1.695) (layer "F.SilkS") hide
+      (effects (font (size 1 1) (thickness 0.15)))
+    )
+    (fp_text value "LED Expansion" (at 0 4.235) (layer "F.Fab")
+      (effects (font (size 1 1) (thickness 0.15)))
+    )
+    (fp_text user "${REFERENCE}" (at 0 1.27 90) (layer "F.Fab")
+      (effects (font (size 1 1) (thickness 0.15)))
+    )
+    (fp_line (start 0.563471 0.76) (end 1.11 0.76) (layer "F.SilkS") (width 0.12))
+    (fp_line (start 0.30753 3.235) (end 1.11 3.235) (layer "F.SilkS") (width 0.12))
+    (fp_line (start -1.11 -0.76) (end 0 -0.76) (layer "F.SilkS") (width 0.12))
+    (fp_line (start -1.11 0) (end -1.11 -0.76) (layer "F.SilkS") (width 0.12))
+    (fp_line (start -1.11 3.235) (end -0.30753 3.235) (layer "F.SilkS") (width 0.12))
+    (fp_line (start -1.11 0.76) (end -0.563471 0.76) (layer "F.SilkS") (width 0.12))
+    (fp_line (start 1.11 0.76) (end 1.11 3.235) (layer "F.SilkS") (width 0.12))
+    (fp_line (start -1.11 0.76) (end -1.11 3.235) (layer "F.SilkS") (width 0.12))
+    (fp_line (start -1.55 -1.15) (end -1.55 3.7) (layer "F.CrtYd") (width 0.05))
+    (fp_line (start 1.55 3.7) (end 1.55 -1.15) (layer "F.CrtYd") (width 0.05))
+    (fp_line (start -1.55 3.7) (end 1.55 3.7) (layer "F.CrtYd") (width 0.05))
+    (fp_line (start 1.55 -1.15) (end -1.55 -1.15) (layer "F.CrtYd") (width 0.05))
+    (fp_line (start -1.05 3.175) (end -1.05 -0.11) (layer "F.Fab") (width 0.1))
+    (fp_line (start -0.525 -0.635) (end 1.05 -0.635) (layer "F.Fab") (width 0.1))
+    (fp_line (start -1.05 -0.11) (end -0.525 -0.635) (layer "F.Fab") (width 0.1))
+    (fp_line (start 1.05 3.175) (end -1.05 3.175) (layer "F.Fab") (width 0.1))
+    (fp_line (start 1.05 -0.635) (end 1.05 3.175) (layer "F.Fab") (width 0.1))
+    (pad "1" thru_hole rect (at 0 0) (size 1 1) (drill 0.65) (layers *.Cu *.Mask)
+      (net 1 "GND") (pinfunction "Pin_1") (pintype "passive"))
+    (pad "2" thru_hole oval (at 0 1.27) (size 1 1) (drill 0.65) (layers *.Cu *.Mask)
+      (net 152 "Net-(LD32-Pad1)") (pinfunction "Pin_2") (pintype "passive"))
+    (pad "3" thru_hole oval (at 0 2.54) (size 1 1) (drill 0.65) (layers *.Cu *.Mask)
+      (net 2 "VBUS") (pinfunction "Pin_3") (pintype "passive"))
+    (model "${KICAD6_3DMODEL_DIR}/Connector_PinHeader_1.27mm.3dshapes/PinHeader_1x03_P1.27mm_Vertical.wrl"
+      (offset (xyz 0 0 0))
+      (scale (xyz 1 1 1))
+      (rotate (xyz 0 0 0))
+    )
+  )
   (footprint "MountingHole:MountingHole_3.2mm_M3" (layer "F.Cu")
     (at 296.06395 128.5794 180)
@@
     (fp_circle (center 0 0) (end 0.8 0) (layer "B.Fab") (width 0.1) (fill none))
     (pad "1" smd rect locked (at 0.75 -0.55) (size 0.7 0.7) (layers "B.Cu" "B.Paste" "B.Mask")
-      (net 152 "unconnected-(LD32-Pad1)") (pinfunction "DOUT") (pintype "output"))
+      (net 152 "Net-(LD32-Pad1)") (pinfunction "DOUT") (pintype "output"))
     (pad "2" smd rect locked (at 0.75 0.55) (size 0.7 0.7) (layers "B.Cu" "B.Paste" "B.Mask")
       (net 1 "GND") (pinfunction "GND") (pintype "power_in"))
@@
       (effects (font (size 1 1) (thickness 0.15)) (justify mirror))
     )
-    (fp_text value "Pin 22" (at 0 -1.55) (layer "B.SilkS")
+    (fp_text value "22" (at 0 -1.55) (layer "B.SilkS")
       (effects (font (size 1 1) (thickness 0.15)) (justify mirror))
     )
@@
     (effects (font (size 1 1) (thickness 0.15)) (justify right mirror))
   )
+  (gr_text "GND\nDATA\n+5V" (at 323.85 109.5375) (layer "B.SilkS")
+    (effects (font (size 1 1) (thickness 0.15)) (justify mirror))
+  )
   (gr_text "SPI-SH\n3v3\nCS\nTX\nRX\nSCK" (at 36.322 108.839) (layer "B.SilkS")
     (effects (font (size 1 1) (thickness 0.15)) (justify right mirror))
@@
     (effects (font (size 1 1) (thickness 0.15)) (justify mirror))
   )
-  (gr_text ".3.1" (at 136.1694 144.2212) (layer "B.SilkS")
+  (gr_text ".5" (at 136.1694 144.2212) (layer "B.SilkS")
     (effects (font (size 1.5 1.5) (thickness 0.3)) (justify left mirror))
   )
@@
   (segment (start 220.533739 108.287989) (end 220.533739 109.687011) (width 0.3) (layer "B.Cu") (net 1))
   (segment (start 160.711653 110.0875) (end 160.311164 109.687011) (width 0.3) (layer "B.Cu") (net 1))
+  (segment (start 315.598225 107.696) (end 318.8335 107.696) (width 0.3) (layer "B.Cu") (net 1))
   (segment (start 298.435128 110.0875) (end 298.73415 110.0875) (width 0.3) (layer "B.Cu") (net 1))
   (segment (start 246.343414 108.287989) (end 246.343414 109.523425) (width 0.3) (layer "B.Cu") (net 1))
@@
   (segment (start 43.305 78.0854) (end 43.305 73.9054) (width 0.3) (layer "B.Cu") (net 1))
   (segment (start 44.22 79.0004) (end 43.305 78.0854) (width 0.3) (layer "B.Cu") (net 1))
+  (segment (start 319.0875 107.95) (end 320.675 107.95) (width 0.3) (layer "B.Cu") (net 1))
   (segment (start 151.707939 109.687011) (end 151.707939 108.47205) (width 0.3) (layer "B.Cu") (net 1))
   (segment (start 306.565989 109.687011) (end 306.966478 110.0875) (width 0.3) (layer "B.Cu") (net 1))
@@
   (segment (start 66.076178 110.0875) (end 65.675689 109.687011) (width 0.3) (layer "B.Cu") (net 1))
   (segment (start 50.875 79.0004) (end 51.03 79.0004) (width 0.3) (layer "B.Cu") (net 1))
+  (segment (start 318.8335 107.696) (end 319.0875 107.95) (width 0.3) (layer "B.Cu") (net 1))
   (segment (start 194.724064 108.287989) (end 194.724064 109.507064) (width 0.3) (layer "B.Cu") (net 1))
   (segment (start 281.185325 107.858978) (end 280.756314 108.287989) (width 0.3) (layer "B.Cu") (net 1))
@@
   (segment (start 73.787 106.553) (end 82.423 106.553) (width 0.3) (layer "B.Cu") (net 2))
   (segment (start 82.08165 108.9875) (end 82.08165 107.9555) (width 0.3) (layer "B.Cu") (net 2))
+  (segment (start 321.525 110.275) (end 321.525 107.2125) (width 0.3) (layer "B.Cu") (net 2))
   (segment (start 133.9605 106.5775) (end 133.985 106.553) (width 0.3) (layer "B.Cu") (net 2))
   (segment (start 280.289 106.553) (end 288.798 106.553) (width 0.3) (layer "B.Cu") (net 2))
@@
   (segment (start 133.701 107.9555) (end 133.9605 107.696) (width 0.3) (layer "B.Cu") (net 2))
   (segment (start 245.802425 107.696) (end 245.802425 106.610425) (width 0.3) (layer "B.Cu") (net 2))
+  (segment (start 321.31 110.49) (end 321.525 110.275) (width 0.3) (layer "B.Cu") (net 2))
   (segment (start 185.32035 107.9555) (end 185.57985 107.696) (width 0.3) (layer "B.Cu") (net 2))
   (segment (start 99.5476 107.696) (end 99.5476 106.5734) (width 0.3) (layer "B.Cu") (net 2))
@@
   (segment (start 263.008875 107.696) (end 263.008875 106.561125) (width 0.3) (layer "B.Cu") (net 2))
   (segment (start 90.944375 107.696) (end 90.944375 106.565375) (width 0.3) (layer "B.Cu") (net 2))
+  (segment (start 321.525 107.2125) (end 320.8655 106.553) (width 0.3) (layer "B.Cu") (net 2))
   (segment (start 125.097775 108.9875) (end 125.097775 107.9555) (width 0.3) (layer "B.Cu") (net 2))
   (segment (start 47.879 81.2855) (end 47.879 81.788) (width 0.3) (layer "B.Cu") (net 2))
@@
   (segment (start 168.3734 107.696) (end 168.3734 106.6514) (width 0.3) (layer "B.Cu") (net 2))
   (segment (start 279.955825 108.9875) (end 279.955825 107.9555) (width 0.3) (layer "B.Cu") (net 2))
+  (segment (start 320.8655 106.553) (end 314.579 106.553) (width 0.3) (layer "B.Cu") (net 2))
   (segment (start 116.713 106.553) (end 125.349 106.553) (width 0.3) (layer "B.Cu") (net 2))
   (segment (start 297.434 106.553) (end 305.943 106.553) (width 0.3) (layer "B.Cu") (net 2))
@@
   (segment (start 73.737925 106.602075) (end 73.787 106.553) (width 0.3) (layer "B.Cu") (net 2))
   (segment (start 108.150825 107.696) (end 108.150825 106.606175) (width 0.3) (layer "B.Cu") (net 2))
+  (segment (start 320.675 110.49) (end 321.31 110.49) (width 0.3) (layer "B.Cu") (net 2))
   (segment (start 288.55905 107.9555) (end 288.81855 107.696) (width 0.3) (layer "B.Cu") (net 2))
   (segment (start 116.75405 106.59405) (end 116.713 106.553) (width 0.3) (layer "B.Cu") (net 2))
@@
   (segment (start 307.2655 108.9875) (end 313.069703 108.9875) (width 0.2) (layer "B.Cu") (net 151))
   (segment (start 313.069703 108.9875) (end 314.169703 110.0875) (width 0.2) (layer "B.Cu") (net 151))
+  (segment (start 318.5375 108.9875) (end 318.77 109.22) (width 0.2) (layer "B.Cu") (net 152))
+  (segment (start 320.675 109.22) (end 318.77 109.22) (width 0.2) (layer "B.Cu") (net 152))
+  (segment (start 315.868725 108.9875) (end 318.5375 108.9875) (width 0.2) (layer "B.Cu") (net 152))
   (segment (start 85.568 98.479) (end 85.568 97.372) (width 0.2) (layer "B.Cu") (net 153))
   (segment (start 85.875 96.266) (end 85.875 97.065) (width 0.2) (layer "B.Cu") (net 153))

Commit message: QSS Upload
Parts:
- removed Z0: EDI Logo, EDI:hlmk7
- added G***: EDI, EDI:EDILogo, B.Cu at (277.0, 90.5)
- added G***: LOGO, EDI:sweethaz, B.Cu at (317.0, 117.0)
- added G***: LOGO, EDI:hackpgh, B.Cu at (258.0, 89.0)
Other:
- board text added: "64% ORTHOLINEAR KEYBOARD"
- board text added: "HackPGH"
- board text added: "MARK 7 HARD LIGHT"
