File: Current/SweetBusiness/sb_mtx.kicad_sch (KiCad schematic)
At the start: 404 parts, among them J1 Toggle Link, K1 OmniSwitch, K10 OmniSwitch, K100 OmniSwitch, K101 OmniSwitch, K102 OmniSwitch, K103 OmniSwitch, K104 OmniSwitch, K105 OmniSwitch, K106 OmniSwitch, K107 OmniSwitch, K108 OmniSwitch, K109 OmniSwitch, K11 OmniSwitch, K110 OmniSwitch, K111 OmniSwitch, K112 OmniSwitch, K113 OmniSwitch, K114 OmniSwitch, K115 OmniSwitch, K116 OmniSwitch, K117 OmniSwitch, K118 OmniSwitch, K119 OmniSwitch, K12 OmniSwitch, K120 OmniSwitch, K121 OmniSwitch, K122 OmniSwitch, K123 OmniSwitch, K123.1 OmniSwitch, K124 OmniSwitch, K125 OmniSwitch, K13 OmniSwitch, K14 OmniSwitch, K15 OmniSwitch, K16 OmniSwitch, K17 OmniSwitch, K18 OmniSwitch, K19 OmniSwitch, K2 OmniSwitch, K20 OmniSwitch, K21 OmniSwitch, K22 OmniSwitch, K23 OmniSwitch, K24 OmniSwitch, K25 OmniSwitch, K26 OmniSwitch, K27 OmniSwitch, K28 OmniSwitch, K29 OmniSwitch, K3 OmniSwitch, K30 OmniSwitch, K31 OmniSwitch, K32 OmniSwitch, K33 OmniSwitch, K34 OmniSwitch, K35 OmniSwitch, K36 OmniSwitch, K37 OmniSwitch, K38 OmniSwitch, K39 OmniSwitch, K4 OmniSwitch, K40 OmniSwitch, K41 OmniSwitch, K42 OmniSwitch, K43 OmniSwitch, K44 OmniSwitch, K45 OmniSwitch, K46 OmniSwitch, K47 OmniSwitch, K48 OmniSwitch, K49 OmniSwitch, K5 OmniSwitch, K50 OmniSwitch, K51 OmniSwitch, K52 OmniSwitch, K53 OmniSwitch, K54 OmniSwitch, K55 OmniSwitch, K56 OmniSwitch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

Commit message: Nice changelog, idiot.
Parts:
- removed CI1, CI3, CI5, CI7: 1uf, EDI:Passive_0402_1005Metric, symbol Device:C_Small
- removed CI2, CI4, CI6, CI8, CI9: 100nF, EDI:Passive_0402_1005Metric, symbol Device:C_Small
- removed LD1, LD10, LD100, LD101, LD102, LD103, LD104, LD105, LD106, LD107, LD108, LD109, LD11, LD110, LD111, LD112, LD113, LD114, LD115, LD116, LD117, LD118, LD119, LD12, LD120, LD121, LD122, LD123, LD123.2, LD124, LD125, LD13, LD14, LD15, LD16, LD17, LD18, LD19, LD2, LD20, LD21, LD22, LD23, LD24, LD25, LD26, LD27, LD28, LD29, LD3, LD30, LD31, LD32, LD33, LD34, LD35, LD36, LD37, LD38, LD39, LD4, LD40, LD41, LD42, LD43, LD44, LD45, LD46, LD47, LD48, LD49, LD5, LD50, LD51, LD52, LD53, LD54, LD55, LD56, LD57, LD58, LD59, LD6, LD60, LD61, LD62, LD63, LD64, LD65, LD66, LD67, LD68, LD69, LD7, LD70, LD71, LD72, LD73, LD73.2, LD74, LD75, LD76, LD77, LD78, LD79, LD8, LD80, LD81, LD82, LD83, LD84, LD85, LD86, LD87, LD88, LD89, LD9, LD90, LD91, LD92, LD93, LD94, LD95, LD96, LD97, LD98, LD99: LED, EDI:SunLED-FlipRGB, symbol EDI:RGB-LED-Flip
- removed RI1, RI2: 2K, EDI:Passive_0402_1005Metric, symbol Device:R_Small
- removed RI3, RI4, RI5: 100K, EDI:Passive_0402_1005Metric, symbol Device:R_Small
- removed U3, U4: IS31FL3743A, Package_DFN_QFN:QFN-40-1EP_5x5mm_P0.4mm_EP3.8x3.8mm, symbol EDI:IS31FL3743A
- K1, K10, K11, K12, K13, K14, K15, K16, K17, K18, K19, K2, K20, K21, K22, K23, K24, K25, K26, K27, K28, K29, K3, K30, K31, K32, K33, K34, K35, K36, K37, K38, K39, K4, K40, K41, K42, K43, K44, K45, K46, K47, K48, K49, K5, K50, K51, K52, K53, K54, K55, K56, K57, K58, K59, K6, K60, K61, K62, K63, K64, K65, K66, K67, K68, K69, K7, K70, K71, K72, K74, K75, K76, K77, K78, K79, K8, K80, K81, K82, K83, K84, K85, K86, K87, K88, K89, K9, K90, K91: footprint EDI:MX-Choc -> EDI:MX-Choc-RGB
- K100: renamed from K99; footprint EDI:MX-Choc -> EDI:MX-Choc-RGB
- K101: renamed from K100; footprint EDI:MX-Choc -> EDI:MX-Choc-RGB
- K102: renamed from K101; footprint EDI:MX-Choc -> EDI:MX-Choc-RGB
- K103: renamed from K102; footprint EDI:MX-Choc -> EDI:MX-Choc-RGB
- K104: renamed from K103; footprint EDI:MX-Choc -> EDI:MX-Choc-RGB
- K105: renamed from K104; footprint EDI:MX-Choc -> EDI:MX-Choc-RGB
- K106: renamed from K105; footprint EDI:MX-Choc -> EDI:MX-Choc-RGB
- K107: renamed from K106; footprint EDI:MX-Choc -> EDI:MX-Choc-RGB
- K108: renamed from K107; footprint EDI:MX-Choc -> EDI:MX-Choc-RGB
- K109: renamed from K108; footprint EDI:MX-Choc -> EDI:MX-Choc-RGB
- K110: renamed from K109; footprint EDI:MX-Choc -> EDI:MX-Choc-RGB
- K111: renamed from K110; footprint EDI:MX-Choc -> EDI:MX-Choc-RGB
- K112: renamed from K111; footprint EDI:MX-Choc -> EDI:MX-Choc-RGB
- K113: renamed from K112; footprint EDI:MX-Choc -> EDI:MX-Choc-RGB
- K114: renamed from K113; footprint EDI:MX-Choc -> EDI:MX-Choc-RGB
- K115: renamed from K114; footprint EDI:MX-Choc -> EDI:MX-Choc-RGB
- K116: renamed from K115; footprint EDI:MX-Choc -> EDI:MX-Choc-RGB
- K117: renamed from K116; footprint EDI:MX-Choc -> EDI:MX-Choc-RGB
- K118: renamed from K117; footprint EDI:MX-Choc -> EDI:MX-Choc-RGB
- K119: renamed from K118; footprint EDI:MX-Choc -> EDI:MX-Choc-RGB
- K120: renamed from K119; footprint EDI:MX-Choc -> EDI:MX-Choc-RGB
- K121: renamed from K120; footprint EDI:MX-Choc -> EDI:MX-Choc-RGB
- K122: renamed from K121; footprint EDI:MX-Choc -> EDI:MX-Choc-RGB
- K123: renamed from K122; footprint EDI:MX-Choc -> EDI:MX-Choc-RGB
- K124: renamed from K123; footprint EDI:MX-Choc-Double -> EDI:MX-Choc-RGB
- K125: renamed from K123.1; footprint EDI:MX-Choc -> EDI:MX-Choc-RGB
- K126: renamed from K124; footprint EDI:MX-Choc -> EDI:MX-Choc-RGB
- K127: renamed from K125; footprint EDI:MX-Choc -> EDI:MX-Choc-RGB
- K73: footprint EDI:MX-Choc-Double -> EDI:MX-Choc-RGB
- K92: renamed from K73.1; footprint EDI:MX-Choc -> EDI:MX-Choc-RGB
- K93: renamed from K92; footprint EDI:MX-Choc -> EDI:MX-Choc-RGB
- K94: renamed from K93; footprint EDI:MX-Choc -> EDI:MX-Choc-RGB
- K95: renamed from K94; footprint EDI:MX-Choc -> EDI:MX-Choc-RGB
- K96: renamed from K95; footprint EDI:MX-Choc -> EDI:MX-Choc-RGB
- K97: renamed from K96; footprint EDI:MX-Choc -> EDI:MX-Choc-RGB
- K98: renamed from K97; footprint EDI:MX-Choc -> EDI:MX-Choc-RGB
- K99: renamed from K98; footprint EDI:MX-Choc -> EDI:MX-Choc-RGB
- RX1: footprint EDI:MX-Choc-Enc -> EDI:MX-Choc-Enc-RGB
- renumbered D99 to D100, D100 to D101, D101 to D102, D102 to D103, D103 to D104, D104 to D105, D105 to D106, D106 to D107, D107 to D108, D108 to D109, D109 to D110, D110 to D111, D111 to D112, D112 to D113, D113 to D114, D114 to D115, D115 to D116, D116 to D117, D117 to D118, D118 to D119, D119 to D120, D120 to D121, D121 to D122, D122 to D123, D123 to D124, D123.1 to D125, D124 to D126, D125 to D127, D73.1 to D92, D92 to D93, D93 to D94, D94 to D95, D95 to D96, D96 to D97, D97 to D98, D98 to D99
Connections:
- net col10: now also K117.1
- net col11: now also K118.1; no longer K117.1
- net col12: now also J1.8 (Pin_8), K119.1; no longer J1.2 (Pin_2), K118.1
- net col13: now also J1.6 (Pin_6), K120.1; no longer J1.4 (Pin_4), K119.1
- net col14: now also J1.4 (Pin_4); no longer J1.6 (Pin_6)
- net col15: now also J1.2 (Pin_2); no longer J1.8 (Pin_8), K120.1
- net col7: now also K116.1
- net col8: no longer K116.1
Other:
- moved on the sheet: D1, D10, D100, D101, D102, D103, D104, D105, D106, D107, D108, D109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

Commit message: Yep, moved some stuff to archives.
Parts:
- added DR2, DR3: SOD-523, EDI:D_SOD-523, symbol Device:D_Small
Connections:
- net col10 is gone; now on net col5: K103.1, K117.1, K19.1, K38.1, K61.1, K8.1, K84.1
- net col11 is gone; now on net col5: K104.1, K118.1, K20.1, K39.1, K62.1, K85.1, K9.1
- net col16 is gone; now on net col8: K10.1, K121.1, K25.1, K44.1, K67.1
- net col17 is gone; now on net col8: K107.1, K11.1, K122.1, K26.1, K45.1, K68.1
- net col18 is gone; now on net col9: K12.1, K123.1, K27.1, K46.1, K69.1
- net col19 is gone; now on net col9: K108.1, K124.1, K47.1, K70.1, K89.1
- net col21 is gone; now on net colA: K110.1, K126.1, K49.1, K72.1, K91.1
- net col22 is gone; now on net colB: K127.1, K50.1, K73.1, K92.1, RX1.1 (S1)
- net col0: now also K112.1, K29.1, K52.1, K75.1, K94.1
- net col1: now also K113.1, K114.1, K30.1, K31.1, K53.1, K54.1, K76.1, K77.1, K95.1, K96.1; no longer K112.1, K29.1, K52.1, K75.1, K94.1
- net col2: now also K115.1, K13.1, K14.1, K2.1, K3.1, K32.1, K33.1, K55.1, K56.1, K78.1, K79.1, K97.1, K98.1; no longer K113.1, K30.1, K53.1, K76.1, K95.1
- net col3: now also K100.1, K116.1, K15.1, K16.1, K34.1, K35.1, K4.1, K5.1, K57.1, K58.1, K80.1, K81.1, K99.1; no longer K114.1, K31.1, K54.1, K77.1, K96.1
- net col4: now also K101.1, K102.1, K17.1, K18.1, K36.1, K37.1, K59.1, K6.1, K60.1, K7.1, K82.1, K83.1; no longer K115.1, K13.1, K2.1, K32.1, K55.1, K78.1, K97.1
- net col5: no longer K14.1, K3.1, K33.1, K56.1, K79.1, K98.1
- net col6: now also J1.2 (Pin_2), J1.4 (Pin_4), K105.1, K106.1, K119.1, K120.1, K21.1, K22.1, K40.1, K41.1, K63.1, K64.1, K86.1, K87.1; no longer K15.1, K34.1, K4.1, K57.1, K80.1, K99.1
- net col7: now also J1.6 (Pin_6), J1.8 (Pin_8), K23.1, K24.1, K42.1, K43.1, K65.1, K66.1, K88.1; no longer K100.1, K116.1, K16.1, K35.1, K5.1, K58.1, K81.1
- net col8: no longer K101.1, K17.1, K36.1, K59.1, K6.1, K82.1
- net col9: no longer K102.1, K18.1, K37.1, K60.1, K7.1, K83.1
- net row0: now also DR2.1 (K); no longer D11.1 (K), D3.1 (K), D5.1 (K), D7.1 (K), D9.1 (K), DR1.1 (K), DT2.1 (K), DT4.1 (K)
- net row1: now also D11.1 (K), D3.1 (K), D5.1 (K), D7.1 (K), D9.1 (K), DT2.1 (K), DT4.1 (K), DR3.1 (K); no longer D13.1 (K), D14.1 (K), D15.1 (K), D16.1 (K), D17.1 (K), D18.1 (K), D19.1 (K), D20.1 (K), D21.1 (K), D22.1 (K), D23.1 (K), D24.1 (K), D25.1 (K), D26.1 (K), D27.1 (K)
- net row2: now also D13.1 (K), D15.1 (K), D17.1 (K), D19.1 (K), D21.1 (K), D23.1 (K), D25.1 (K), D27.1 (K), DR1.1 (K); no longer D28.1 (K), D29.1 (K), D30.1 (K), D31.1 (K), D32.1 (K), D33.1 (K), D34.1 (K), D35.1 (K), D36.1 (K), D37.1 (K), D38.1 (K), D39.1 (K), D40.1 (K), D41.1 (K), D42.1 (K), D43.1 (K), D44.1 (K), D45.1 (K), D46.1 (K), D47.1 (K), D48.1 (K), D49.1 (K), D50.1 (K)
- net row3: now also D14.1 (K), D16.1 (K), D18.1 (K), D20.1 (K), D22.1 (K), D24.1 (K), D26.1 (K); no longer D51.1 (K), D52.1 (K), D53.1 (K), D54.1 (K), D55.1 (K), D56.1 (K), D57.1 (K), D58.1 (K), D59.1 (K), D60.1 (K), D61.1 (K), D62.1 (K), D63.1 (K), D64.1 (K), D65.1 (K), D66.1 (K), D67.1 (K), D68.1 (K), D69.1 (K), D70.1 (K), D71.1 (K), D72.1 (K), D73.1 (K)
- net row4: now also D28.1 (K), D30.1 (K), D32.1 (K), D34.1 (K), D36.1 (K), D38.1 (K), D40.1 (K), D42.1 (K), D44.1 (K), D46.1 (K), D48.1 (K), D50.1 (K); no longer D74.1 (K), D75.1 (K), D76.1 (K), D77.1 (K), D78.1 (K), D79.1 (K), D80.1 (K), D81.1 (K), D82.1 (K), D83.1 (K), D84.1 (K), D85.1 (K), D86.1 (K), D87.1 (K), D88.1 (K), D89.1 (K), D90.1 (K), D91.1 (K), D92.1 (K)
- net row5: now also D29.1 (K), D31.1 (K), D33.1 (K), D35.1 (K), D37.1 (K), D39.1 (K), D41.1 (K), D43.1 (K), D45.1 (K), D47.1 (K), D49.1 (K); no longer D100.1 (K), D101.1 (K), D102.1 (K), D103.1 (K), D104.1 (K), D105.1 (K), D106.1 (K), D107.1 (K), D108.1 (K), D109.1 (K), D110.1 (K), D93.1 (K), D94.1 (K), D95.1 (K), D96.1 (K), D97.1 (K), D98.1 (K), D99.1 (K)
- net row6: now also D51.1 (K), D53.1 (K), D55.1 (K), D57.1 (K), D59.1 (K), D61.1 (K), D63.1 (K), D65.1 (K), D67.1 (K), D69.1 (K), D71.1 (K), D73.1 (K); no longer D111.1 (K), D112.1 (K), D113.1 (K), D114.1 (K), D115.1 (K), D116.1 (K), D117.1 (K), D118.1 (K), D119.1 (K), D120.1 (K), D121.1 (K), D122.1 (K), D123.1 (K), D124.1 (K), D125.1 (K), D126.1 (K), D127.1 (K)
- net GND renamed colB
- removed net col12: J1.8 (Pin_8), K105.1, K119.1, K21.1, K40.1, K63.1, K86.1
- removed net col13: J1.6 (Pin_6), K106.1, K120.1, K22.1, K41.1, K64.1, K87.1
- removed net col14: J1.4 (Pin_4), K23.1, K42.1, K65.1, K88.1
- removed net col15: J1.2 (Pin_2), K24.1, K43.1, K66.1
- net col20 renamed colA
- net enc0A: no longer names the net of RX1.A
- net enc0A: now also DR2.2 (A)
- net enc0B: no longer names the net of RX1.B
- net enc0B: now also DR3.2 (A)
- new net row7: D52.1 (K), D54.1 (K), D56.1 (K), D58.1 (K), D60.1 (K), D62.1 (K), D64.1 (K), D66.1 (K), D68.1 (K), D70.1 (K), D72.1 (K)
- new net row8: D74.1 (K), D76.1 (K), D78.1 (K), D80.1 (K), D82.1 (K), D84.1 (K), D86.1 (K), D88.1 (K), D90.1 (K), D92.1 (K)
- new net row9: D75.1 (K), D77.1 (K), D79.1 (K), D81.1 (K), D83.1 (K), D85.1 (K), D87.1 (K), D89.1 (K), D91.1 (K)
- new net rowA: D101.1 (K), D103.1 (K), D105.1 (K), D109.1 (K), D93.1 (K), D95.1 (K), D97.1 (K), D99.1 (K)
- new net rowB: D100.1 (K), D102.1 (K), D104.1 (K), D106.1 (K), D107.1 (K), D108.1 (K), D110.1 (K), D94.1 (K), D96.1 (K), D98.1 (K)
- new net rowC: D111.1 (K), D113.1 (K), D115.1 (K), D117.1 (K), D119.1 (K), D121.1 (K), D123.1 (K), D125.1 (K), D127.1 (K)
- new net rowD: D112.1 (K), D114.1 (K), D116.1 (K), D118.1 (K), D120.1 (K), D122.1 (K), D124.1 (K), D126.1 (K)
Other:
- moved on the sheet: D100, D102, D104, D106, D107, D108, D11, D110, D112, D114, D116, D118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

Commit message: So much stuff
Wow it's been a while.
Parts:
- removed DR3: SOD-523, EDI:D_SOD-523, symbol Device:D_Small
- removed J1: Toggle Link, Connector_PinHeader_2.54mm:PinHeader_2x04_P2.54mm_Vertical, symbol Connector_Generic:Conn_02x04_Odd_Even
- removed RX1: Media, EDI:MX-Choc-Enc-RGB, symbol Device:Rotary_Encoder_Switch
- added KT1, KT2, KT3, KT4: OmniSwitch, EDI:KeyToggle, symbol HL-Mk3-rescue:KEYSW-keyboard_parts-HL-Mk2-rescue
- added LC1, LC10, LC100, LC101, LC102, LC103, LC104, LC105, LC106, LC107, LC108, LC109, LC11, LC110, LC111, LC112, LC113, LC114, LC115, LC116, LC117, LC118, LC119, LC12, LC120, LC121, LC122, LC123, LC124, LC125, LC126, LC127, LC13, LC14, LC15, LC16, LC17, LC18, LC19, LC2, LC20, LC21, LC22, LC23, LC24, LC25, LC26, LC27, LC28, LC29, LC3, LC30, LC31, LC32, LC33, LC34, LC35, LC36, LC37, LC38, LC39, LC4, LC40, LC41, LC42, LC43, LC44, LC45, LC46, LC47, LC48, LC49, LC5, LC50, LC51, LC52, LC53, LC54, LC55, LC56, LC57, LC58, LC59, LC6, LC60, LC61, LC62, LC63, LC64, LC65, LC66, LC67, LC68, LC69, LC7, LC70, LC71, LC72, LC73, LC74, LC75, LC76, LC77, LC78, LC79, LC8, LC80, LC81, LC82, LC83, LC84, LC85, LC86, LC87, LC88, LC89, LC9, LC90, LC91, LC92, LC93, LC94, LC95, LC96, LC97, LC98, LC99: 100nF, EDI:Passive_0402_1005Metric, symbol Device:C_Small
- added LD1, LD10, LD100, LD101, LD102, LD103, LD104, LD105, LD106, LD107, LD108, LD109, LD11, LD110, LD111, LD112, LD113, LD114, LD115, LD116, LD117, LD118, LD119, LD12, LD120, LD121, LD122, LD123, LD124, LD125, LD126, LD127, LD13, LD14, LD15, LD16, LD17, LD18, LD19, LD2, LD20, LD21, LD22, LD23, LD24, LD25, LD26, LD27, LD28, LD29, LD3, LD30, LD31, LD32, LD33, LD34, LD35, LD36, LD37, LD38, LD39, LD4, LD40, LD41, LD42, LD43, LD44, LD45, LD46, LD47, LD48, LD49, LD5, LD50, LD51, LD52, LD53, LD54, LD55, LD56, LD57, LD58, LD59, LD6, LD60, LD61, LD62, LD63, LD64, LD65, LD66, LD67, LD68, LD69, LD7, LD70, LD71, LD72, LD73, LD74, LD75, LD76, LD77, LD78, LD79, LD8, LD80, LD81, LD82, LD83, LD84, LD85, LD86, LD87, LD88, LD89, LD9, LD90, LD91, LD92, LD93, LD94, LD95, LD96, LD97, LD98, LD99: WS2812C, EDI:WS2812C_2020, symbol LED:WS2812B
- added SWA1: SW_SPDT, EDI:KeyToggle-SPDT, symbol Switch:SW_SPDT
- K1, K10, K100, K101, K102, K103, K104, K105, K106, K107, K108, K109, K11, K110, K111, K112, K113, K114, K115, K116, K117, K118, K119, K12, K120, K121, K122, K123, K124, K125, K126, K127, K13, K14, K15, K16, K17, K18, K19, K2, K20, K21, K22, K23, K24, K25, K26, K27, K28, K29, K3, K30, K31, K32, K33, K34, K35, K36, K37, K38, K39, K4, K40, K41, K42, K43, K44, K45, K46, K47, K48, K49, K5, K50, K51, K52, K53, K54, K55, K56, K57, K58, K59, K6, K60, K61, K62, K63, K64, K65, K66, K67, K68, K69, K7, K70, K71, K72, K73, K74, K75, K76, K77, K78, K79, K8, K80, K81, K82, K83, K84, K85, K86, K87, K88, K89, K9, K90, K91, K92, K93, K94, K95, K96, K97, K98, K99: footprint EDI:MX-Choc-RGB -> EDI:SW_MX
- renumbered DR1 to DA1, DR2 to DA2
Connections:
- net col6: now also KT1.1, KT2.1
- net col7: now also KT3.1, KT4.1
- net colB: now also SWA1.2 (B)
- net row0: now also DA1.1 (K); no longer DA2.1 (K)
- net row1: now also DA2.1 (K)
- net row2: no longer DA1.1 (K)
- net at DT1.2 (A): now also KT1.2
- net at DA2.2 (A): now also SWA1.3 (C)
- net at DA1.2 (A): now also SWA1.1 (A)
- net at DT2.2 (A): now also KT2.2
- net at DT4.2 (A): now also KT4.2
- net at DT3.2 (A): now also KT3.2
- new net: LD6.2 (DOUT), LD7.4 (DIN)
- new net: LD5.2 (DOUT), LD6.4 (DIN)
- new net: LD66.4 (DIN), LD67.2 (DOUT)
- new net: LD67.4 (DIN), LD68.2 (DOUT)
- new net: LD2.2 (DOUT), LD3.4 (DIN)
- new net: LD1.2 (DOUT), LD2.4 (DIN)
- new net: LD112.2 (DOUT), LD113.4 (DIN)
- new net: LD111.2 (DOUT), LD112.4 (DIN)
- new net: LD90.2 (DOUT), LD91.4 (DIN)
- new net: LD89.2 (DOUT), LD90.4 (DIN)
- new net: LD47.2 (DOUT), LD48.4 (DIN)
- new net: LD46.2 (DOUT), LD47.4 (DIN)
- new net: LD102.4 (DIN), LD103.2 (DOUT)
- new net: LD103.4 (DIN), LD104.2 (DOUT)
- new net: LD39.2 (DOUT), LD40.4 (DIN)
- new net: LD38.2 (DOUT), LD39.4 (DIN)
- new net: LD105.4 (DIN), LD106.2 (DOUT)
- new net: LD106.4 (DIN), LD107.2 (DOUT)
- new net: LD20.4 (DIN), LD21.2 (DOUT)
- new net: LD21.4 (DIN), LD22.2 (DOUT)
- new net: LD35.2 (DOUT), LD36.4 (DIN)
- new net: LD34.2 (DOUT), LD35.4 (DIN)
- new net: LD43.2 (DOUT), LD44.4 (DIN)
- new net: LD42.2 (DOUT), LD43.4 (DIN)
- new net: LD25.4 (DIN), LD26.2 (DOUT)
- new net: LD26.4 (DIN), LD27.2 (DOUT)
- new net: LD28.2 (DOUT), LD29.4 (DIN)
- new net: LD13.2 (DOUT), LD28.4 (DIN)
- new net: LD59.4 (DIN), LD60.2 (DOUT)
- new net: LD60.4 (DIN), LD61.2 (DOUT)
- new net: LD118.2 (DOUT), LD119.4 (DIN)
- new net: LD117.2 (DOUT), LD118.4 (DIN)
- new net: LD78.2 (DOUT), LD79.4 (DIN)
- new net: LD77.2 (DOUT), LD78.4 (DIN)
- new net: LD17.4 (DIN), LD18.2 (DOUT)
- new net: LD18.4 (DIN), LD19.2 (DOUT)
- new net: LD68.4 (DIN), LD69.2 (DOUT)
- new net: LD95.4 (DIN), LD96.2 (DOUT)
- new net: LD96.4 (DIN), LD97.2 (DOUT)
- new net: LD84.2 (DOUT), LD85.4 (DIN)
- new net: LD83.2 (DOUT), LD84.4 (DIN)
- new net: LD75.2 (DOUT), LD76.4 (DIN)
- new net: LD74.2 (DOUT), LD75.4 (DIN)
- new net: LD80.2 (DOUT), LD81.4 (DIN)
- new net: LD79.2 (DOUT), LD80.4 (DIN)
- new net: LD58.4 (DIN), LD59.2 (DOUT)
- new net: LD72.4 (DIN), LD73.2 (DOUT)
- new net: LD50.2 (DOUT), LD73.4 (DIN)
- new net: LD101.4 (DIN), LD102.2 (DOUT)
- new net: LD110.4 (DIN), LD92.2 (DOUT)
- new net: LD91.2 (DOUT), LD92.4 (DIN)
- new net: LD108.4 (DIN), LD109.2 (DOUT)
- new net: LD109.4 (DIN), LD110.2 (DOUT)
- new net: LD33.2 (DOUT), LD34.4 (DIN)
- new net: LD93.4 (DIN), LD94.2 (DOUT)
- new net: LD94.4 (DIN), LD95.2 (DOUT)
- new net: LD121.2 (DOUT), LD122.4 (DIN)
- new net: LD120.2 (DOUT), LD121.4 (DIN)
- new net: LD100.4 (DIN), LD101.2 (DOUT)
- new net: LD111.4 (DIN), LD93.2 (DOUT)
- new net: LD52.4 (DIN), LD53.2 (DOUT)
- new net: LD53.4 (DIN), LD54.2 (DOUT)
- new net: LD37.2 (DOUT), LD38.4 (DIN)
- new net: LD124.2 (DOUT), LD125.4 (DIN)
- new net: LD123.2 (DOUT), LD124.4 (DIN)
- new net: LD107.4 (DIN), LD108.2 (DOUT)
- new net: LD51.4 (DIN), LD52.2 (DOUT)
- new net: LD10.4 (DIN), LD9.2 (DOUT)
- new net: LD8.2 (DOUT), LD9.4 (DIN)
- new net: LD23.4 (DIN), LD24.2 (DOUT)
- new net: LD24.4 (DIN), LD25.2 (DOUT)
- new net: LD45.2 (DOUT), LD46.4 (DIN)
- new net: LD44.2 (DOUT), LD45.4 (DIN)
- new net: LD69.4 (DIN), LD70.2 (DOUT)
- new net: LD119.2 (DOUT), LD120.4 (DIN)
- new net: LD32.2 (DOUT), LD33.4 (DIN)
- new net: LD31.2 (DOUT), LD32.4 (DIN)
- new net: LD126.2 (DOUT), LD127.4 (DIN)
- new net: LD61.4 (DIN), LD62.2 (DOUT)
- new net: LD62.4 (DIN), LD63.2 (DOUT)
- new net: LD49.2 (DOUT), LD50.4 (DIN)
- new net: LD100.2 (DOUT), LD99.4 (DIN)
- new net: LD97.4 (DIN), LD98.2 (DOUT)
- new net: LD85.2 (DOUT), LD86.4 (DIN)
- new net: LD81.2 (DOUT), LD82.4 (DIN)
- new net: LD122.2 (DOUT), LD123.4 (DIN)
- new net: LD14.4 (DIN), LD15.2 (DOUT)
- new net: LD15.4 (DIN), LD16.2 (DOUT)
- new net: LD51.2 (DOUT), LD74.4 (DIN)
- new net: LD76.2 (DOUT), LD77.4 (DIN)
- new net: LD30.2 (DOUT), LD31.4 (DIN)
- new net: LD41.2 (DOUT), LD42.4 (DIN)
- new net: LD54.4 (DIN), LD55.2 (DOUT)
- new net: LD71.4 (DIN), LD72.2 (DOUT)
- new net: LD65.4 (DIN), LD66.2 (DOUT)
- new net: LD22.4 (DIN), LD23.2 (DOUT)
- new net: LD12.2 (DOUT), LD27.4 (DIN)
- new net: LD11.2 (DOUT), LD12.4 (DIN)
- new net: LD116.2 (DOUT), LD117.4 (DIN)
- new net: LD115.2 (DOUT), LD116.4 (DIN)
- new net: LD125.2 (DOUT), LD126.4 (DIN)
- new net: LD98.4 (DIN), LD99.2 (DOUT)
- new net: LD70.4 (DIN), LD71.2 (DOUT)
- new net: LD104.4 (DIN), LD105.2 (DOUT)
- new net: LD4.2 (DOUT), LD5.4 (DIN)
- new net: LD3.2 (DOUT), LD4.4 (DIN)
- new net: LD114.2 (DOUT), LD115.4 (DIN)
- new net: LD40.2 (DOUT), LD41.4 (DIN)
- new net: LD88.2 (DOUT), LD89.4 (DIN)
- new net: LD87.2 (DOUT), LD88.4 (DIN)
- new net: LD86.2 (DOUT), LD87.4 (DIN)
- new net: LD57.4 (DIN), LD58.2 (DOUT)
- new net: LD36.2 (DOUT), LD37.4 (DIN)
- new net: LD16.4 (DIN), LD17.2 (DOUT)
- new net: LD55.4 (DIN), LD56.2 (DOUT)
- new net: LD56.4 (DIN), LD57.2 (DOUT)
- new net: LD113.2 (DOUT), LD114.4 (DIN)
- new net: LD82.2 (DOUT), LD83.4 (DIN)
- new net: LD10.2 (DOUT), LD11.4 (DIN)
- new net: LD7.2 (DOUT), LD8.4 (DIN)
- new net: LD48.2 (DOUT), LD49.4 (DIN)
- new net: LD63.4 (DIN), LD64.2 (DOUT)
- new net: LD29.2 (DOUT), LD30.4 (DIN)
- new net: LD13.4 (DIN), LD14.2 (DOUT)
- new net: LD19.4 (DIN), LD20.2 (DOUT)
- new net: LD64.4 (DIN), LD65.2 (DOUT)
- new net +3V3: LC1.2, LC10.2, LC100.2, LC101.2, LC102.2, LC103.2, LC104.2, LC105.2, LC106.2, LC107.2, LC108.2, LC109.2, LC11.2, LC110.2, LC111.2, LC112.2, LC113.2, LC114.2, LC115.2, LC116.2, LC117.2, LC118.2, LC119.2, LC12.2, LC120.2, LC121.2, LC122.2, LC123.2, LC124.2, LC125.2, LC126.2, LC127.2, LC13.2, LC14.2, LC15.2, LC16.2, LC17.2, LC18.2, LC19.2, LC2.2, LC20.2, LC21.2, LC22.2, LC23.2, LC24.2, LC25.2, LC26.2, LC27.2, LC28.2, LC29.2, LC3.2, LC30.2, LC31.2, LC32.2, LC33.2, LC34.2, LC35.2, LC36.2, LC37.2, LC38.2, LC39.2, LC4.2, LC40.2, LC41.2, LC42.2, LC43.2, LC44.2, LC45.2, LC46.2, LC47.2, LC48.2, LC49.2, LC5.2, LC50.2, LC51.2, LC52.2, LC53.2, LC54.2, LC55.2, LC56.2, LC57.2, LC58.2, LC59.2, LC6.2, LC60.2, LC61.2, LC62.2, LC63.2, LC64.2, LC65.2, LC66.2, LC67.2, LC68.2, LC69.2, LC7.2, LC70.2, LC71.2, LC72.2, LC73.2, LC74.2, LC75.2, LC76.2, LC77.2, LC78.2, LC79.2, LC8.2, LC80.2, LC81.2, LC82.2, LC83.2, LC84.2, LC85.2, LC86.2, LC87.2, LC88.2, LC89.2, LC9.2, LC90.2, LC91.2, LC92.2, LC93.2, LC94.2, LC95.2, LC96.2, LC97.2, LC98.2, LC99.2, LD1.1 (VDD), LD10.1 (VDD), LD100.1 (VDD), LD101.1 (VDD), LD102.1 (VDD), LD103.1 (VDD), LD104.1 (VDD), LD105.1 (VDD), LD106.1 (VDD), LD107.1 (VDD), LD108.1 (VDD), LD109.1 (VDD), LD11.1 (VDD), LD110.1 (VDD), LD111.1 (VDD), LD112.1 (VDD), LD113.1 (VDD), LD114.1 (VDD), LD115.1 (VDD), LD116.1 (VDD), LD117.1 (VDD), LD118.1 (VDD), LD119.1 (VDD), LD12.1 (VDD), LD120.1 (VDD), LD121.1 (VDD), LD122.1 (VDD), LD123.1 (VDD), LD124.1 (VDD), LD125.1 (VDD), LD126.1 (VDD), LD127.1 (VDD), LD13.1 (VDD), LD14.1 (VDD), LD15.1 (VDD), LD16.1 (VDD), LD17.1 (VDD), LD18.1 (VDD), LD19.1 (VDD), LD2.1 (VDD), LD20.1 (VDD), LD21.1 (VDD), LD22.1 (VDD), LD23.1 (VDD), LD24.1 (VDD), LD25.1 (VDD), LD26.1 (VDD), LD27.1 (VDD), LD28.1 (VDD), LD29.1 (VDD), LD3.1 (VDD), LD30.1 (VDD), LD31.1 (VDD), LD32.1 (VDD), LD33.1 (VDD), LD34.1 (VDD), LD35.1 (VDD), LD36.1 (VDD), LD37.1 (VDD), LD38.1 (VDD), LD39.1 (VDD), LD4.1 (VDD), LD40.1 (VDD), LD41.1 (VDD), LD42.1 (VDD), LD43.1 (VDD), LD44.1 (VDD), LD45.1 (VDD), LD46.1 (VDD), LD47.1 (VDD), LD48.1 (VDD), LD49.1 (VDD), LD5.1 (VDD), LD50.1 (VDD), LD51.1 (VDD), LD52.1 (VDD), LD53.1 (VDD), LD54.1 (VDD), LD55.1 (VDD), LD56.1 (VDD), LD57.1 (VDD), LD58.1 (VDD), LD59.1 (VDD), LD6.1 (VDD), LD60.1 (VDD), LD61.1 (VDD), LD62.1 (VDD), LD63.1 (VDD), LD64.1 (VDD), LD65.1 (VDD), LD66.1 (VDD), LD67.1 (VDD), LD68.1 (VDD), LD69.1 (VDD), LD7.1 (VDD), LD70.1 (VDD), LD71.1 (VDD), LD72.1 (VDD), LD73.1 (VDD), LD74.1 (VDD), LD75.1 (VDD), LD76.1 (VDD), LD77.1 (VDD), LD78.1 (VDD), LD79.1 (VDD), LD8.1 (VDD), LD80.1 (VDD), LD81.1 (VDD), LD82.1 (VDD), LD83.1 (VDD), LD84.1 (VDD), LD85.1 (VDD), LD86.1 (VDD), LD87.1 (VDD), LD88.1 (VDD), LD89.1 (VDD), LD9.1 (VDD), LD90.1 (VDD), LD91.1 (VDD), LD92.1 (VDD), LD93.1 (VDD), LD94.1 (VDD), LD95.1 (VDD), LD96.1 (VDD), LD97.1 (VDD), LD98.1 (VDD), LD99.1 (VDD)
- new net GND: LC1.1, LC10.1, LC100.1, LC101.1, LC102.1, LC103.1, LC104.1, LC105.1, LC106.1, LC107.1, LC108.1, LC109.1, LC11.1, LC110.1, LC111.1, LC112.1, LC113.1, LC114.1, LC115.1, LC116.1, LC117.1, LC118.1, LC119.1, LC12.1, LC120.1, LC121.1, LC122.1, LC123.1, LC124.1, LC125.1, LC126.1, LC127.1, LC13.1, LC14.1, LC15.1, LC16.1, LC17.1, LC18.1, LC19.1, LC2.1, LC20.1, LC21.1, LC22.1, LC23.1, LC24.1, LC25.1, LC26.1, LC27.1, LC28.1, LC29.1, LC3.1, LC30.1, LC31.1, LC32.1, LC33.1, LC34.1, LC35.1, LC36.1, LC37.1, LC38.1, LC39.1, LC4.1, LC40.1, LC41.1, LC42.1, LC43.1, LC44.1, LC45.1, LC46.1, LC47.1, LC48.1, LC49.1, LC5.1, LC50.1, LC51.1, LC52.1, LC53.1, LC54.1, LC55.1, LC56.1, LC57.1, LC58.1, LC59.1, LC6.1, LC60.1, LC61.1, LC62.1, LC63.1, LC64.1, LC65.1, LC66.1, LC67.1, LC68.1, LC69.1, LC7.1, LC70.1, LC71.1, LC72.1, LC73.1, LC74.1, LC75.1, LC76.1, LC77.1, LC78.1, LC79.1, LC8.1, LC80.1, LC81.1, LC82.1, LC83.1, LC84.1, LC85.1, LC86.1, LC87.1, LC88.1, LC89.1, LC9.1, LC90.1, LC91.1, LC92.1, LC93.1, LC94.1, LC95.1, LC96.1, LC97.1, LC98.1, LC99.1, LD1.3 (VSS), LD10.3 (VSS), LD100.3 (VSS), LD101.3 (VSS), LD102.3 (VSS), LD103.3 (VSS), LD104.3 (VSS), LD105.3 (VSS), LD106.3 (VSS), LD107.3 (VSS), LD108.3 (VSS), LD109.3 (VSS), LD11.3 (VSS), LD110.3 (VSS), LD111.3 (VSS), LD112.3 (VSS), LD113.3 (VSS), LD114.3 (VSS), LD115.3 (VSS), LD116.3 (VSS), LD117.3 (VSS), LD118.3 (VSS), LD119.3 (VSS), LD12.3 (VSS), LD120.3 (VSS), LD121.3 (VSS), LD122.3 (VSS), LD123.3 (VSS), LD124.3 (VSS), LD125.3 (VSS), LD126.3 (VSS), LD127.3 (VSS), LD13.3 (VSS), LD14.3 (VSS), LD15.3 (VSS), LD16.3 (VSS), LD17.3 (VSS), LD18.3 (VSS), LD19.3 (VSS), LD2.3 (VSS), LD20.3 (VSS), LD21.3 (VSS), LD22.3 (VSS), LD23.3 (VSS), LD24.3 (VSS), LD25.3 (VSS), LD26.3 (VSS), LD27.3 (VSS), LD28.3 (VSS), LD29.3 (VSS), LD3.3 (VSS), LD30.3 (VSS), LD31.3 (VSS), LD32.3 (VSS), LD33.3 (VSS), LD34.3 (VSS), LD35.3 (VSS), LD36.3 (VSS), LD37.3 (VSS), LD38.3 (VSS), LD39.3 (VSS), LD4.3 (VSS), LD40.3 (VSS), LD41.3 (VSS), LD42.3 (VSS), LD43.3 (VSS), LD44.3 (VSS), LD45.3 (VSS), LD46.3 (VSS), LD47.3 (VSS), LD48.3 (VSS), LD49.3 (VSS), LD5.3 (VSS), LD50.3 (VSS), LD51.3 (VSS), LD52.3 (VSS), LD53.3 (VSS), LD54.3 (VSS), LD55.3 (VSS), LD56.3 (VSS), LD57.3 (VSS), LD58.3 (VSS), LD59.3 (VSS), LD6.3 (VSS), LD60.3 (VSS), LD61.3 (VSS), LD62.3 (VSS), LD63.3 (VSS), LD64.3 (VSS), LD65.3 (VSS), LD66.3 (VSS), LD67.3 (VSS), LD68.3 (VSS), LD69.3 (VSS), LD7.3 (VSS), LD70.3 (VSS), LD71.3 (VSS), LD72.3 (VSS), LD73.3 (VSS), LD74.3 (VSS), LD75.3 (VSS), LD76.3 (VSS), LD77.3 (VSS), LD78.3 (VSS), LD79.3 (VSS), LD8.3 (VSS), LD80.3 (VSS), LD81.3 (VSS), LD82.3 (VSS), LD83.3 (VSS), LD84.3 (VSS), LD85.3 (VSS), LD86.3 (VSS), LD87.3 (VSS), LD88.3 (VSS), LD89.3 (VSS), LD9.3 (VSS), LD90.3 (VSS), LD91.3 (VSS), LD92.3 (VSS), LD93.3 (VSS), LD94.3 (VSS), LD95.3 (VSS), LD96.3 (VSS), LD97.3 (VSS), LD98.3 (VSS), LD99.3 (VSS)
- new net LED: LD1.4 (DIN)
- no-connect marks 0 -> 1
Other:
- moved on the sheet: D1, D10, D100, D101, D102, D103, D104, D105, D106, D107, D108, D109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

Commit message: Bulk catchup commit 2023-01-21
Parts:
- LD1, LD10, LD100, LD101, LD102, LD103, LD104, LD105, LD106, LD107, LD108, LD109, LD11, LD110, LD111, LD112, LD113, LD114, LD115, LD116, LD117, LD118, LD119, LD12, LD120, LD121, LD122, LD123, LD124, LD125, LD126, LD127, LD13, LD14, LD15, LD16, LD17, LD18, LD19, LD2, LD20, LD21, LD22, LD23, LD24, LD25, LD26, LD27, LD28, LD29, LD3, LD30, LD31, LD32, LD33, LD34, LD35, LD36, LD37, LD38, LD39, LD4, LD40, LD41, LD42, LD43, LD44, LD45, LD46, LD47, LD48, LD49, LD5, LD50, LD51, LD52, LD53, LD54, LD55, LD56, LD57, LD58, LD59, LD6, LD60, LD61, LD62, LD63, LD64, LD65, LD66, LD67, LD68, LD69, LD7, LD70, LD71, LD72, LD73, LD74, LD75, LD76, LD77, LD78, LD79, LD8, LD80, LD81, LD82, LD83, LD84, LD85, LD86, LD87, LD88, LD89, LD9, LD90, LD91, LD92, LD93, LD94, LD95, LD96, LD97, LD98, LD99: footprint EDI:WS2812C_2020 -> EDI:WS2812B_2020; symbol LED:WS2812B -> EDI:WS2812C
Connections:
- net +3V3: now also LD1.4 (VDD), LD10.4 (VDD), LD100.4 (VDD), LD101.4 (VDD), LD102.4 (VDD), LD103.4 (VDD), LD104.4 (VDD), LD105.4 (VDD), LD106.4 (VDD), LD107.4 (VDD), LD108.4 (VDD), LD109.4 (VDD), LD11.4 (VDD), LD110.4 (VDD), LD111.4 (VDD), LD112.4 (VDD), LD113.4 (VDD), LD114.4 (VDD), LD115.4 (VDD), LD116.4 (VDD), LD117.4 (VDD), LD118.4 (VDD), LD119.4 (VDD), LD12.4 (VDD), LD120.4 (VDD), LD121.4 (VDD), LD122.4 (VDD), LD123.4 (VDD), LD124.4 (VDD), LD125.4 (VDD), LD126.4 (VDD), LD127.4 (VDD), LD13.4 (VDD), LD14.4 (VDD), LD15.4 (VDD), LD16.4 (VDD), LD17.4 (VDD), LD18.4 (VDD), LD19.4 (VDD), LD2.4 (VDD), LD20.4 (VDD), LD21.4 (VDD), LD22.4 (VDD), LD23.4 (VDD), LD24.4 (VDD), LD25.4 (VDD), LD26.4 (VDD), LD27.4 (VDD), LD28.4 (VDD), LD29.4 (VDD), LD3.4 (VDD), LD30.4 (VDD), LD31.4 (VDD), LD32.4 (VDD), LD33.4 (VDD), LD34.4 (VDD), LD35.4 (VDD), LD36.4 (VDD), LD37.4 (VDD), LD38.4 (VDD), LD39.4 (VDD), LD4.4 (VDD), LD40.4 (VDD), LD41.4 (VDD), LD42.4 (VDD), LD43.4 (VDD), LD44.4 (VDD), LD45.4 (VDD), LD46.4 (VDD), LD47.4 (VDD), LD48.4 (VDD), LD49.4 (VDD), LD5.4 (VDD), LD50.4 (VDD), LD51.4 (VDD), LD52.4 (VDD), LD53.4 (VDD), LD54.4 (VDD), LD55.4 (VDD), LD56.4 (VDD), LD57.4 (VDD), LD58.4 (VDD), LD59.4 (VDD), LD6.4 (VDD), LD60.4 (VDD), LD61.4 (VDD), LD62.4 (VDD), LD63.4 (VDD), LD64.4 (VDD), LD65.4 (VDD), LD66.4 (VDD), LD67.4 (VDD), LD68.4 (VDD), LD69.4 (VDD), LD7.4 (VDD), LD70.4 (VDD), LD71.4 (VDD), LD72.4 (VDD), LD73.4 (VDD), LD74.4 (VDD), LD75.4 (VDD), LD76.4 (VDD), LD77.4 (VDD), LD78.4 (VDD), LD79.4 (VDD), LD8.4 (VDD), LD80.4 (VDD), LD81.4 (VDD), LD82.4 (VDD), LD83.4 (VDD), LD84.4 (VDD), LD85.4 (VDD), LD86.4 (VDD), LD87.4 (VDD), LD88.4 (VDD), LD89.4 (VDD), LD9.4 (VDD), LD90.4 (VDD), LD91.4 (VDD), LD92.4 (VDD), LD93.4 (VDD), LD94.4 (VDD), LD95.4 (VDD), LD96.4 (VDD), LD97.4 (VDD), LD98.4 (VDD), LD99.4 (VDD); no longer LD1.1 (VDD), LD10.1 (VDD), LD100.1 (VDD), LD101.1 (VDD), LD102.1 (VDD), LD103.1 (VDD), LD104.1 (VDD), LD105.1 (VDD), LD106.1 (VDD), LD107.1 (VDD), LD108.1 (VDD), LD109.1 (VDD), LD11.1 (VDD), LD110.1 (VDD), LD111.1 (VDD), LD112.1 (VDD), LD113.1 (VDD), LD114.1 (VDD), LD115.1 (VDD), LD116.1 (VDD), LD117.1 (VDD), LD118.1 (VDD), LD119.1 (VDD), LD12.1 (VDD), LD120.1 (VDD), LD121.1 (VDD), LD122.1 (VDD), LD123.1 (VDD), LD124.1 (VDD), LD125.1 (VDD), LD126.1 (VDD), LD127.1 (VDD), LD13.1 (VDD), LD14.1 (VDD), LD15.1 (VDD), LD16.1 (VDD), LD17.1 (VDD), LD18.1 (VDD), LD19.1 (VDD), LD2.1 (VDD), LD20.1 (VDD), LD21.1 (VDD), LD22.1 (VDD), LD23.1 (VDD), LD24.1 (VDD), LD25.1 (VDD), LD26.1 (VDD), LD27.1 (VDD), LD28.1 (VDD), LD29.1 (VDD), LD3.1 (VDD), LD30.1 (VDD), LD31.1 (VDD), LD32.1 (VDD), LD33.1 (VDD), LD34.1 (VDD), LD35.1 (VDD), LD36.1 (VDD), LD37.1 (VDD), LD38.1 (VDD), LD39.1 (VDD), LD4.1 (VDD), LD40.1 (VDD), LD41.1 (VDD), LD42.1 (VDD), LD43.1 (VDD), LD44.1 (VDD), LD45.1 (VDD), LD46.1 (VDD), LD47.1 (VDD), LD48.1 (VDD), LD49.1 (VDD), LD5.1 (VDD), LD50.1 (VDD), LD51.1 (VDD), LD52.1 (VDD), LD53.1 (VDD), LD54.1 (VDD), LD55.1 (VDD), LD56.1 (VDD), LD57.1 (VDD), LD58.1 (VDD), LD59.1 (VDD), LD6.1 (VDD), LD60.1 (VDD), LD61.1 (VDD), LD62.1 (VDD), LD63.1 (VDD), LD64.1 (VDD), LD65.1 (VDD), LD66.1 (VDD), LD67.1 (VDD), LD68.1 (VDD), LD69.1 (VDD), LD7.1 (VDD), LD70.1 (VDD), LD71.1 (VDD), LD72.1 (VDD), LD73.1 (VDD), LD74.1 (VDD), LD75.1 (VDD), LD76.1 (VDD), LD77.1 (VDD), LD78.1 (VDD), LD79.1 (VDD), LD8.1 (VDD), LD80.1 (VDD), LD81.1 (VDD), LD82.1 (VDD), LD83.1 (VDD), LD84.1 (VDD), LD85.1 (VDD), LD86.1 (VDD), LD87.1 (VDD), LD88.1 (VDD), LD89.1 (VDD), LD9.1 (VDD), LD90.1 (VDD), LD91.1 (VDD), LD92.1 (VDD), LD93.1 (VDD), LD94.1 (VDD), LD95.1 (VDD), LD96.1 (VDD), LD97.1 (VDD), LD98.1 (VDD), LD99.1 (VDD)
- net GND: now also LD1.2 (GND), LD10.2 (GND), LD100.2 (GND), LD101.2 (GND), LD102.2 (GND), LD103.2 (GND), LD104.2 (GND), LD105.2 (GND), LD106.2 (GND), LD107.2 (GND), LD108.2 (GND), LD109.2 (GND), LD11.2 (GND), LD110.2 (GND), LD111.2 (GND), LD112.2 (GND), LD113.2 (GND), LD114.2 (GND), LD115.2 (GND), LD116.2 (GND), LD117.2 (GND), LD118.2 (GND), LD119.2 (GND), LD12.2 (GND), LD120.2 (GND), LD121.2 (GND), LD122.2 (GND), LD123.2 (GND), LD124.2 (GND), LD125.2 (GND), LD126.2 (GND), LD127.2 (GND), LD13.2 (GND), LD14.2 (GND), LD15.2 (GND), LD16.2 (GND), LD17.2 (GND), LD18.2 (GND), LD19.2 (GND), LD2.2 (GND), LD20.2 (GND), LD21.2 (GND), LD22.2 (GND), LD23.2 (GND), LD24.2 (GND), LD25.2 (GND), LD26.2 (GND), LD27.2 (GND), LD28.2 (GND), LD29.2 (GND), LD3.2 (GND), LD30.2 (GND), LD31.2 (GND), LD32.2 (GND), LD33.2 (GND), LD34.2 (GND), LD35.2 (GND), LD36.2 (GND), LD37.2 (GND), LD38.2 (GND), LD39.2 (GND), LD4.2 (GND), LD40.2 (GND), LD41.2 (GND), LD42.2 (GND), LD43.2 (GND), LD44.2 (GND), LD45.2 (GND), LD46.2 (GND), LD47.2 (GND), LD48.2 (GND), LD49.2 (GND), LD5.2 (GND), LD50.2 (GND), LD51.2 (GND), LD52.2 (GND), LD53.2 (GND), LD54.2 (GND), LD55.2 (GND), LD56.2 (GND), LD57.2 (GND), LD58.2 (GND), LD59.2 (GND), LD6.2 (GND), LD60.2 (GND), LD61.2 (GND), LD62.2 (GND), LD63.2 (GND), LD64.2 (GND), LD65.2 (GND), LD66.2 (GND), LD67.2 (GND), LD68.2 (GND), LD69.2 (GND), LD7.2 (GND), LD70.2 (GND), LD71.2 (GND), LD72.2 (GND), LD73.2 (GND), LD74.2 (GND), LD75.2 (GND), LD76.2 (GND), LD77.2 (GND), LD78.2 (GND), LD79.2 (GND), LD8.2 (GND), LD80.2 (GND), LD81.2 (GND), LD82.2 (GND), LD83.2 (GND), LD84.2 (GND), LD85.2 (GND), LD86.2 (GND), LD87.2 (GND), LD88.2 (GND), LD89.2 (GND), LD9.2 (GND), LD90.2 (GND), LD91.2 (GND), LD92.2 (GND), LD93.2 (GND), LD94.2 (GND), LD95.2 (GND), LD96.2 (GND), LD97.2 (GND), LD98.2 (GND), LD99.2 (GND); no longer LD1.3 (VSS), LD10.3 (VSS), LD100.3 (VSS), LD101.3 (VSS), LD102.3 (VSS), LD103.3 (VSS), LD104.3 (VSS), LD105.3 (VSS), LD106.3 (VSS), LD107.3 (VSS), LD108.3 (VSS), LD109.3 (VSS), LD11.3 (VSS), LD110.3 (VSS), LD111.3 (VSS), LD112.3 (VSS), LD113.3 (VSS), LD114.3 (VSS), LD115.3 (VSS), LD116.3 (VSS), LD117.3 (VSS), LD118.3 (VSS), LD119.3 (VSS), LD12.3 (VSS), LD120.3 (VSS), LD121.3 (VSS), LD122.3 (VSS), LD123.3 (VSS), LD124.3 (VSS), LD125.3 (VSS), LD126.3 (VSS), LD127.3 (VSS), LD13.3 (VSS), LD14.3 (VSS), LD15.3 (VSS), LD16.3 (VSS), LD17.3 (VSS), LD18.3 (VSS), LD19.3 (VSS), LD2.3 (VSS), LD20.3 (VSS), LD21.3 (VSS), LD22.3 (VSS), LD23.3 (VSS), LD24.3 (VSS), LD25.3 (VSS), LD26.3 (VSS), LD27.3 (VSS), LD28.3 (VSS), LD29.3 (VSS), LD3.3 (VSS), LD30.3 (VSS), LD31.3 (VSS), LD32.3 (VSS), LD33.3 (VSS), LD34.3 (VSS), LD35.3 (VSS), LD36.3 (VSS), LD37.3 (VSS), LD38.3 (VSS), LD39.3 (VSS), LD4.3 (VSS), LD40.3 (VSS), LD41.3 (VSS), LD42.3 (VSS), LD43.3 (VSS), LD44.3 (VSS), LD45.3 (VSS), LD46.3 (VSS), LD47.3 (VSS), LD48.3 (VSS), LD49.3 (VSS), LD5.3 (VSS), LD50.3 (VSS), LD51.3 (VSS), LD52.3 (VSS), LD53.3 (VSS), LD54.3 (VSS), LD55.3 (VSS), LD56.3 (VSS), LD57.3 (VSS), LD58.3 (VSS), LD59.3 (VSS), LD6.3 (VSS), LD60.3 (VSS), LD61.3 (VSS), LD62.3 (VSS), LD63.3 (VSS), LD64.3 (VSS), LD65.3 (VSS), LD66.3 (VSS), LD67.3 (VSS), LD68.3 (VSS), LD69.3 (VSS), LD7.3 (VSS), LD70.3 (VSS), LD71.3 (VSS), LD72.3 (VSS), LD73.3 (VSS), LD74.3 (VSS), LD75.3 (VSS), LD76.3 (VSS), LD77.3 (VSS), LD78.3 (VSS), LD79.3 (VSS), LD8.3 (VSS), LD80.3 (VSS), LD81.3 (VSS), LD82.3 (VSS), LD83.3 (VSS), LD84.3 (VSS), LD85.3 (VSS), LD86.3 (VSS), LD87.3 (VSS), LD88.3 (VSS), LD89.3 (VSS), LD9.3 (VSS), LD90.3 (VSS), LD91.3 (VSS), LD92.3 (VSS), LD93.3 (VSS), LD94.3 (VSS), LD95.3 (VSS), LD96.3 (VSS), LD97.3 (VSS), LD98.3 (VSS), LD99.3 (VSS)
- net LED: now also LD1.3 (DIN); no longer LD1.4 (DIN)
- new net: LD6.1 (DOUT), LD7.3 (DIN)
- new net: LD5.1 (DOUT), LD6.3 (DIN)
- new net: LD66.3 (DIN), LD67.1 (DOUT)
- new net: LD67.3 (DIN), LD68.1 (DOUT)
- new net: LD2.1 (DOUT), LD3.3 (DIN)
- new net: LD1.1 (DOUT), LD2.3 (DIN)
- new net: LD112.1 (DOUT), LD113.3 (DIN)
- new net: LD111.1 (DOUT), LD112.3 (DIN)
- new net: LD90.1 (DOUT), LD91.3 (DIN)
- new net: LD89.1 (DOUT), LD90.3 (DIN)
- new net: LD47.1 (DOUT), LD48.3 (DIN)
- new net: LD46.1 (DOUT), LD47.3 (DIN)
- new net: LD102.3 (DIN), LD103.1 (DOUT)
- new net: LD103.3 (DIN), LD104.1 (DOUT)
- new net: LD39.1 (DOUT), LD40.3 (DIN)
- new net: LD38.1 (DOUT), LD39.3 (DIN)
- new net: LD105.3 (DIN), LD106.1 (DOUT)
- new net: LD106.3 (DIN), LD107.1 (DOUT)
- new net: LD20.3 (DIN), LD21.1 (DOUT)
- new net: LD21.3 (DIN), LD22.1 (DOUT)
- new net: LD35.1 (DOUT), LD36.3 (DIN)
- new net: LD34.1 (DOUT), LD35.3 (DIN)
- new net: LD43.1 (DOUT), LD44.3 (DIN)
- new net: LD42.1 (DOUT), LD43.3 (DIN)
- new net: LD25.3 (DIN), LD26.1 (DOUT)
- new net: LD26.3 (DIN), LD27.1 (DOUT)
- new net: LD28.1 (DOUT), LD29.3 (DIN)
- new net: LD13.1 (DOUT), LD28.3 (DIN)
- new net: LD59.3 (DIN), LD60.1 (DOUT)
- new net: LD60.3 (DIN), LD61.1 (DOUT)
- new net: LD118.1 (DOUT), LD119.3 (DIN)
- new net: LD117.1 (DOUT), LD118.3 (DIN)
- new net: LD78.1 (DOUT), LD79.3 (DIN)
- new net: LD77.1 (DOUT), LD78.3 (DIN)
- new net: LD17.3 (DIN), LD18.1 (DOUT)
- new net: LD18.3 (DIN), LD19.1 (DOUT)
- new net: LD68.3 (DIN), LD69.1 (DOUT)
- new net: LD95.3 (DIN), LD96.1 (DOUT)
- new net: LD96.3 (DIN), LD97.1 (DOUT)
- new net: LD84.1 (DOUT), LD85.3 (DIN)
- new net: LD83.1 (DOUT), LD84.3 (DIN)
- new net: LD75.1 (DOUT), LD76.3 (DIN)
- new net: LD74.1 (DOUT), LD75.3 (DIN)
- new net: LD80.1 (DOUT), LD81.3 (DIN)
- new net: LD79.1 (DOUT), LD80.3 (DIN)
- new net: LD58.3 (DIN), LD59.1 (DOUT)
- new net: LD72.3 (DIN), LD73.1 (DOUT)
- new net: LD50.1 (DOUT), LD73.3 (DIN)
- new net: LD101.3 (DIN), LD102.1 (DOUT)
- new net: LD110.3 (DIN), LD92.1 (DOUT)
- new net: LD91.1 (DOUT), LD92.3 (DIN)
- new net: LD108.3 (DIN), LD109.1 (DOUT)
- new net: LD109.3 (DIN), LD110.1 (DOUT)
- new net: LD33.1 (DOUT), LD34.3 (DIN)
- new net: LD93.3 (DIN), LD94.1 (DOUT)
- new net: LD94.3 (DIN), LD95.1 (DOUT)
- new net: LD121.1 (DOUT), LD122.3 (DIN)
- new net: LD120.1 (DOUT), LD121.3 (DIN)
- new net: LD100.3 (DIN), LD101.1 (DOUT)
- new net: LD111.3 (DIN), LD93.1 (DOUT)
- new net: LD52.3 (DIN), LD53.1 (DOUT)
- new net: LD53.3 (DIN), LD54.1 (DOUT)
- new net: LD37.1 (DOUT), LD38.3 (DIN)
- new net: LD124.1 (DOUT), LD125.3 (DIN)
- new net: LD123.1 (DOUT), LD124.3 (DIN)
- new net: LD107.3 (DIN), LD108.1 (DOUT)
- new net: LD51.3 (DIN), LD52.1 (DOUT)
- new net: LD10.3 (DIN), LD9.1 (DOUT)
- new net: LD8.1 (DOUT), LD9.3 (DIN)
- new net: LD23.3 (DIN), LD24.1 (DOUT)
- new net: LD24.3 (DIN), LD25.1 (DOUT)
- new net: LD45.1 (DOUT), LD46.3 (DIN)
- new net: LD44.1 (DOUT), LD45.3 (DIN)
- new net: LD69.3 (DIN), LD70.1 (DOUT)
- new net: LD119.1 (DOUT), LD120.3 (DIN)
- new net: LD32.1 (DOUT), LD33.3 (DIN)
- new net: LD31.1 (DOUT), LD32.3 (DIN)
- new net: LD126.1 (DOUT), LD127.3 (DIN)
- new net: LD61.3 (DIN), LD62.1 (DOUT)
- new net: LD62.3 (DIN), LD63.1 (DOUT)
- new net: LD49.1 (DOUT), LD50.3 (DIN)
- new net: LD100.1 (DOUT), LD99.3 (DIN)
- new net: LD97.3 (DIN), LD98.1 (DOUT)
- new net: LD85.1 (DOUT), LD86.3 (DIN)
- new net: LD81.1 (DOUT), LD82.3 (DIN)
- new net: LD122.1 (DOUT), LD123.3 (DIN)
- new net: LD14.3 (DIN), LD15.1 (DOUT)
- new net: LD15.3 (DIN), LD16.1 (DOUT)
- new net: LD51.1 (DOUT), LD74.3 (DIN)
- new net: LD76.1 (DOUT), LD77.3 (DIN)
- new net: LD30.1 (DOUT), LD31.3 (DIN)
- new net: LD41.1 (DOUT), LD42.3 (DIN)
- new net: LD54.3 (DIN), LD55.1 (DOUT)
- new net: LD71.3 (DIN), LD72.1 (DOUT)
- new net: LD65.3 (DIN), LD66.1 (DOUT)
- new net: LD22.3 (DIN), LD23.1 (DOUT)
- new net: LD12.1 (DOUT), LD27.3 (DIN)
- new net: LD11.1 (DOUT), LD12.3 (DIN)
- new net: LD116.1 (DOUT), LD117.3 (DIN)
- new net: LD115.1 (DOUT), LD116.3 (DIN)
- new net: LD125.1 (DOUT), LD126.3 (DIN)
- new net: LD98.3 (DIN), LD99.1 (DOUT)
- new net: LD70.3 (DIN), LD71.1 (DOUT)
- new net: LD104.3 (DIN), LD105.1 (DOUT)
- new net: LD4.1 (DOUT), LD5.3 (DIN)
- new net: LD3.1 (DOUT), LD4.3 (DIN)
- new net: LD114.1 (DOUT), LD115.3 (DIN)
- new net: LD40.1 (DOUT), LD41.3 (DIN)
- new net: LD88.1 (DOUT), LD89.3 (DIN)
- new net: LD87.1 (DOUT), LD88.3 (DIN)
- new net: LD86.1 (DOUT), LD87.3 (DIN)
- new net: LD57.3 (DIN), LD58.1 (DOUT)
- new net: LD36.1 (DOUT), LD37.3 (DIN)
- new net: LD16.3 (DIN), LD17.1 (DOUT)
- new net: LD55.3 (DIN), LD56.1 (DOUT)
- new net: LD56.3 (DIN), LD57.1 (DOUT)
- new net: LD113.1 (DOUT), LD114.3 (DIN)
- new net: LD82.1 (DOUT), LD83.3 (DIN)
- new net: LD10.1 (DOUT), LD11.3 (DIN)
- new net: LD7.1 (DOUT), LD8.3 (DIN)
- new net: LD48.1 (DOUT), LD49.3 (DIN)
- new net: LD63.3 (DIN), LD64.1 (DOUT)
- new net: LD29.1 (DOUT), LD30.3 (DIN)
- new net: LD13.3 (DIN), LD14.1 (DOUT)
- new net: LD19.3 (DIN), LD20.1 (DOUT)
- new net: LD64.3 (DIN), LD65.1 (DOUT)

Commit message: Final Warning begins. Sweet Business done.
Parts:
- added K124.2, K73.2: OmniSwitch, EDI:SW_MX, symbol HL-Mk3-rescue:KEYSW-keyboard_parts-HL-Mk2-rescue
- LD1, LD10, LD100, LD101, LD102, LD103, LD104, LD105, LD106, LD107, LD108, LD109, LD11, LD110, LD111, LD112, LD113, LD114, LD115, LD116, LD117, LD118, LD119, LD12, LD120, LD121, LD122, LD123, LD124, LD125, LD126, LD127, LD13, LD14, LD15, LD16, LD17, LD18, LD19, LD2, LD20, LD21, LD22, LD23, LD24, LD25, LD26, LD27, LD28, LD29, LD3, LD30, LD31, LD32, LD33, LD34, LD35, LD36, LD37, LD38, LD39, LD4, LD40, LD41, LD42, LD43, LD44, LD45, LD46, LD47, LD48, LD49, LD5, LD50, LD51, LD52, LD53, LD54, LD55, LD56, LD57, LD58, LD59, LD6, LD60, LD61, LD62, LD63, LD64, LD65, LD66, LD67, LD68, LD69, LD7, LD70, LD71, LD72, LD73, LD74, LD75, LD76, LD77, LD78, LD79, LD8, LD80, LD81, LD82, LD83, LD84, LD85, LD86, LD87, LD88, LD89, LD9, LD90, LD91, LD92, LD93, LD94, LD95, LD96, LD97, LD98, LD99: footprint EDI:WS2812B_2020 -> EDI:WS2812C_2020
Connections:
- net col9: now also K124.2.1
- net colB: now also K73.2.1
- net at D73.2 (A), K73.2: now also K73.2.2
- net at D124.2 (A), K124.2: now also K124.2.2
